File: PDU-Board/PDU-Board.sch (KiCad schematic (older format))
At the start: 7 parts, among them J0 Main Feed, J1 Motor-1, J2 Motor-2, J3 Mother Board, U0 VICOR-DC-DC, U1 VICOR-DC-DC

Commit message: little fixes on PDB
Parts:
- removed 30A1: Fuse, Vicor:30a Fuse, symbol Device:Fuse
- added U?: VICOR-DC-DC, Vicor:Vicor-DCDC-Q, symbol PDU-Board-rescue:VICOR-DC-DC-PDU-Board-cache
- U0, U1: symbol PDU-Board-cache:VICOR-DC-DC -> PDU-Board-rescue:VICOR-DC-DC-PDU-Board-cache
Connections:
- net labels removed: 12v-Gnd, 48v, 48v-Gnd
- wire segments 42 -> 9
Changed lines of the file:
@@
 $EndComp
 $Comp
-L PDU-Board-cache:VICOR-DC-DC U1
+L PDU-Board-rescue:VICOR-DC-DC-PDU-Board-cache U1
 U 1 1 5BE0F800
-P 4800 3750
-F 0 "U1" H 4725 4415 50  0000 C CNN
-F 1 "VICOR-DC-DC" H 4725 4324 50  0000 C CNN
-F 2 "Vicor:Vicor-DCDC-Q" H 4800 3750 50  0001 C CNN
-F 3 "" H 4800 3750 50  0001 C CNN
-	1    4800 3750
+P 4775 4250
+F 0 "U1" H 4775 4825 50  0000 C CNN
+F 1 "VICOR-DC-DC" H 4725 3875 50  0000 C CNN
+F 2 "Vicor:Vicor-DCDC-Q" H 4775 4250 50  0001 C CNN
+F 3 "" H 4775 4250 50  0001 C CNN
+	1    4775 4250
 	1    0    0    1
 $EndComp
-Wire Wire Line
-	2850 3350 3500 3350
-Wire Wire Line
-	6500 3350 5900 3350
-Connection ~ 5900 3350
-Wire Wire Line
-	5900 3900 6500 3900
-Wire Wire Line
-	6100 4000 6500 4000
-Wire Wire Line
-	6100 3450 6500 3450
-Wire Wire Line
-	6100 2950 6500 2950
-Connection ~ 6100 3450
-Wire Wire Line
-	6100 2950 6100 3250
-Connection ~ 6100 3250
-Wire Wire Line
-	6100 3250 6100 3450
 $Comp
-L Device:Fuse 30A1
-U 1 1 5BE135F8
-P 3250 3750
-F 0 "30A1" V 3053 3750 50  0000 C CNN
-F 1 "Fuse" V 3144 3750 50  0000 C CNN
-F 2 "Vicor:30a Fuse" V 3180 3750 50  0001 C CNN
-F 3 "~" H 3250 3750 50  0001 C CNN
-	1    3250 3750
-	0    -1   1    0
-$EndComp
-Wire Wire Line
-	3100 3450 3100 3750
-Wire Wire Line
-	3400 3750 3650 3750
-Wire Wire Line
-	5450 3250 6100 3250
-$Comp
-L PDU-Board-cache:VICOR-DC-DC U0
+L PDU-Board-rescue:VICOR-DC-DC-PDU-Board-cache U0
 U 1 1 5BE0F643
 P 4800 2850
@@
 $EndComp
 Wire Wire Line
-	3500 2700 4000 2700
-Wire Wire Line
-	3500 2700 3500 3350
-Wire Wire Line
-	3650 3750 3650 3150
-Wire Wire Line
-	3650 3150 4150 3150
-Wire Wire Line
-	3650 3750 3650 4050
-Wire Wire Line
-	3650 4050 4150 4050
-Connection ~ 3650 3750
-Wire Wire Line
-	3500 3350 3500 3600
-Wire Wire Line
-	3500 3600 4050 3600
-Connection ~ 3500 3350
-Wire Wire Line
 	4150 3850 4050 3850
 Wire Wire Line
 	4050 3850 4050 3600
-Connection ~ 4050 3600
 Wire Wire Line
 	4050 3600 4150 3600
-Wire Wire Line
-	4150 2950 4000 2950
-Wire Wire Line
-	4000 2950 4000 2700
-Connection ~ 4000 2700
-Wire Wire Line
-	4000 2700 4150 2700
 Wire Wire Line
 	5450 2850 5300 2850
 Wire Wire Line
 	5450 2850 5450 3250
-Wire Wire Line
-	5900 3350 5900 3900
-Wire Wire Line
-	5300 3750 6100 3750
-Wire Wire Line
-	6100 3450 6100 3750
-Connection ~ 6100 3750
-Wire Wire Line
-	6100 3750 6100 4000
-Wire Wire Line
-	5900 3900 5900 4100
-Wire Wire Line
-	5900 4100 5300 4100
-Connection ~ 5900 3900
-Wire Wire Line
-	5300 3200 5900 3200
-Wire Wire Line
-	5900 3200 5900 3350
-Wire Wire Line
-	5900 2850 5900 3200
-Wire Wire Line
-	6500 2850 5900 2850
-Connection ~ 5900 3200
-Text GLabel 3500 2800 0    50   Input ~ 0
-48v-Gnd
-Text GLabel 3650 3950 2    50   Input ~ 0
-48v
-Text GLabel 5900 4100 2    50   Input ~ 0
-12v-Gnd
 Text GLabel 5450 3000 0    50   Input ~ 0
 12v
@@
 Wire Wire Line
 	2800 3300 2800 3450
-Wire Wire Line
-	2800 3450 3100 3450
+$Comp
+L PDU-Board-rescue:VICOR-DC-DC-PDU-Board-cache U?
+U 1 1 5C2557D7
+P 6175 2050
+F 0 "U?" H 6100 1585 50  0000 C CNN
+F 1 "VICOR-DC-DC" H 6100 1676 50  0000 C CNN
+F 2 "Vicor:Vicor-DCDC-Q" H 6175 2050 50  0001 C CNN
+F 3 "" H 6175 2050 50  0001 C CNN
+	1    6175 2050
+	1    0    0    1
+$EndComp
 $EndSCHEMATC
