File: PDU-Board/PDU-Board.sch (KiCad schematic (older format))
At the start: 7 parts, among them J0 Main Feed, J1 Motor-1, J2 Motor-2, J3 Mother Board, U0 VICOR-DC-DC, U1 VICOR-DC-DC

Commit message: PDU Board work
Parts:
- removed 30A1: Fuse, Vicor:30a Fuse, symbol Device:Fuse
- removed U0, U1: VICOR-DC-DC, Vicor:Vicor-DCDC-Q, symbol PDU-Board-cache:VICOR-DC-DC
- added F1: 30a, Fuse:Fuse_1206_3216Metric, symbol Device:Fuse
- added U1, U2, U3, U4: VICOR-DC-DC, Vicor:VICOR_VIA_DCM3414, symbol Vicor-Q-DCDC:VICOR-DC-DC
- J0, J1, J2, J3: symbol Connector:Conn_01x02_Female -> Connector_Generic:Conn_01x02
Connections:
- net labels added: +12V, +48V, 48v_GND, GND
- net labels removed: 12v, 12v-Gnd, 48v, 48v-Gnd
- wire segments 42 -> 0

Commit message: Begun PDU layout
Parts:
- removed F1: 30a, Fuse:Fuse_1206_3216Metric, symbol Device:Fuse
Changed lines of the file:
@@
-$EndComp
-$Comp
-L Device:Fuse F1
-U 1 1 5C2EAB10
-P 3100 3100
-F 0 "F1" V 3200 3150 50  0000 C CNN
-F 1 "30a" V 3200 3000 50  0000 C CNN
-F 2 "Fuse:Fuse_1206_3216Metric" V 3030 3100 50  0001 C CNN
-F 3 "~" H 3100 3100 50  0001 C CNN
-	1    3100 3100
-	0    1    1    0
 $EndComp
 $Comp
 L power:+48V #PWR0101
 U 1 1 5C2EAE50
-P 3250 3100
-F 0 "#PWR0101" H 3250 2950 50  0001 C CNN
-F 1 "+48V" V 3265 3228 50  0000 L CNN
-F 2 "" H 3250 3100 50  0001 C CNN
-F 3 "" H 3250 3100 50  0001 C CNN
-	1    3250 3100
+P 2950 3100
+F 0 "#PWR0101" H 2950 2950 50  0001 C CNN
+F 1 "+48V" V 2965 3228 50  0000 L CNN
+F 2 "" H 2950 3100 50  0001 C CNN
+F 3 "" H 2950 3100 50  0001 C CNN
+	1    2950 3100
 	0    1    1    0
 $EndComp
@@
 $EndComp
 $Comp
-L power:+12V #PWR?
+L power:+12V #PWR0114
 U 1 1 5C2EB697
 P 5450 4950
-F 0 "#PWR?" H 5450 4800 50  0001 C CNN
+F 0 "#PWR0114" H 5450 4800 50  0001 C CNN
 F 1 "+12V" V 5465 5078 50  0000 L CNN
 F 2 "" H 5450 4950 50  0001 C CNN
@@
 $EndComp
 $Comp
-L power:+48V #PWR?
+L power:+48V #PWR0115
 U 1 1 5C2EB69D
 P 4300 4950
-F 0 "#PWR?" H 4300 4800 50  0001 C CNN
+F 0 "#PWR0115" H 4300 4800 50  0001 C CNN
 F 1 "+48V" V 4315 5078 50  0000 L CNN
 F 2 "" H 4300 4950 50  0001 C CNN
@@
 48v_GND
 $Comp
-L power:GND #PWR?
+L power:GND #PWR0116
 U 1 1 5C2EB6A4
 P 5450 5300
-F 0 "#PWR?" H 5450 5050 50  0001 C CNN
+F 0 "#PWR0116" H 5450 5050 50  0001 C CNN
 F 1 "GND" V 5455 5172 50  0000 R CNN
 F 2 "" H 5450 5300 50  0001 C CNN
@@
 $EndComp
 $Comp
-L power:+12V #PWR?
+L power:+12V #PWR0117
 U 1 1 5C2EB8DE
 P 5450 6000
-F 0 "#PWR?" H 5450 5850 50  0001 C CNN
+F 0 "#PWR0117" H 5450 5850 50  0001 C CNN
 F 1 "+12V" V 5465 6128 50  0000 L CNN
 F 2 "" H 5450 6000 50  0001 C CNN
@@
 $EndComp
 $Comp
-L power:+48V #PWR?
+L power:+48V #PWR0118
 U 1 1 5C2EB8E4
 P 4300 6000
-F 0 "#PWR?" H 4300 5850 50  0001 C CNN
+F 0 "#PWR0118" H 4300 5850 50  0001 C CNN
 F 1 "+48V" V 4315 6128 50  0000 L CNN
 F 2 "" H 4300 6000 50  0001 C CNN
@@
 48v_GND
 $Comp
-L power:GND #PWR?
+L power:GND #PWR0119
 U 1 1 5C2EB8EB
 P 5450 6350
-F 0 "#PWR?" H 5450 6100 50  0001 C CNN
+F 0 "#PWR0119" H 5450 6100 50  0001 C CNN
 F 1 "GND" V 5455 6222 50  0000 R CNN
 F 2 "" H 5450 6350 50  0001 C CNN
@@
 	0    -1   -1   0
 $EndComp
+$Comp
+L power:+12V #PWR0120
+U 1 1 5C3063DA
+P 5900 1950
+F 0 "#PWR0120" H 5900 1800 50  0001 C CNN
+F 1 "+12V" V 5915 2078 50  0000 L CNN
+F 2 "" H 5900 1950 50  0001 C CNN
+F 3 "" H 5900 1950 50  0001 C CNN
+	1    5900 1950
+	-1   0    0    1
+$EndComp
+$Comp
+L power:GND #PWR0121
+U 1 1 5C3063F5
+P 6350 1950
+F 0 "#PWR0121" H 6350 1700 50  0001 C CNN
+F 1 "GND" V 6355 1822 50  0000 R CNN
+F 2 "" H 6350 1950 50  0001 C CNN
+F 3 "" H 6350 1950 50  0001 C CNN
+	1    6350 1950
+	1    0    0    -1
+$EndComp
+$Comp
+L power:+48V #PWR0122
+U 1 1 5C306410
+P 5450 1950
+F 0 "#PWR0122" H 5450 1800 50  0001 C CNN
+F 1 "+48V" V 5465 2078 50  0000 L CNN
+F 2 "" H 5450 1950 50  0001 C CNN
+F 3 "" H 5450 1950 50  0001 C CNN
+	1    5450 1950
+	-1   0    0    1
+$EndComp
+$Comp
+L power:PWR_FLAG #FLG0101
+U 1 1 5C30649D
+P 5450 1950
+F 0 "#FLG0101" H 5450 2025 50  0001 C CNN
+F 1 "PWR_FLAG" H 5450 2124 50  0000 C CNN
+F 2 "" H 5450 1950 50  0001 C CNN
+F 3 "~" H 5450 1950 50  0001 C CNN
+	1    5450 1950
+	1    0    0    -1
+$EndComp
+$Comp
+L power:PWR_FLAG #FLG0102
+U 1 1 5C306651
+P 5900 1950
+F 0 "#FLG0102" H 5900 2025 50  0001 C CNN
+F 1 "PWR_FLAG" H 5900 2124 50  0000 C CNN
+F 2 "" H 5900 1950 50  0001 C CNN
+F 3 "~" H 5900 1950 50  0001 C CNN
+	1    5900 1950
+	1    0    0    -1
+$EndComp
+$Comp
+L power:PWR_FLAG #FLG0103
+U 1 1 5C30666C
+P 6350 1950
+F 0 "#FLG0103" H 6350 2025 50  0001 C CNN
+F 1 "PWR_FLAG" H 6350 2124 50  0000 C CNN
+F 2 "" H 6350 1950 50  0001 C CNN
+F 3 "~" H 6350 1950 50  0001 C CNN
+	1    6350 1950
+	1    0    0    -1
+$EndComp
 $EndSCHEMATC

Commit message: Finalzed Boards ready for production
YEah
Parts:
- added J4: RJ45, Connectors:RJ45_8, symbol Connector:RJ45
- added MH1, MH2, MH3, MH4: MountingHole, Blue_ESC:MountingHole_3mm_custom, symbol Mechanical:MountingHole
- added U5, U6: ESC:TMP235A2DBZT, TO_SOT_Packages_SMD:SOT-23, symbol TMP235:ESC:TMP235A2DBZT
Connections:
- net labels added: +3.3V, Ext_Temp_0, Ext_Temp_1
- no-connect marks 0 -> 4
Changed lines of the file:
@@
+	1    0    0    -1
+$EndComp
+$Comp
+L Connector:RJ45 J4
+U 1 1 5C32F03A
+P 9450 4000
+F 0 "J4" V 9552 3570 50  0000 R CNN
+F 1 "RJ45" V 9461 3570 50  0000 R CNN
+F 2 "Connectors:RJ45_8" V 9450 4025 50  0001 C CNN
+F 3 "~" V 9450 4025 50  0001 C CNN
+	1    9450 4000
+	0    -1   -1   0
+$EndComp
+$Comp
+L ESC-Board-cache:+3.3V #PWR0123
+U 1 1 5C330122
+P 9450 3600
+F 0 "#PWR0123" H 9450 3450 50  0001 C CNN
+F 1 "+3.3V" V 9450 3850 50  0000 C CNN
+F 2 "" H 9450 3600 50  0001 C CNN
+F 3 "" H 9450 3600 50  0001 C CNN
+	1    9450 3600
+	1    0    0    -1
+$EndComp
+Text GLabel 9350 3600 1    50   Input ~ 0
+Ext_Temp_0
+Text GLabel 9250 3600 1    50   Input ~ 0
+Ext_Temp_1
+$Comp
+L power:GND #PWR0124
+U 1 1 5C330F45
+P 9550 3600
+F 0 "#PWR0124" H 9550 3350 50  0001 C CNN
+F 1 "GND" V 9550 3400 50  0000 C CNN
+F 2 "" H 9550 3600 50  0001 C CNN
+F 3 "" H 9550 3600 50  0001 C CNN
+	1    9550 3600
+	-1   0    0    1
+$EndComp
+$Comp
+L power:GND #PWR0125
+U 1 1 5C330FC9
+P 9650 2750
+F 0 "#PWR0125" H 9650 2500 50  0001 C CNN
+F 1 "GND" V 9650 2550 50  0000 C CNN
+F 2 "" H 9650 2750 50  0001 C CNN
+F 3 "" H 9650 2750 50  0001 C CNN
+	1    9650 2750
+	0    1    1    0
+$EndComp
+$Comp
+L power:GND #PWR0126
+U 1 1 5C3312D5
+P 8300 2750
+F 0 "#PWR0126" H 8300 2500 50  0001 C CNN
+F 1 "GND" V 8300 2550 50  0000 C CNN
+F 2 "" H 8300 2750 50  0001 C CNN
+F 3 "" H 8300 2750 50  0001 C CNN
+	1    8300 2750
+	0    1    1    0
+$EndComp
+NoConn ~ 9750 3600
+NoConn ~ 9650 3600
+NoConn ~ 9150 3600
+NoConn ~ 9050 3600
+Text GLabel 9150 2600 2    50   Input ~ 0
+Ext_Temp_1
+Text GLabel 10500 2600 2    50   Input ~ 0
+Ext_Temp_0
+$Comp
+L ESC-Board-cache:+3.3V #PWR0127
+U 1 1 5C331877
+P 8300 2450
+F 0 "#PWR0127" H 8300 2300 50  0001 C CNN
+F 1 "+3.3V" V 8300 2700 50  0000 C CNN
+F 2 "" H 8300 2450 50  0001 C CNN
+F 3 "" H 8300 2450 50  0001 C CNN
+	1    8300 2450
+	0    -1   -1   0
+$EndComp
+$Comp
+L ESC-Board-cache:+3.3V #PWR0128
+U 1 1 5C3318B9
+P 9650 2450
+F 0 "#PWR0128" H 9650 2300 50  0001 C CNN
+F 1 "+3.3V" V 9650 2700 50  0000 C CNN
+F 2 "" H 9650 2450 50  0001 C CNN
+F 3 "" H 9650 2450 50  0001 C CNN
+	1    9650 2450
+	0    -1   -1   0
+$EndComp
+$Comp
+L Mechanical:MountingHole MH1
+U 1 1 5C331EC5
+P 8550 4800
+F 0 "MH1" H 8650 4846 50  0000 L CNN
+F 1 "MountingHole" H 8650 4755 50  0000 L CNN
+F 2 "Blue_ESC:MountingHole_3mm_custom" H 8550 4800 50  0001 C CNN
+F 3 "~" H 8550 4800 50  0001 C CNN
+	1    8550 4800
+	1    0    0    -1
+$EndComp
+$Comp
+L Mechanical:MountingHole MH2
+U 1 1 5C332065
+P 8550 5000
+F 0 "MH2" H 8650 5046 50  0000 L CNN
+F 1 "MountingHole" H 8650 4955 50  0000 L CNN
+F 2 "Blue_ESC:MountingHole_3mm_custom" H 8550 5000 50  0001 C CNN
+F 3 "~" H 8550 5000 50  0001 C CNN
+	1    8550 5000
+	1    0    0    -1
+$EndComp
+$Comp
+L Mechanical:MountingHole MH3
+U 1 1 5C33209F
+P 8550 5200
+F 0 "MH3" H 8650 5246 50  0000 L CNN
+F 1 "MountingHole" H 8650 5155 50  0000 L CNN
+F 2 "Blue_ESC:MountingHole_3mm_custom" H 8550 5200 50  0001 C CNN
+F 3 "~" H 8550 5200 50  0001 C CNN
+	1    8550 5200
+	1    0    0    -1
+$EndComp
+$Comp
+L Mechanical:MountingHole MH4
+U 1 1 5C3320EB
+P 8550 5400
+F 0 "MH4" H 8650 5446 50  0000 L CNN
+F 1 "MountingHole" H 8650 5355 50  0000 L CNN
+F 2 "Blue_ESC:MountingHole_3mm_custom" H 8550 5400 50  0001 C CNN
+F 3 "~" H 8550 5400 50  0001 C CNN
+	1    8550 5400
+	1    0    0    -1
+$EndComp
+$Comp
+L TMP235:ESC:TMP235A2DBZT U5
+U 1 1 5C333407
+P 8750 2600
+F 0 "U5" H 8725 3015 50  0000 C CNN
+F 1 "ESC:TMP235A2DBZT" H 8725 2924 50  0000 C CNN
+F 2 "TO_SOT_Packages_SMD:SOT-23" H 8950 2650 50  0001 C CNN
+F 3 "" H 8950 2650 50  0001 C CNN
+	1    8750 2600
+	1    0    0    -1
+$EndComp
+$Comp
+L TMP235:ESC:TMP235A2DBZT U6
+U 1 1 5C333447
+P 10100 2600
+F 0 "U6" H 10075 3015 50  0000 C CNN
+F 1 "ESC:TMP235A2DBZT" H 10075 2924 50  0000 C CNN
+F 2 "TO_SOT_Packages_SMD:SOT-23" H 10300 2650 50  0001 C CNN
+F 3 "" H 10300 2650 50  0001 C CNN
+	1    10100 2600
 	1    0    0    -1
 $EndComp

Commit message: Re designed PDU pre mec spec
Parts:
- removed MH1, MH2, MH3, MH4: MountingHole, Blue_ESC:MountingHole_3mm_custom, symbol Mechanical:MountingHole
- added J5: RJ45, Connectors:RJ45_8, symbol Connector:RJ45
- U5, U6: symbol TMP235:ESC:TMP235A2DBZT -> TMP235:ESC_TMP235A2DBZT
Connections:
- wire segments 0 -> 8
Changed lines of the file:
@@
 	0    1    1    0
 $EndComp
-NoConn ~ 9750 3600
-NoConn ~ 9650 3600
 NoConn ~ 9150 3600
 NoConn ~ 9050 3600
@@
 $EndComp
 $Comp
-L Mechanical:MountingHole MH1
-U 1 1 5C331EC5
-P 8550 4800
-F 0 "MH1" H 8650 4846 50  0000 L CNN
-F 1 "MountingHole" H 8650 4755 50  0000 L CNN
-F 2 "Blue_ESC:MountingHole_3mm_custom" H 8550 4800 50  0001 C CNN
-F 3 "~" H 8550 4800 50  0001 C CNN
-	1    8550 4800
-	1    0    0    -1
-$EndComp
-$Comp
-L Mechanical:MountingHole MH2
-U 1 1 5C332065
-P 8550 5000
-F 0 "MH2" H 8650 5046 50  0000 L CNN
-F 1 "MountingHole" H 8650 4955 50  0000 L CNN
-F 2 "Blue_ESC:MountingHole_3mm_custom" H 8550 5000 50  0001 C CNN
-F 3 "~" H 8550 5000 50  0001 C CNN
-	1    8550 5000
-	1    0    0    -1
-$EndComp
-$Comp
-L Mechanical:MountingHole MH3
-U 1 1 5C33209F
-P 8550 5200
-F 0 "MH3" H 8650 5246 50  0000 L CNN
-F 1 "MountingHole" H 8650 5155 50  0000 L CNN
-F 2 "Blue_ESC:MountingHole_3mm_custom" H 8550 5200 50  0001 C CNN
-F 3 "~" H 8550 5200 50  0001 C CNN
-	1    8550 5200
-	1    0    0    -1
-$EndComp
-$Comp
-L Mechanical:MountingHole MH4
-U 1 1 5C3320EB
-P 8550 5400
-F 0 "MH4" H 8650 5446 50  0000 L CNN
-F 1 "MountingHole" H 8650 5355 50  0000 L CNN
-F 2 "Blue_ESC:MountingHole_3mm_custom" H 8550 5400 50  0001 C CNN
-F 3 "~" H 8550 5400 50  0001 C CNN
-	1    8550 5400
-	1    0    0    -1
-$EndComp
-$Comp
-L TMP235:ESC:TMP235A2DBZT U5
+L TMP235:ESC_TMP235A2DBZT U5
 U 1 1 5C333407
 P 8750 2600
@@
 $EndComp
 $Comp
-L TMP235:ESC:TMP235A2DBZT U6
+L TMP235:ESC_TMP235A2DBZT U6
 U 1 1 5C333447
 P 10100 2600
@@
 	1    0    0    -1
 $EndComp
+$Comp
+L Connector:RJ45 J5
+U 1 1 5C4E792D
+P 9450 5600
+F 0 "J5" V 9552 5170 50  0000 R CNN
+F 1 "RJ45" V 9461 5170 50  0000 R CNN
+F 2 "Connectors:RJ45_8" V 9450 5625 50  0001 C CNN
+F 3 "~" V 9450 5625 50  0001 C CNN
+	1    9450 5600
+	0    -1   -1   0
+$EndComp
+Text GLabel 9250 5200 1    50   Input ~ 0
+Ext_Temp_1
+Text GLabel 9350 5200 1    50   Input ~ 0
+Ext_Temp_0
+$Comp
+L ESC-Board-cache:+3.3V #PWR0129
+U 1 1 5C4E7B27
+P 9450 5200
+F 0 "#PWR0129" H 9450 5050 50  0001 C CNN
+F 1 "+3.3V" V 9450 5450 50  0000 C CNN
+F 2 "" H 9450 5200 50  0001 C CNN
+F 3 "" H 9450 5200 50  0001 C CNN
+	1    9450 5200
+	1    0    0    -1
+$EndComp
+$Comp
+L power:GND #PWR0130
+U 1 1 5C4E7B4A
+P 9550 5200
+F 0 "#PWR0130" H 9550 4950 50  0001 C CNN
+F 1 "GND" V 9550 5000 50  0000 C CNN
+F 2 "" H 9550 5200 50  0001 C CNN
+F 3 "" H 9550 5200 50  0001 C CNN
+	1    9550 5200
+	-1   0    0    1
+$EndComp
+Wire Wire Line
+	9750 3600 10250 3600
+Wire Wire Line
+	10250 3600 10250 5200
+Wire Wire Line
+	10250 5200 9750 5200
+Wire Wire Line
+	9650 5200 9650 5100
+Wire Wire Line
+	9650 5100 10350 5100
+Wire Wire Line
+	10350 5100 10350 3550
+Wire Wire Line
+	10350 3550 9650 3550
+Wire Wire Line
+	9650 3550 9650 3600
+NoConn ~ 9150 5200
+NoConn ~ 9050 5200
 $EndSCHEMATC

Commit message: Updated PDU and ESC for leak sensor
Connections:
- net labels added: Water_Sensor
- no-connect marks 4 -> 2
Changed lines of the file:
@@
 	0    1    1    0
 $EndComp
-NoConn ~ 9150 3600
 NoConn ~ 9050 3600
 Text GLabel 9150 2600 2    50   Input ~ 0
@@
 Wire Wire Line
 	9650 3550 9650 3600
-NoConn ~ 9150 5200
 NoConn ~ 9050 5200
+Text GLabel 9150 5200 1    50   Input ~ 0
+Water_Sensor
+Text GLabel 9150 3600 1    50   Input ~ 0
+Water_Sensor
 $EndSCHEMATC

Commit message: Added 5v
Connections:
- wire segments 8 -> 11
- no-connect marks 2 -> 0
Changed lines of the file:
@@
 	0    1    1    0
 $EndComp
-NoConn ~ 9050 3600
 Text GLabel 9150 2600 2    50   Input ~ 0
 Ext_Temp_1
@@
 Wire Wire Line
 	9650 3550 9650 3600
-NoConn ~ 9050 5200
 Text GLabel 9150 5200 1    50   Input ~ 0
 Water_Sensor
 Text GLabel 9150 3600 1    50   Input ~ 0
 Water_Sensor
+Wire Wire Line
+	9050 3600 8650 3600
+Wire Wire Line
+	8650 3600 8650 5200
+Wire Wire Line
+	8650 5200 9050 5200
 $EndSCHEMATC
