File: ESC-Board/ESC-Board.sch (KiCad schematic (older format))
At the start: 19 parts, among them J1 XT_60, P1 Conn_01x06_Female, P2 Conn_01x06_Female, U1 Blue_ESC, U2 Blue_ESC, U3 Blue_ESC, U4 Blue_ESC

Commit message: basic fix
Connections:
- net labels added: GND
- wire segments 92 -> 87
Changed lines of the file:
@@
 	1    0    0    -1
 $EndComp
-Text GLabel 1950 4000 1    50   Input ~ 0
-PWM_Ground
-Text GLabel 10500 1000 0    50   Input ~ 0
-12v_Ground
 Text GLabel 10500 900  0    50   Input ~ 0
 12v_Power
@@
 Text GLabel 10700 2450 1    50   Input ~ 0
 PWM_Ground
-Text GLabel 3600 4000 1    50   Input ~ 0
-PWM_Ground
-Text GLabel 5450 4050 1    50   Input ~ 0
-PWM_Ground
-Text GLabel 7000 4050 1    50   Input ~ 0
-PWM_Ground
 Text GLabel 2150 4000 1    50   Input ~ 0
 U1_PWM
@@
 Wire Wire Line
 	10500 900  10650 900
-Wire Wire Line
-	10650 1000 10500 1000
 Wire Wire Line
 	14050 3750 14700 3750
@@
 Wire Wire Line
 	14700 3750 14900 3750
-Text GLabel 3550 2150 3    50   Input ~ 0
-Gnd
-Wire Wire Line
-	3550 2150 3550 1900
-Text GLabel 5250 2150 3    50   Input ~ 0
-Gnd
-Wire Wire Line
-	5250 2150 5250 1900
-Text GLabel 1850 2150 3    50   Input ~ 0
-Gnd
-Wire Wire Line
-	1850 2150 1850 1900
-Text GLabel 6950 2150 3    50   Input ~ 0
-Gnd
-Wire Wire Line
-	6950 2150 6950 1900
 Text GLabel 14650 2750 2    50   Input ~ 0
 A0
@@
 Text Notes 5000 3150 2    50   ~ 0
 ESC to Connectors\n
+$Comp
+L power:GND #PWR?
+U 1 1 5C26AD26
+P 3550 3450
+F 0 "#PWR?" H 3550 3200 50  0001 C CNN
+F 1 "GND" H 3555 3277 50  0000 C CNN
+F 2 "" H 3550 3450 50  0001 C CNN
+F 3 "" H 3550 3450 50  0001 C CNN
+	1    3550 3450
+	1    0    0    -1
+$EndComp
 $EndSCHEMATC

Commit message: Second Draft (in progress)
Starting clean up of sch
Parts:
- removed P1, P2: Conn_01x06_Female, symbol Connector:Conn_01x06_Female
- added J1, J?: Conn_01x06, symbol Connector_Generic:Conn_01x06
- F1, F2, F3, F4: value Fuse -> 10/15
- F5: value Fuse_500ma -> 500m
- U2, U4: footprint Blue_ESC:Blue_ESC -> (none)
Connections:
- net labels added: +12V, +5V, ESC_1_PWM, ESC_1_Power, ESC_2_Power, ESC_3_Power, ESC_4_Power, PWM_ESC_1
- net labels removed: +5v, U1_PWM, U1_Phase_1, U1_Phase_2, U1_Phase_3, U1_Power, U2_Phase_1, U2_Phase_2, U2_Phase_3, U2_Power, U3_Phase_1, U3_Phase_2, U3_Phase_3, U3_Power, U4_Phase_1, U4_Phase_2, U4_Phase_3, U4_Power
- wire segments 87 -> 76
- no-connect marks 0 -> 17

Commit message: Second Draft(In Progress) v2
Connections:
- net labels added: Power_ESC_1, Power_ESC_2, Power_ESC_3, Power_ESC_4
- net labels removed: 12v_Ground, 12v_Power, ESC_1_Power, ESC_2_Power, ESC_3_Power, ESC_4_Power, Gnd
- wire segments 76 -> 68
- no-connect marks 17 -> 21
Changed lines of the file:
@@
 U 1 1 5C172736
 P 13950 2750
-F 0 "A1" H 13950 1664 50  0000 C CNN
-F 1 "Arduino_Nano_v3.x" H 13950 1573 50  0000 C CNN
+F 0 "A1" H 14450 3600 50  0000 C CNN
+F 1 "Arduino_Nano_v3.x" H 14750 1900 50  0000 C CNN
 F 2 "Module:Arduino_Nano" H 14100 1800 50  0001 L CNN
 F 3 "http://www.mouser.com/pdfdocs/Gravitech_Arduino_Nano3_0.pdf" H 13950 1750 50  0001 C CNN
@@
 L Device:Fuse F5
 U 1 1 5C1BC00C
-P 13850 1450
-F 0 "F5" H 13910 1496 50  0000 L CNN
-F 1 "500m" H 13910 1405 50  0000 L CNN
-F 2 "" V 13780 1450 50  0001 C CNN
-F 3 "~" H 13850 1450 50  0001 C CNN
-	1    13850 1450
-	1    0    0    -1
-$EndComp
-Wire Wire Line
-	13850 1600 13850 1750
+P 13850 1600
+F 0 "F5" H 13900 1650 50  0000 L CNN
+F 1 "500m" H 13900 1550 50  0000 L CNN
+F 2 "" V 13780 1600 50  0001 C CNN
+F 3 "~" H 13850 1600 50  0001 C CNN
+	1    13850 1600
+	1    0    0    -1
+$EndComp
 $Comp
 L Connector:RJ45 I1
@@
 Wire Wire Line
 	12800 3150 13450 3150
-Text GLabel 12800 3750 0    50   Input ~ 0
-PWM_Ground
 Text GLabel 10700 2450 1    50   Input ~ 0
 PWM_Ground
 Text GLabel 2150 9400 0    50   Input ~ 0
 PWM_ESC_1
-Text GLabel 14900 3750 2    50   Input ~ 0
-12v_Ground
-Text GLabel 12800 1200 0    50   Input ~ 0
-12v_Power
-Wire Wire Line
-	14050 3750 14700 3750
-Wire Wire Line
-	12800 1200 13850 1200
-Wire Wire Line
-	13850 1200 13850 1300
 Wire Notes Line
 	11650 4350 11650 600
@@
 Wire Notes Line
 	15950 600  15950 4350
-Text GLabel 14900 3850 2    50   Input ~ 0
-Gnd
 Wire Notes Line
 	11500 600  9650 600
@@
 $EndComp
 Text GLabel 1400 1450 1    50   Input ~ 0
-ESC_1_Power
+Power_ESC_1
 Text GLabel 3100 1450 1    50   Input ~ 0
-ESC_2_Power
+Power_ESC_2
 Text GLabel 4800 1450 1    50   Input ~ 0
-ESC_3_Power
+Power_ESC_3
 Text GLabel 6500 1450 1    50   Input ~ 0
-ESC_4_Power
+Power_ESC_4
 Wire Wire Line
 	6500 1450 6500 1500
@@
 Wire Wire Line
 	4800 1700 4850 1700
-Wire Wire Line
-	12800 3750 13950 3750
-Wire Wire Line
-	14900 3850 14700 3850
-Wire Wire Line
-	14700 3850 14700 3750
-Connection ~ 14700 3750
-Wire Wire Line
-	14700 3750 14900 3750
 Text GLabel 14650 2750 2    50   Input ~ 0
 A0
@@
 	1    0    0    -1
 $EndComp
+$Comp
+L power:GND #PWR?
+U 1 1 5C3103D6
+P 10650 1000
+F 0 "#PWR?" H 10650 750 50  0001 C CNN
+F 1 "GND" V 10655 872 50  0000 R CNN
+F 2 "" H 10650 1000 50  0001 C CNN
+F 3 "" H 10650 1000 50  0001 C CNN
+	1    10650 1000
+	0    1    1    0
+$EndComp
+$Comp
+L power:+12V #PWR?
+U 1 1 5C3126B1
+P 13850 1450
+F 0 "#PWR?" H 13850 1300 50  0001 C CNN
+F 1 "+12V" H 13865 1623 50  0000 C CNN
+F 2 "" H 13850 1450 50  0001 C CNN
+F 3 "" H 13850 1450 50  0001 C CNN
+	1    13850 1450
+	1    0    0    -1
+$EndComp
+$Comp
+L power:+5V #PWR?
+U 1 1 5C312ED2
+P 14150 1750
+F 0 "#PWR?" H 14150 1600 50  0001 C CNN
+F 1 "+5V" H 14250 1800 50  0000 C CNN
+F 2 "" H 14150 1750 50  0001 C CNN
+F 3 "" H 14150 1750 50  0001 C CNN
+	1    14150 1750
+	1    0    0    -1
+$EndComp
+$Comp
+L power:GND #PWR?
+U 1 1 5C3168F6
+P 14050 3750
+F 0 "#PWR?" H 14050 3500 50  0001 C CNN
+F 1 "GND" H 14200 3650 50  0000 C CNN
+F 2 "" H 14050 3750 50  0001 C CNN
+F 3 "" H 14050 3750 50  0001 C CNN
+	1    14050 3750
+	1    0    0    -1
+$EndComp
+$Comp
+L power:GND #PWR?
+U 1 1 5C316D7F
+P 13950 3750
+F 0 "#PWR?" H 13950 3500 50  0001 C CNN
+F 1 "GND" H 13800 3650 50  0000 C CNN
+F 2 "" H 13950 3750 50  0001 C CNN
+F 3 "" H 13950 3750 50  0001 C CNN
+	1    13950 3750
+	1    0    0    -1
+$EndComp
+NoConn ~ 13450 2350
+NoConn ~ 13450 2250
+NoConn ~ 13450 2150
+NoConn ~ 14450 2550
+Text GLabel 2150 9900 0    50   Input ~ 0
+Power_ESC_1
+Text GLabel 2150 8250 0    50   Input ~ 0
+Power_ESC_2
+Text GLabel 2200 6400 0    50   Input ~ 0
+Power_ESC_3
+Text GLabel 2200 4850 0    50   Input ~ 0
+Power_ESC_4
 $EndSCHEMATC

Commit message: Second Draft(in progess) v3
Parts:
- removed U1, U3: Blue_ESC, Blue_ESC:Blue_ESC, symbol ESC:Blue_ESC
- removed U2, U4: Blue_ESC, symbol ESC:Blue_ESC
- added U? (x4): ESC:Blue_ESC, symbol ESC-Board-cache:ESC:Blue_ESC
Connections:
- net labels added: I2C_SDA, I2C_SLC, PWM_ESC_2, PWM_ESC_3, PWM_ESC_4
- net labels removed: ESC_1_PWM, PWM_Ground, SDA_I2c, SLC_I2c, U2_PWM, U3_PWM, U4_PWM
- wire segments 68 -> 60
Changed lines of the file:
@@
 $EndDescr
-$Comp
-L ESC:Blue_ESC U1
-U 1 1 5C16F1D7
-P 3150 9500
-F 0 "U1" V 2550 9500 50  0000 L CNN
-F 1 "Blue_ESC" V 3750 9500 50  0000 L CNN
-F 2 "Blue_ESC:Blue_ESC" H 3150 9500 50  0001 C CNN
-F 3 "" H 3150 9500 50  0001 C CNN
-	1    3150 9500
-	0    -1   -1   0
-$EndComp
-$Comp
-L ESC:Blue_ESC U2
-U 1 1 5C16F2CB
-P 3150 7850
-F 0 "U2" V 2550 7850 50  0000 L CNN
-F 1 "Blue_ESC" V 3750 7850 50  0000 L CNN
-F 2 "" H 3150 7850 50  0001 C CNN
-F 3 "" H 3150 7850 50  0001 C CNN
-	1    3150 7850
-	0    -1   -1   0
-$EndComp
-$Comp
-L ESC:Blue_ESC U3
-U 1 1 5C16F349
-P 3200 6000
-F 0 "U3" V 2600 6000 50  0000 L CNN
-F 1 "Blue_ESC" V 3800 6000 50  0000 L CNN
-F 2 "Blue_ESC:Blue_ESC" H 3200 6000 50  0001 C CNN
-F 3 "" H 3200 6000 50  0001 C CNN
-	1    3200 6000
-	0    -1   -1   0
-$EndComp
-$Comp
-L ESC:Blue_ESC U4
-U 1 1 5C16F3CD
-P 3200 4450
-F 0 "U4" V 2600 4450 50  0000 L CNN
-F 1 "Blue_ESC" V 3800 4450 50  0000 L CNN
-F 2 "" H 3200 4450 50  0001 C CNN
-F 3 "" H 3200 4450 50  0001 C CNN
-	1    3200 4450
-	0    -1   -1   0
-$EndComp
 $Comp
 L Connector:Conn_01x02_Female J1
@@
 	1    0    0    -1
 $EndComp
-Text GLabel 12800 2450 0    50   Input ~ 0
-ESC_1_PWM
-Text GLabel 12800 2750 0    50   Input ~ 0
-U2_PWM
-Text GLabel 12800 3050 0    50   Input ~ 0
-U3_PWM
-Text GLabel 12800 3150 0    50   Input ~ 0
-U4_PWM
+Text GLabel 13450 2750 0    50   Input ~ 0
+PWM_ESC_2
+Text GLabel 13450 3050 0    50   Input ~ 0
+PWM_ESC_3
+Text GLabel 13450 3150 0    50   Input ~ 0
+PWM_ESC_4
 Wire Wire Line
 	4250 9900 4800 9900
@@
 	0    -1   -1   0
 $EndComp
-Wire Wire Line
-	12800 2650 13450 2650
-Text GLabel 10900 2450 1    50   Input ~ 0
-SDA_I2c
-Text GLabel 10800 2450 1    50   Input ~ 0
-SLC_I2c
 $Comp
 L Sensor_Current:ACS780xLRTR-100U D1
@@
 	1    0    0    -1
 $EndComp
-Text GLabel 12800 2550 0    50   Input ~ 0
-SDA_I2c
-Text GLabel 12800 2650 0    50   Input ~ 0
-SLC_I2c
-Wire Wire Line
-	13450 2550 12800 2550
-Wire Wire Line
-	12800 2450 13450 2450
-Wire Wire Line
-	12800 2750 13450 2750
-Wire Wire Line
-	12800 3050 13450 3050
-Wire Wire Line
-	12800 3150 13450 3150
-Text GLabel 10700 2450 1    50   Input ~ 0
-PWM_Ground
+Text GLabel 13450 2550 0    50   Input ~ 0
+I2C_SDA
+Text GLabel 13450 2650 0    50   Input ~ 0
+I2C_SLC
 Text GLabel 2150 9400 0    50   Input ~ 0
 PWM_ESC_1
@@
 Text Notes 13600 750  0    50   ~ 0
 Ardunio Nano
-Wire Wire Line
-	10700 2450 10700 2550
 Wire Wire Line
 	10800 2450 10800 2550
@@
 	0    -1   -1   0
 $EndComp
-Text GLabel 10900 4350 1    50   Input ~ 0
-SDA_I2c
-Text GLabel 10800 4350 1    50   Input ~ 0
-SLC_I2c
-Text GLabel 10700 4350 1    50   Input ~ 0
-PWM_Ground
-Wire Wire Line
-	10700 4350 10700 4450
 Wire Wire Line
 	10800 4350 10800 4450
@@
 Text GLabel 2200 4850 0    50   Input ~ 0
 Power_ESC_4
+$Comp
+L ESC-Board-cache:ESC:Blue_ESC U?
+U 1 1 5C31FC02
+P 3200 4450
+F 0 "U?" V 3915 4400 50  0000 C CNN
+F 1 "ESC:Blue_ESC" V 3824 4400 50  0000 C CNN
+F 2 "" H 3200 4450 50  0001 C CNN
+F 3 "" H 3200 4450 50  0001 C CNN
+	1    3200 4450
+	0    -1   -1   0
+$EndComp
+$Comp
+L ESC-Board-cache:ESC:Blue_ESC U?
+U 1 1 5C324647
+P 3200 6000
+F 0 "U?" V 3915 5950 50  0000 C CNN
+F 1 "ESC:Blue_ESC" V 3824 5950 50  0000 C CNN
+F 2 "" H 3200 6000 50  0001 C CNN
+F 3 "" H 3200 6000 50  0001 C CNN
+	1    3200 6000
+	0    -1   -1   0
+$EndComp
+$Comp
+L ESC-Board-cache:ESC:Blue_ESC U?
+U 1 1 5C32481F
+P 3150 7850
+F 0 "U?" V 3865 7800 50  0000 C CNN
+F 1 "ESC:Blue_ESC" V 3774 7800 50  0000 C CNN
+F 2 "" H 3150 7850 50  0001 C CNN
+F 3 "" H 3150 7850 50  0001 C CNN
+	1    3150 7850
+	0    -1   -1   0
+$EndComp
+$Comp
+L ESC-Board-cache:ESC:Blue_ESC U?
+U 1 1 5C324A6D
+P 3150 9500
+F 0 "U?" V 3865 9450 50  0000 C CNN
+F 1 "ESC:Blue_ESC" V 3774 9450 50  0000 C CNN
+F 2 "" H 3150 9500 50  0001 C CNN
+F 3 "" H 3150 9500 50  0001 C CNN
+	1    3150 9500
+	0    -1   -1   0
+$EndComp
+Text GLabel 13450 2450 0    50   Input ~ 0
+PWM_ESC_1
+Text GLabel 10900 2450 1    50   Input ~ 0
+I2C_SDA
+Text GLabel 10900 4350 1    50   Input ~ 0
+I2C_SDA
+Text GLabel 10800 4350 1    50   Input ~ 0
+I2C_SLC
+Text GLabel 10800 2450 1    50   Input ~ 0
+I2C_SLC
+$Comp
+L power:GND #PWR?
+U 1 1 5C325D70
+P 10700 2550
+F 0 "#PWR?" H 10700 2300 50  0001 C CNN
+F 1 "GND" H 10800 2450 50  0000 C CNN
+F 2 "" H 10700 2550 50  0001 C CNN
+F 3 "" H 10700 2550 50  0001 C CNN
+	1    10700 2550
+	-1   0    0    1
+$EndComp
+$Comp
+L power:GND #PWR?
+U 1 1 5C325EAF
+P 10700 4450
+F 0 "#PWR?" H 10700 4200 50  0001 C CNN
+F 1 "GND" H 10800 4350 50  0000 C CNN
+F 2 "" H 10700 4450 50  0001 C CNN
+F 3 "" H 10700 4450 50  0001 C CNN
+	1    10700 4450
+	-1   0    0    1
+$EndComp
 $EndSCHEMATC

Commit message: Second Draft(Final version)
Alex pls
Parts:
- F1, F2, F3, F4: footprint Blue_ESC:Slow_Blow_Fuse_UST_1206 -> (none)
- I1, I2: footprint Connectors:RJ45_8 -> (none)
- J1: footprint Blue_ESC:XT60 -> (none)
- gave numbers to parts that had none: 5

Commit message: Final Draft
Parts:
- added MH1, MH2, MH3, MH4, MH5, MH6, MH7, MH8: MountingHole, symbol Mechanical:MountingHole
- J3: renamed from J1; symbol Connector:Conn_01x02_Female -> Connector_Generic:Conn_01x02
- U1, U2, U3, U4: symbol ESC-Board-cache:ESC:Blue_ESC -> ESC:Blue_ESC
Connections:
- net labels added: Current_A0, Current_A1, Current_A2, Current_A3
- net labels removed: A0, A1, A2, A3
Other:
- note added: "Mounting Holes\n"
Changed lines of the file:
@@
 $EndDescr
 $Comp
-L Connector:Conn_01x02_Female J1
+L Connector_Generic:Conn_01x02 J3
 U 1 1 5C16FC6D
 P 10850 900
-F 0 "J1" H 10878 876 50  0000 L CNN
-F 1 "XT_60" H 10878 785 50  0000 L CNN
+F 0 "J3" H 10900 1000 50  0000 L CNN
+F 1 "XT_60" H 10900 700 50  0000 L CNN
 F 2 "" H 10850 900 50  0001 C CNN
 F 3 "" H 10850 900 50  0001 C CNN
@@
 	4800 1700 4850 1700
 Text GLabel 14650 2750 2    50   Input ~ 0
-A0
+Current_A0
 Text GLabel 14650 2850 2    50   Input ~ 0
-A1
+Current_A1
 Text GLabel 14650 2950 2    50   Input ~ 0
-A2
+Current_A2
 Text GLabel 14650 3050 2    50   Input ~ 0
-A3
+Current_A3
 Wire Wire Line
 	14450 2750 14650 2750
@@
 	14650 3050 14450 3050
 Text GLabel 2250 1600 2    50   Input ~ 0
-A0
+Current_A0
 Text GLabel 3950 1600 2    50   Input ~ 0
-A1
+Current_A1
 Text GLabel 5650 1600 2    50   Input ~ 0
-A2
+Current_A2
 Text GLabel 7350 1600 2    50   Input ~ 0
-A3
+Current_A3
 Wire Notes Line
 	8300 600  8300 2800
@@
 Power_ESC_4
 $Comp
-L ESC-Board-cache:ESC:Blue_ESC U4
+L ESC:Blue_ESC U4
 U 1 1 5C31FC02
 P 3100 4000
@@
 $EndComp
 $Comp
-L ESC-Board-cache:ESC:Blue_ESC U3
+L ESC:Blue_ESC U3
 U 1 1 5C324647
 P 3100 5550
@@
 $EndComp
 $Comp
-L ESC-Board-cache:ESC:Blue_ESC U2
+L ESC:Blue_ESC U2
 U 1 1 5C32481F
 P 3050 7400
@@
 $EndComp
 $Comp
-L ESC-Board-cache:ESC:Blue_ESC U1
+L ESC:Blue_ESC U1
 U 1 1 5C324A6D
 P 3050 9050
@@
 Text GLabel 2100 3900 0    50   Input ~ 0
 PWM_ESC_4
+$Comp
+L Mechanical:MountingHole MH1
+U 1 1 5C29DF4F
+P 14500 4850
+F 0 "MH1" H 14600 4896 50  0000 L CNN
+F 1 "MountingHole" H 14600 4805 50  0000 L CNN
+F 2 "" H 14500 4850 50  0001 C CNN
+F 3 "~" H 14500 4850 50  0001 C CNN
+	1    14500 4850
+	1    0    0    -1
+$EndComp
+$Comp
+L Mechanical:MountingHole MH2
+U 1 1 5C29E098
+P 14500 5050
+F 0 "MH2" H 14600 5096 50  0000 L CNN
+F 1 "MountingHole" H 14600 5005 50  0000 L CNN
+F 2 "" H 14500 5050 50  0001 C CNN
+F 3 "~" H 14500 5050 50  0001 C CNN
+	1    14500 5050
+	1    0    0    -1
+$EndComp
+$Comp
+L Mechanical:MountingHole MH4
+U 1 1 5C29E0EA
+P 14500 5450
+F 0 "MH4" H 14600 5496 50  0000 L CNN
+F 1 "MountingHole" H 14600 5405 50  0000 L CNN
+F 2 "" H 14500 5450 50  0001 C CNN
+F 3 "~" H 14500 5450 50  0001 C CNN
+	1    14500 5450
+	1    0    0    -1
+$EndComp
+$Comp
+L Mechanical:MountingHole MH3
+U 1 1 5C29E146
+P 14500 5250
+F 0 "MH3" H 14600 5296 50  0000 L CNN
+F 1 "MountingHole" H 14600 5205 50  0000 L CNN
+F 2 "" H 14500 5250 50  0001 C CNN
+F 3 "~" H 14500 5250 50  0001 C CNN
+	1    14500 5250
+	1    0    0    -1
+$EndComp
+$Comp
+L Mechanical:MountingHole MH5
+U 1 1 5C29E1ED
+P 15250 4850
+F 0 "MH5" H 15350 4896 50  0000 L CNN
+F 1 "MountingHole" H 15350 4805 50  0000 L CNN
+F 2 "" H 15250 4850 50  0001 C CNN
+F 3 "~" H 15250 4850 50  0001 C CNN
+	1    15250 4850
+	1    0    0    -1
+$EndComp
+$Comp
+L Mechanical:MountingHole MH6
+U 1 1 5C29E245
+P 15250 5050
+F 0 "MH6" H 15350 5096 50  0000 L CNN
+F 1 "MountingHole" H 15350 5005 50  0000 L CNN
+F 2 "" H 15250 5050 50  0001 C CNN
+F 3 "~" H 15250 5050 50  0001 C CNN
+	1    15250 5050
+	1    0    0    -1
+$EndComp
+$Comp
+L Mechanical:MountingHole MH7
+U 1 1 5C29E29F
+P 15250 5250
+F 0 "MH7" H 15350 5296 50  0000 L CNN
+F 1 "MountingHole" H 15350 5205 50  0000 L CNN
+F 2 "" H 15250 5250 50  0001 C CNN
+F 3 "~" H 15250 5250 50  0001 C CNN
+	1    15250 5250
+	1    0    0    -1
+$EndComp
+$Comp
+L Mechanical:MountingHole MH8
+U 1 1 5C29E2FB
+P 15250 5450
+F 0 "MH8" H 15350 5496 50  0000 L CNN
+F 1 "MountingHole" H 15350 5405 50  0000 L CNN
+F 2 "" H 15250 5450 50  0001 C CNN
+F 3 "~" H 15250 5450 50  0001 C CNN
+	1    15250 5450
+	1    0    0    -1
+$EndComp
+Wire Notes Line
+	14250 5600 15950 5600
+Wire Notes Line
+	15950 5600 15950 4450
+Wire Notes Line
+	15950 4450 14250 4450
+Wire Notes Line
+	14250 4450 14250 5600
+Text Notes 14800 4600 0    50   ~ 0
+Mounting Holes\n
 $EndSCHEMATC
