File: ESC-Board/ESC-Board.sch (KiCad schematic (older format))
At the start: 27 parts, among them J1 Conn_01x06, J2 Conn_01x06, J3 XT_60, U1 ESC:Blue_ESC, U2 ESC:Blue_ESC, U3 ESC:Blue_ESC, U4 ESC:Blue_ESC

Commit message: Final Draft
Parts:
- J1, J2: value Conn_01x06 -> Molex
Connections:
- no-connect marks 21 -> 24
Changed lines of the file:
@@
 ESC to Connectors\n
 $Comp
-L power:GND #PWR?
+L power:GND #PWR0101
 U 1 1 5C26AD26
 P 2050 7500
-F 0 "#PWR?" H 2050 7250 50  0001 C CNN
+F 0 "#PWR0101" H 2050 7250 50  0001 C CNN
 F 1 "GND" H 2055 7327 50  0000 C CNN
 F 2 "" H 2050 7500 50  0001 C CNN
@@
 P 5100 4750
 F 0 "J1" H 5050 5100 50  0000 L CNN
-F 1 "Conn_01x06" H 4750 4300 50  0000 L CNN
+F 1 "Molex" H 4950 4300 50  0000 L CNN
 F 2 "" H 5100 4750 50  0001 C CNN
 F 3 "" H 5100 4750 50  0001 C CNN
@@
 P 5050 8200
 F 0 "J2" H 5000 8550 50  0000 L CNN
-F 1 "Conn_01x06" H 4700 7750 50  0000 L CNN
+F 1 "Molex" H 4950 7750 50  0000 L CNN
 F 2 "" H 5050 8200 50  0001 C CNN
 F 3 "" H 5050 8200 50  0001 C CNN
@@
 $EndComp
 $Comp
-L power:+12V #PWR?
+L power:+12V #PWR0102
 U 1 1 5C2D3E63
 P 10650 900
-F 0 "#PWR?" H 10650 750 50  0001 C CNN
+F 0 "#PWR0102" H 10650 750 50  0001 C CNN
 F 1 "+12V" V 10665 1028 50  0000 L CNN
 F 2 "" H 10650 900 50  0001 C CNN
@@
 $EndComp
 $Comp
-L power:+12V #PWR?
+L power:+12V #PWR0103
 U 1 1 5C2D57ED
 P 4800 2050
-F 0 "#PWR?" H 4800 1900 50  0001 C CNN
+F 0 "#PWR0103" H 4800 1900 50  0001 C CNN
 F 1 "+12V" H 4815 2223 50  0000 C CNN
 F 2 "" H 4800 2050 50  0001 C CNN
@@
 $EndComp
 $Comp
-L power:+12V #PWR?
+L power:+12V #PWR0104
 U 1 1 5C2D59C4
 P 1400 2050
-F 0 "#PWR?" H 1400 1900 50  0001 C CNN
+F 0 "#PWR0104" H 1400 1900 50  0001 C CNN
 F 1 "+12V" H 1415 2223 50  0000 C CNN
 F 2 "" H 1400 2050 50  0001 C CNN
@@
 $EndComp
 $Comp
-L power:+12V #PWR?
+L power:+12V #PWR0105
 U 1 1 5C2D5B75
 P 3100 2050
-F 0 "#PWR?" H 3100 1900 50  0001 C CNN
+F 0 "#PWR0105" H 3100 1900 50  0001 C CNN
 F 1 "+12V" H 3115 2223 50  0000 C CNN
 F 2 "" H 3100 2050 50  0001 C CNN
@@
 $EndComp
 $Comp
-L power:+12V #PWR?
+L power:+12V #PWR0106
 U 1 1 5C2D5DEF
 P 6500 2050
-F 0 "#PWR?" H 6500 1900 50  0001 C CNN
+F 0 "#PWR0106" H 6500 1900 50  0001 C CNN
 F 1 "+12V" H 6515 2223 50  0000 C CNN
 F 2 "" H 6500 2050 50  0001 C CNN
@@
 $EndComp
 $Comp
-L power:GND #PWR?
+L power:GND #PWR0107
 U 1 1 5C2E83EA
 P 2100 5650
-F 0 "#PWR?" H 2100 5400 50  0001 C CNN
+F 0 "#PWR0107" H 2100 5400 50  0001 C CNN
 F 1 "GND" H 2105 5477 50  0000 C CNN
 F 2 "" H 2100 5650 50  0001 C CNN
@@
 $EndComp
 $Comp
-L power:GND #PWR?
+L power:GND #PWR0108
 U 1 1 5C2E9FED
 P 2100 5150
-F 0 "#PWR?" H 2100 4900 50  0001 C CNN
+F 0 "#PWR0108" H 2100 4900 50  0001 C CNN
 F 1 "GND" H 2105 4977 50  0000 C CNN
 F 2 "" H 2100 5150 50  0001 C CNN
@@
 $EndComp
 $Comp
-L power:GND #PWR?
+L power:GND #PWR0109
 U 1 1 5C2EBBCA
 P 2100 3600
-F 0 "#PWR?" H 2100 3350 50  0001 C CNN
+F 0 "#PWR0109" H 2100 3350 50  0001 C CNN
 F 1 "GND" H 2105 3427 50  0000 C CNN
 F 2 "" H 2100 3600 50  0001 C CNN
@@
 $EndComp
 $Comp
-L power:GND #PWR?
+L power:GND #PWR0110
 U 1 1 5C2ED68A
 P 2100 4100
-F 0 "#PWR?" H 2100 3850 50  0001 C CNN
+F 0 "#PWR0110" H 2100 3850 50  0001 C CNN
 F 1 "GND" H 2105 3927 50  0000 C CNN
 F 2 "" H 2100 4100 50  0001 C CNN
@@
 $EndComp
 $Comp
-L power:GND #PWR?
+L power:GND #PWR0111
 U 1 1 5C2EF397
 P 2050 7000
-F 0 "#PWR?" H 2050 6750 50  0001 C CNN
+F 0 "#PWR0111" H 2050 6750 50  0001 C CNN
 F 1 "GND" H 2055 6827 50  0000 C CNN
 F 2 "" H 2050 7000 50  0001 C CNN
@@
 $EndComp
 $Comp
-L power:GND #PWR?
+L power:GND #PWR0112
 U 1 1 5C2F0F3B
 P 2050 9150
-F 0 "#PWR?" H 2050 8900 50  0001 C CNN
+F 0 "#PWR0112" H 2050 8900 50  0001 C CNN
 F 1 "GND" H 2055 8977 50  0000 C CNN
 F 2 "" H 2050 9150 50  0001 C CNN
@@
 $EndComp
 $Comp
-L power:GND #PWR?
+L power:GND #PWR0113
 U 1 1 5C2F29FB
 P 2050 8650
-F 0 "#PWR?" H 2050 8400 50  0001 C CNN
+F 0 "#PWR0113" H 2050 8400 50  0001 C CNN
 F 1 "GND" H 2055 8477 50  0000 C CNN
 F 2 "" H 2050 8650 50  0001 C CNN
@@
 $EndComp
 $Comp
-L power:GND #PWR?
+L power:GND #PWR0114
 U 1 1 5C2FCCC9
 P 3550 1900
-F 0 "#PWR?" H 3550 1650 50  0001 C CNN
+F 0 "#PWR0114" H 3550 1650 50  0001 C CNN
 F 1 "GND" H 3555 1727 50  0000 C CNN
 F 2 "" H 3550 1900 50  0001 C CNN
@@
 $EndComp
 $Comp
-L power:GND #PWR?
+L power:GND #PWR0115
 U 1 1 5C2FE789
 P 5250 1900
-F 0 "#PWR?" H 5250 1650 50  0001 C CNN
+F 0 "#PWR0115" H 5250 1650 50  0001 C CNN
 F 1 "GND" H 5255 1727 50  0000 C CNN
 F 2 "" H 5250 1900 50  0001 C CNN
@@
 $EndComp
 $Comp
-L power:GND #PWR?
+L power:GND #PWR0116
 U 1 1 5C30031A
 P 6950 1900
-F 0 "#PWR?" H 6950 1650 50  0001 C CNN
+F 0 "#PWR0116" H 6950 1650 50  0001 C CNN
 F 1 "GND" H 6955 1727 50  0000 C CNN
 F 2 "" H 6950 1900 50  0001 C CNN
@@
 $EndComp
 $Comp
-L power:GND #PWR?
+L power:GND #PWR0117
 U 1 1 5C301ED1
 P 1850 1900
-F 0 "#PWR?" H 1850 1650 50  0001 C CNN
+F 0 "#PWR0117" H 1850 1650 50  0001 C CNN
 F 1 "GND" H 1855 1727 50  0000 C CNN
 F 2 "" H 1850 1900 50  0001 C CNN
@@
 $EndComp
 $Comp
-L power:+5V #PWR?
+L power:+5V #PWR0118
 U 1 1 5C30594E
 P 1850 1300
-F 0 "#PWR?" H 1850 1150 50  0001 C CNN
+F 0 "#PWR0118" H 1850 1150 50  0001 C CNN
 F 1 "+5V" H 1865 1473 50  0000 C CNN
 F 2 "" H 1850 1300 50  0001 C CNN
@@
 $EndComp
 $Comp
-L power:+5V #PWR?
+L power:+5V #PWR0119
 U 1 1 5C306127
 P 3550 1300
-F 0 "#PWR?" H 3550 1150 50  0001 C CNN
+F 0 "#PWR0119" H 3550 1150 50  0001 C CNN
 F 1 "+5V" H 3565 1473 50  0000 C CNN
 F 2 "" H 3550 1300 50  0001 C CNN
@@
 $EndComp
 $Comp
-L power:+5V #PWR?
+L power:+5V #PWR0120
 U 1 1 5C307BE7
 P 5250 1300
-F 0 "#PWR?" H 5250 1150 50  0001 C CNN
+F 0 "#PWR0120" H 5250 1150 50  0001 C CNN
 F 1 "+5V" H 5265 1473 50  0000 C CNN
 F 2 "" H 5250 1300 50  0001 C CNN
@@
 $EndComp
 $Comp
-L power:+5V #PWR?
+L power:+5V #PWR0121
 U 1 1 5C3096A7
 P 6950 1300
-F 0 "#PWR?" H 6950 1150 50  0001 C CNN
+F 0 "#PWR0121" H 6950 1150 50  0001 C CNN
 F 1 "+5V" H 6965 1473 50  0000 C CNN
 F 2 "" H 6950 1300 50  0001 C CNN
@@
 $EndComp
 $Comp
-L power:GND #PWR?
+L power:GND #PWR0122
 U 1 1 5C3103D6
 P 10650 1000
-F 0 "#PWR?" H 10650 750 50  0001 C CNN
+F 0 "#PWR0122" H 10650 750 50  0001 C CNN
 F 1 "GND" V 10655 872 50  0000 R CNN
 F 2 "" H 10650 1000 50  0001 C CNN
@@
 $EndComp
 $Comp
-L power:+12V #PWR?
+L power:+12V #PWR0123
 U 1 1 5C3126B1
 P 13850 1450
-F 0 "#PWR?" H 13850 1300 50  0001 C CNN
+F 0 "#PWR0123" H 13850 1300 50  0001 C CNN
 F 1 "+12V" H 13865 1623 50  0000 C CNN
 F 2 "" H 13850 1450 50  0001 C CNN
@@
 $EndComp
 $Comp
-L power:+5V #PWR?
+L power:+5V #PWR0124
 U 1 1 5C312ED2
 P 14150 1750
-F 0 "#PWR?" H 14150 1600 50  0001 C CNN
+F 0 "#PWR0124" H 14150 1600 50  0001 C CNN
 F 1 "+5V" H 14250 1800 50  0000 C CNN
 F 2 "" H 14150 1750 50  0001 C CNN
@@
 $EndComp
 $Comp
-L power:GND #PWR?
+L power:GND #PWR0125
 U 1 1 5C3168F6
 P 14050 3750
-F 0 "#PWR?" H 14050 3500 50  0001 C CNN
+F 0 "#PWR0125" H 14050 3500 50  0001 C CNN
 F 1 "GND" H 14200 3650 50  0000 C CNN
 F 2 "" H 14050 3750 50  0001 C CNN
@@
 $EndComp
 $Comp
-L power:GND #PWR?
+L power:GND #PWR0126
 U 1 1 5C316D7F
 P 13950 3750
-F 0 "#PWR?" H 13950 3500 50  0001 C CNN
+F 0 "#PWR0126" H 13950 3500 50  0001 C CNN
 F 1 "GND" H 13800 3650 50  0000 C CNN
 F 2 "" H 13950 3750 50  0001 C CNN
@@
 I2C_SLC
 $Comp
-L power:GND #PWR?
+L power:GND #PWR0127
 U 1 1 5C325D70
 P 10700 2550
-F 0 "#PWR?" H 10700 2300 50  0001 C CNN
+F 0 "#PWR0127" H 10700 2300 50  0001 C CNN
 F 1 "GND" H 10800 2450 50  0000 C CNN
 F 2 "" H 10700 2550 50  0001 C CNN
@@
 $EndComp
 $Comp
-L power:GND #PWR?
+L power:GND #PWR0128
 U 1 1 5C325EAF
 P 10700 4450
-F 0 "#PWR?" H 10700 4200 50  0001 C CNN
+F 0 "#PWR0128" H 10700 4200 50  0001 C CNN
 F 1 "GND" H 10800 4350 50  0000 C CNN
 F 2 "" H 10700 4450 50  0001 C CNN
@@
 Text Notes 14800 4600 0    50   ~ 0
 Mounting Holes\n
+NoConn ~ 14450 2250
+NoConn ~ 14450 2150
+NoConn ~ 7350 4500
+$Comp
+L power:PWR_FLAG #FLG0101
+U 1 1 5C2A9A76
+P 9900 850
+F 0 "#FLG0101" H 9900 925 50  0001 C CNN
+F 1 "PWR_FLAG" H 9900 1024 50  0000 C CNN
+F 2 "" H 9900 850 50  0001 C CNN
+F 3 "~" H 9900 850 50  0001 C CNN
+	1    9900 850
+	1    0    0    -1
+$EndComp
+$Comp
+L power:+12V #PWR0129
+U 1 1 5C2A9ABE
+P 9900 850
+F 0 "#PWR0129" H 9900 700 50  0001 C CNN
+F 1 "+12V" V 9915 978 50  0000 L CNN
+F 2 "" H 9900 850 50  0001 C CNN
+F 3 "" H 9900 850 50  0001 C CNN
+	1    9900 850
+	-1   0    0    1
+$EndComp
+$Comp
+L power:PWR_FLAG #FLG0102
+U 1 1 5C2A9DB2
+P 14650 1600
+F 0 "#FLG0102" H 14650 1675 50  0001 C CNN
+F 1 "PWR_FLAG" H 14650 1774 50  0000 C CNN
+F 2 "" H 14650 1600 50  0001 C CNN
+F 3 "~" H 14650 1600 50  0001 C CNN
+	1    14650 1600
+	1    0    0    -1
+$EndComp
+$Comp
+L power:+5V #PWR0130
+U 1 1 5C2A9DFA
+P 14650 1600
+F 0 "#PWR0130" H 14650 1450 50  0001 C CNN
+F 1 "+5V" H 14750 1650 50  0000 C CNN
+F 2 "" H 14650 1600 50  0001 C CNN
+F 3 "" H 14650 1600 50  0001 C CNN
+	1    14650 1600
+	-1   0    0    1
+$EndComp
 $EndSCHEMATC
