File: ESC-Board/ESC-Board.sch (KiCad schematic (older format))
At the start: 27 parts, among them J1 Molex, J2 Molex, J3 XT_60, U1 ESC:Blue_ESC, U2 ESC:Blue_ESC, U3 ESC:Blue_ESC, U4 ESC:Blue_ESC

Commit message: Final Draft(with net list)
Parts:
- A1: footprint Module:Arduino_Nano -> Blue_ESC:Arduino_Nano
- D1, D2, D3, D4: footprint Sensor_Current:Allegro_PSOF-7_4.8x6.4mm_P1.60mm -> Blue_ESC:Allegro_PSOF-7_4.8x6.4mm_Pitch1.60mm
- F1, F2, F3, F4, F5: footprint (none) -> Fuse_Holders_and_Fuses:Fuse_SMD1206_HandSoldering
- I1, I2: footprint (none) -> Connectors:RJ45_8
- J1, J2: footprint (none) -> Blue_ESC:Molex_6pin
- J3: footprint (none) -> Blue_ESC:XT60
- MH1, MH2, MH3, MH4, MH5, MH6, MH7, MH8: footprint (none) -> Mounting_Holes:MountingHole_3mm
- U1, U2, U3, U4: footprint (none) -> Blue_ESC:Blue_ESC
Connections:
- no-connect marks 24 -> 23
Changed lines of the file:
@@
 F 0 "J3" H 10900 1000 50  0000 L CNN
 F 1 "XT_60" H 10900 700 50  0000 L CNN
-F 2 "" H 10850 900 50  0001 C CNN
+F 2 "Blue_ESC:XT60" H 10850 900 50  0001 C CNN
 F 3 "" H 10850 900 50  0001 C CNN
 	1    10850 900
@@
 F 0 "A1" H 14450 3600 50  0000 C CNN
 F 1 "Arduino_Nano_v3.x" H 14750 1900 50  0000 C CNN
-F 2 "Module:Arduino_Nano" H 14100 1800 50  0001 L CNN
+F 2 "Blue_ESC:Arduino_Nano" H 14100 1800 50  0001 L CNN
 F 3 "" H 13950 1750 50  0001 C CNN
 	1    13950 2750
@@
 F 0 "F5" H 13900 1650 50  0000 L CNN
 F 1 "500m" H 13900 1550 50  0000 L CNN
-F 2 "" V 13780 1600 50  0001 C CNN
+F 2 "Fuse_Holders_and_Fuses:Fuse_SMD1206_HandSoldering" V 13780 1600 50  0001 C CNN
 F 3 "" H 13850 1600 50  0001 C CNN
 	1    13850 1600
@@
 F 0 "I1" V 10702 2520 50  0000 R CNN
 F 1 "RJ45" V 10611 2520 50  0000 R CNN
-F 2 "" V 10600 2975 50  0001 C CNN
+F 2 "Connectors:RJ45_8" V 10600 2975 50  0001 C CNN
 F 3 "" V 10600 2975 50  0001 C CNN
 	1    10600 2950
@@
 F 0 "D1" H 2050 1850 50  0000 L CNN
 F 1 "ACS780xLRTR-100U" H 1950 1200 50  0000 L CNN
-F 2 "Sensor_Current:Allegro_PSOF-7_4.8x6.4mm_P1.60mm" H 1850 1600 50  0001 C CNN
+F 2 "Blue_ESC:Allegro_PSOF-7_4.8x6.4mm_Pitch1.60mm" H 1850 1600 50  0001 C CNN
 F 3 "" H 1850 1600 50  0001 C CNN
 	1    1850 1600
@@
 F 0 "I2" V 10702 4420 50  0000 R CNN
 F 1 "RJ45" V 10611 4420 50  0000 R CNN
-F 2 "" V 10600 4875 50  0001 C CNN
+F 2 "Connectors:RJ45_8" V 10600 4875 50  0001 C CNN
 F 3 "" V 10600 4875 50  0001 C CNN
 	1    10600 4850
@@
 F 0 "D2" H 3750 1850 50  0000 L CNN
 F 1 "ACS780xLRTR-100U" H 3650 1200 50  0000 L CNN
-F 2 "Sensor_Current:Allegro_PSOF-7_4.8x6.4mm_P1.60mm" H 3550 1600 50  0001 C CNN
+F 2 "Blue_ESC:Allegro_PSOF-7_4.8x6.4mm_Pitch1.60mm" H 3550 1600 50  0001 C CNN
 F 3 "" H 3550 1600 50  0001 C CNN
 	1    3550 1600
@@
 F 0 "D3" H 5450 1950 50  0000 L CNN
 F 1 "ACS780xLRTR-100U" H 5350 1200 50  0000 L CNN
-F 2 "Sensor_Current:Allegro_PSOF-7_4.8x6.4mm_P1.60mm" H 5250 1600 50  0001 C CNN
+F 2 "Blue_ESC:Allegro_PSOF-7_4.8x6.4mm_Pitch1.60mm" H 5250 1600 50  0001 C CNN
 F 3 "" H 5250 1600 50  0001 C CNN
 	1    5250 1600
@@
 F 0 "D4" H 7150 1900 50  0000 L CNN
 F 1 "ACS780xLRTR-100U" H 7150 1200 50  0000 L CNN
-F 2 "Sensor_Current:Allegro_PSOF-7_4.8x6.4mm_P1.60mm" H 6950 1600 50  0001 C CNN
+F 2 "Blue_ESC:Allegro_PSOF-7_4.8x6.4mm_Pitch1.60mm" H 6950 1600 50  0001 C CNN
 F 3 "" H 6950 1600 50  0001 C CNN
 	1    6950 1600
@@
 F 0 "F1" H 1460 1946 50  0000 L CNN
 F 1 "10/15" H 1460 1855 50  0000 L CNN
-F 2 "" V 1330 1900 50  0001 C CNN
+F 2 "Fuse_Holders_and_Fuses:Fuse_SMD1206_HandSoldering" V 1330 1900 50  0001 C CNN
 F 3 "" H 1400 1900 50  0001 C CNN
 	1    1400 1900
@@
 F 0 "F2" H 3160 1946 50  0000 L CNN
 F 1 "10/15" H 3160 1855 50  0000 L CNN
-F 2 "" V 3030 1900 50  0001 C CNN
+F 2 "Fuse_Holders_and_Fuses:Fuse_SMD1206_HandSoldering" V 3030 1900 50  0001 C CNN
 F 3 "" H 3100 1900 50  0001 C CNN
 	1    3100 1900
@@
 F 0 "F3" H 4860 1946 50  0000 L CNN
 F 1 "10/15" H 4860 1855 50  0000 L CNN
-F 2 "" V 4730 1900 50  0001 C CNN
+F 2 "Fuse_Holders_and_Fuses:Fuse_SMD1206_HandSoldering" V 4730 1900 50  0001 C CNN
 F 3 "" H 4800 1900 50  0001 C CNN
 	1    4800 1900
@@
 F 0 "F4" H 6560 1946 50  0000 L CNN
 F 1 "10/15" H 6560 1855 50  0000 L CNN
-F 2 "" V 6430 1900 50  0001 C CNN
+F 2 "Fuse_Holders_and_Fuses:Fuse_SMD1206_HandSoldering" V 6430 1900 50  0001 C CNN
 F 3 "" H 6500 1900 50  0001 C CNN
 	1    6500 1900
@@
 F 0 "J1" H 5050 5100 50  0000 L CNN
 F 1 "Molex" H 4950 4300 50  0000 L CNN
-F 2 "" H 5100 4750 50  0001 C CNN
+F 2 "Blue_ESC:Molex_6pin" H 5100 4750 50  0001 C CNN
 F 3 "" H 5100 4750 50  0001 C CNN
 	1    5100 4750
@@
 F 0 "J2" H 5000 8550 50  0000 L CNN
 F 1 "Molex" H 4950 7750 50  0000 L CNN
-F 2 "" H 5050 8200 50  0001 C CNN
+F 2 "Blue_ESC:Molex_6pin" H 5050 8200 50  0001 C CNN
 F 3 "" H 5050 8200 50  0001 C CNN
 	1    5050 8200
@@
 F 0 "U4" V 2450 4000 50  0000 C CNN
 F 1 "ESC:Blue_ESC" V 3724 3950 50  0000 C CNN
-F 2 "" H 3100 4000 50  0001 C CNN
+F 2 "Blue_ESC:Blue_ESC" H 3100 4000 50  0001 C CNN
 F 3 "" H 3100 4000 50  0001 C CNN
 	1    3100 4000
@@
 F 0 "U3" V 2450 5550 50  0000 C CNN
 F 1 "ESC:Blue_ESC" V 3724 5500 50  0000 C CNN
-F 2 "" H 3100 5550 50  0001 C CNN
+F 2 "Blue_ESC:Blue_ESC" H 3100 5550 50  0001 C CNN
 F 3 "" H 3100 5550 50  0001 C CNN
 	1    3100 5550
@@
 F 0 "U2" V 2450 7400 50  0000 C CNN
 F 1 "ESC:Blue_ESC" V 3674 7350 50  0000 C CNN
-F 2 "" H 3050 7400 50  0001 C CNN
+F 2 "Blue_ESC:Blue_ESC" H 3050 7400 50  0001 C CNN
 F 3 "" H 3050 7400 50  0001 C CNN
 	1    3050 7400
@@
 F 0 "U1" V 2450 9050 50  0000 C CNN
 F 1 "ESC:Blue_ESC" V 3674 9000 50  0000 C CNN
-F 2 "" H 3050 9050 50  0001 C CNN
+F 2 "Blue_ESC:Blue_ESC" H 3050 9050 50  0001 C CNN
 F 3 "" H 3050 9050 50  0001 C CNN
 	1    3050 9050
@@
 F 0 "MH1" H 14600 4896 50  0000 L CNN
 F 1 "MountingHole" H 14600 4805 50  0000 L CNN
-F 2 "" H 14500 4850 50  0001 C CNN
+F 2 "Mounting_Holes:MountingHole_3mm" H 14500 4850 50  0001 C CNN
 F 3 "~" H 14500 4850 50  0001 C CNN
 	1    14500 4850
@@
 F 0 "MH2" H 14600 5096 50  0000 L CNN
 F 1 "MountingHole" H 14600 5005 50  0000 L CNN
-F 2 "" H 14500 5050 50  0001 C CNN
+F 2 "Mounting_Holes:MountingHole_3mm" H 14500 5050 50  0001 C CNN
 F 3 "~" H 14500 5050 50  0001 C CNN
 	1    14500 5050
@@
 F 0 "MH4" H 14600 5496 50  0000 L CNN
 F 1 "MountingHole" H 14600 5405 50  0000 L CNN
-F 2 "" H 14500 5450 50  0001 C CNN
+F 2 "Mounting_Holes:MountingHole_3mm" H 14500 5450 50  0001 C CNN
 F 3 "~" H 14500 5450 50  0001 C CNN
 	1    14500 5450
@@
 F 0 "MH3" H 14600 5296 50  0000 L CNN
 F 1 "MountingHole" H 14600 5205 50  0000 L CNN
-F 2 "" H 14500 5250 50  0001 C CNN
+F 2 "Mounting_Holes:MountingHole_3mm" H 14500 5250 50  0001 C CNN
 F 3 "~" H 14500 5250 50  0001 C CNN
 	1    14500 5250
@@
 F 0 "MH5" H 15350 4896 50  0000 L CNN
 F 1 "MountingHole" H 15350 4805 50  0000 L CNN
-F 2 "" H 15250 4850 50  0001 C CNN
+F 2 "Mounting_Holes:MountingHole_3mm" H 15250 4850 50  0001 C CNN
 F 3 "~" H 15250 4850 50  0001 C CNN
 	1    15250 4850
@@
 F 0 "MH6" H 15350 5096 50  0000 L CNN
 F 1 "MountingHole" H 15350 5005 50  0000 L CNN
-F 2 "" H 15250 5050 50  0001 C CNN
+F 2 "Mounting_Holes:MountingHole_3mm" H 15250 5050 50  0001 C CNN
 F 3 "~" H 15250 5050 50  0001 C CNN
 	1    15250 5050
@@
 F 0 "MH7" H 15350 5296 50  0000 L CNN
 F 1 "MountingHole" H 15350 5205 50  0000 L CNN
-F 2 "" H 15250 5250 50  0001 C CNN
+F 2 "Mounting_Holes:MountingHole_3mm" H 15250 5250 50  0001 C CNN
 F 3 "~" H 15250 5250 50  0001 C CNN
 	1    15250 5250
@@
 F 0 "MH8" H 15350 5496 50  0000 L CNN
 F 1 "MountingHole" H 15350 5405 50  0000 L CNN
-F 2 "" H 15250 5450 50  0001 C CNN
+F 2 "Mounting_Holes:MountingHole_3mm" H 15250 5450 50  0001 C CNN
 F 3 "~" H 15250 5450 50  0001 C CNN
 	1    15250 5450
@@
 NoConn ~ 14450 2250
 NoConn ~ 14450 2150
-NoConn ~ 7350 4500
 $Comp
 L power:PWR_FLAG #FLG0101
@@
 $EndComp
 $Comp
-L power:PWR_FLAG #FLG?
+L power:PWR_FLAG #FLG0103
 U 1 1 5C2AC515
 P 9900 1250
-F 0 "#FLG?" H 9900 1325 50  0001 C CNN
+F 0 "#FLG0103" H 9900 1325 50  0001 C CNN
 F 1 "PWR_FLAG" H 9900 1424 50  0000 C CNN
 F 2 "" H 9900 1250 50  0001 C CNN
@@
 $EndComp
 $Comp
-L power:GND #PWR?
+L power:GND #PWR0131
 U 1 1 5C2AC55D
 P 9900 1250
-F 0 "#PWR?" H 9900 1000 50  0001 C CNN
+F 0 "#PWR0131" H 9900 1000 50  0001 C CNN
 F 1 "GND" H 9850 1150 50  0000 R CNN
 F 2 "" H 9900 1250 50  0001 C CNN

Commit message: e
Parts:
- MH1, MH2, MH3, MH4, MH5, MH6, MH7, MH8: footprint Mounting_Holes:MountingHole_3mm -> Mounting_Holes:MountingHole_3.2mm_M3
Changed lines of the file:
@@
 F 0 "MH1" H 14600 4896 50  0000 L CNN
 F 1 "MountingHole" H 14600 4805 50  0000 L CNN
-F 2 "Mounting_Holes:MountingHole_3mm" H 14500 4850 50  0001 C CNN
+F 2 "Mounting_Holes:MountingHole_3.2mm_M3" H 14500 4850 50  0001 C CNN
 F 3 "~" H 14500 4850 50  0001 C CNN
 	1    14500 4850
@@
 F 0 "MH2" H 14600 5096 50  0000 L CNN
 F 1 "MountingHole" H 14600 5005 50  0000 L CNN
-F 2 "Mounting_Holes:MountingHole_3mm" H 14500 5050 50  0001 C CNN
+F 2 "Mounting_Holes:MountingHole_3.2mm_M3" H 14500 5050 50  0001 C CNN
 F 3 "~" H 14500 5050 50  0001 C CNN
 	1    14500 5050
@@
 F 0 "MH4" H 14600 5496 50  0000 L CNN
 F 1 "MountingHole" H 14600 5405 50  0000 L CNN
-F 2 "Mounting_Holes:MountingHole_3mm" H 14500 5450 50  0001 C CNN
+F 2 "Mounting_Holes:MountingHole_3.2mm_M3" H 14500 5450 50  0001 C CNN
 F 3 "~" H 14500 5450 50  0001 C CNN
 	1    14500 5450
@@
 F 0 "MH3" H 14600 5296 50  0000 L CNN
 F 1 "MountingHole" H 14600 5205 50  0000 L CNN
-F 2 "Mounting_Holes:MountingHole_3mm" H 14500 5250 50  0001 C CNN
+F 2 "Mounting_Holes:MountingHole_3.2mm_M3" H 14500 5250 50  0001 C CNN
 F 3 "~" H 14500 5250 50  0001 C CNN
 	1    14500 5250
@@
 F 0 "MH5" H 15350 4896 50  0000 L CNN
 F 1 "MountingHole" H 15350 4805 50  0000 L CNN
-F 2 "Mounting_Holes:MountingHole_3mm" H 15250 4850 50  0001 C CNN
+F 2 "Mounting_Holes:MountingHole_3.2mm_M3" H 15250 4850 50  0001 C CNN
 F 3 "~" H 15250 4850 50  0001 C CNN
 	1    15250 4850
@@
 F 0 "MH6" H 15350 5096 50  0000 L CNN
 F 1 "MountingHole" H 15350 5005 50  0000 L CNN
-F 2 "Mounting_Holes:MountingHole_3mm" H 15250 5050 50  0001 C CNN
+F 2 "Mounting_Holes:MountingHole_3.2mm_M3" H 15250 5050 50  0001 C CNN
 F 3 "~" H 15250 5050 50  0001 C CNN
 	1    15250 5050
@@
 F 0 "MH7" H 15350 5296 50  0000 L CNN
 F 1 "MountingHole" H 15350 5205 50  0000 L CNN
-F 2 "Mounting_Holes:MountingHole_3mm" H 15250 5250 50  0001 C CNN
+F 2 "Mounting_Holes:MountingHole_3.2mm_M3" H 15250 5250 50  0001 C CNN
 F 3 "~" H 15250 5250 50  0001 C CNN
 	1    15250 5250
@@
 F 0 "MH8" H 15350 5496 50  0000 L CNN
 F 1 "MountingHole" H 15350 5405 50  0000 L CNN
-F 2 "Mounting_Holes:MountingHole_3mm" H 15250 5450 50  0001 C CNN
+F 2 "Mounting_Holes:MountingHole_3.2mm_M3" H 15250 5450 50  0001 C CNN
 F 3 "~" H 15250 5450 50  0001 C CNN
 	1    15250 5450

Commit message: Board Finalized
E
Parts:
- removed MH5, MH6, MH7, MH8: MountingHole, Mounting_Holes:MountingHole_3.2mm_M3, symbol Mechanical:MountingHole
- added R1, R2: R, Resistors_SMD:R_0805, symbol Device:R
Connections:
- net labels added: +3.3V
- wire segments 60 -> 64
Changed lines of the file:
@@
 	1    0    0    -1
 $EndComp
+Text GLabel 13450 3050 0    50   Input ~ 0
+PWM_ESC_2
 Text GLabel 13450 2750 0    50   Input ~ 0
-PWM_ESC_2
-Text GLabel 13450 3050 0    50   Input ~ 0
 PWM_ESC_3
-Text GLabel 13450 3150 0    50   Input ~ 0
+Text GLabel 13450 2450 0    50   Input ~ 0
 PWM_ESC_4
 Wire Wire Line
@@
 U 1 1 5C1BC00C
 P 13850 1600
-F 0 "F5" H 13900 1650 50  0000 L CNN
-F 1 "500m" H 13900 1550 50  0000 L CNN
+F 0 "F5" H 13650 1650 50  0000 L CNN
+F 1 "500m" H 13600 1550 50  0000 L CNN
 F 2 "Fuse_Holders_and_Fuses:Fuse_SMD1206_HandSoldering" V 13780 1600 50  0001 C CNN
 F 3 "" H 13850 1600 50  0001 C CNN
@@
 	1    0    0    -1
 $EndComp
-Text GLabel 13450 2550 0    50   Input ~ 0
+Text GLabel 12500 2550 0    50   Input ~ 0
 I2C_SDA
-Text GLabel 13450 2650 0    50   Input ~ 0
+Text GLabel 12500 2650 0    50   Input ~ 0
 I2C_SLC
 Text GLabel 2050 8950 0    50   Input ~ 0
@@
 	0    -1   -1   0
 $EndComp
-Text GLabel 13450 2450 0    50   Input ~ 0
+Text GLabel 13450 3150 0    50   Input ~ 0
 PWM_ESC_1
 Text GLabel 10900 2450 1    50   Input ~ 0
@@
 	1    0    0    -1
 $EndComp
-$Comp
-L Mechanical:MountingHole MH5
-U 1 1 5C29E1ED
-P 15250 4850
-F 0 "MH5" H 15350 4896 50  0000 L CNN
-F 1 "MountingHole" H 15350 4805 50  0000 L CNN
-F 2 "Mounting_Holes:MountingHole_3.2mm_M3" H 15250 4850 50  0001 C CNN
-F 3 "~" H 15250 4850 50  0001 C CNN
-	1    15250 4850
-	1    0    0    -1
-$EndComp
-$Comp
-L Mechanical:MountingHole MH6
-U 1 1 5C29E245
-P 15250 5050
-F 0 "MH6" H 15350 5096 50  0000 L CNN
-F 1 "MountingHole" H 15350 5005 50  0000 L CNN
-F 2 "Mounting_Holes:MountingHole_3.2mm_M3" H 15250 5050 50  0001 C CNN
-F 3 "~" H 15250 5050 50  0001 C CNN
-	1    15250 5050
-	1    0    0    -1
-$EndComp
-$Comp
-L Mechanical:MountingHole MH7
-U 1 1 5C29E29F
-P 15250 5250
-F 0 "MH7" H 15350 5296 50  0000 L CNN
-F 1 "MountingHole" H 15350 5205 50  0000 L CNN
-F 2 "Mounting_Holes:MountingHole_3.2mm_M3" H 15250 5250 50  0001 C CNN
-F 3 "~" H 15250 5250 50  0001 C CNN
-	1    15250 5250
-	1    0    0    -1
-$EndComp
-$Comp
-L Mechanical:MountingHole MH8
-U 1 1 5C29E2FB
-P 15250 5450
-F 0 "MH8" H 15350 5496 50  0000 L CNN
-F 1 "MountingHole" H 15350 5405 50  0000 L CNN
-F 2 "Mounting_Holes:MountingHole_3.2mm_M3" H 15250 5450 50  0001 C CNN
-F 3 "~" H 15250 5450 50  0001 C CNN
-	1    15250 5450
-	1    0    0    -1
-$EndComp
 Wire Notes Line
 	14250 5600 15950 5600
@@
 	1    0    0    -1
 $EndComp
+$Comp
+L Device:R R1
+U 1 1 5C2F31D4
+P 12600 2400
+F 0 "R1" H 12670 2446 50  0000 L CNN
+F 1 "R" H 12670 2355 50  0000 L CNN
+F 2 "Resistors_SMD:R_0805" V 12530 2400 50  0001 C CNN
+F 3 "~" H 12600 2400 50  0001 C CNN
+	1    12600 2400
+	1    0    0    -1
+$EndComp
+$Comp
+L Device:R R2
+U 1 1 5C2F324A
+P 12600 2800
+F 0 "R2" H 12670 2846 50  0000 L CNN
+F 1 "R" H 12670 2755 50  0000 L CNN
+F 2 "Resistors_SMD:R_0805" V 12530 2800 50  0001 C CNN
+F 3 "~" H 12600 2800 50  0001 C CNN
+	1    12600 2800
+	1    0    0    -1
+$EndComp
+Wire Wire Line
+	13450 2550 12600 2550
+Connection ~ 12600 2550
+Wire Wire Line
+	12600 2550 12500 2550
+Wire Wire Line
+	13450 2650 12600 2650
+Connection ~ 12600 2650
+Wire Wire Line
+	12600 2650 12500 2650
+$Comp
+L power:+3.3V #PWR0132
+U 1 1 5C2F7A02
+P 14050 1750
+F 0 "#PWR0132" H 14050 1600 50  0001 C CNN
+F 1 "+3.3V" H 14000 1950 50  0000 C CNN
+F 2 "" H 14050 1750 50  0001 C CNN
+F 3 "" H 14050 1750 50  0001 C CNN
+	1    14050 1750
+	1    0    0    -1
+$EndComp
+$Comp
+L power:+3.3V #PWR0133
+U 1 1 5C2F7B83
+P 12600 2250
+F 0 "#PWR0133" H 12600 2100 50  0001 C CNN
+F 1 "+3.3V" H 12550 2450 50  0000 C CNN
+F 2 "" H 12600 2250 50  0001 C CNN
+F 3 "" H 12600 2250 50  0001 C CNN
+	1    12600 2250
+	1    0    0    -1
+$EndComp
+$Comp
+L power:+3.3V #PWR0134
+U 1 1 5C2F7BC8
+P 12600 2950
+F 0 "#PWR0134" H 12600 2800 50  0001 C CNN
+F 1 "+3.3V" H 12550 3150 50  0000 C CNN
+F 2 "" H 12600 2950 50  0001 C CNN
+F 3 "" H 12600 2950 50  0001 C CNN
+	1    12600 2950
+	-1   0    0    1
+$EndComp
+$Comp
+L power:+3.3V #PWR0135
+U 1 1 5C2F7C47
+P 15250 1600
+F 0 "#PWR0135" H 15250 1450 50  0001 C CNN
+F 1 "+3.3V" H 15400 1650 50  0000 C CNN
+F 2 "" H 15250 1600 50  0001 C CNN
+F 3 "" H 15250 1600 50  0001 C CNN
+	1    15250 1600
+	-1   0    0    1
+$EndComp
+$Comp
+L power:PWR_FLAG #FLG0104
+U 1 1 5C2F7CC6
+P 15250 1600
+F 0 "#FLG0104" H 15250 1675 50  0001 C CNN
+F 1 "PWR_FLAG" H 15250 1774 50  0000 C CNN
+F 2 "" H 15250 1600 50  0001 C CNN
+F 3 "~" H 15250 1600 50  0001 C CNN
+	1    15250 1600
+	1    0    0    -1
+$EndComp

Commit message: Fixed names
Parts:
- renumbered D1 to U1, D2 to U2, D3 to U3, D4 to U4, U4 to U5, U3 to U6, U2 to U7, U1 to U8
Changed lines of the file:
@@
 $EndComp
 $Comp
-L Sensor_Current:ACS780xLRTR-100U D1
+L Sensor_Current:ACS780xLRTR-100U U1
 U 1 1 5C198CA7
 P 1850 1600
-F 0 "D1" H 2050 1850 50  0000 L CNN
+F 0 "U1" H 2050 1850 50  0000 L CNN
 F 1 "ACS780xLRTR-100U" H 1950 1200 50  0000 L CNN
 F 2 "Blue_ESC:Allegro_PSOF-7_4.8x6.4mm_Pitch1.60mm" H 1850 1600 50  0001 C CNN
@@
 I2C RJ45 Connector\n
 $Comp
-L Sensor_Current:ACS780xLRTR-100U D2
+L Sensor_Current:ACS780xLRTR-100U U2
 U 1 1 5C2A52B8
 P 3550 1600
-F 0 "D2" H 3750 1850 50  0000 L CNN
+F 0 "U2" H 3750 1850 50  0000 L CNN
 F 1 "ACS780xLRTR-100U" H 3650 1200 50  0000 L CNN
 F 2 "Blue_ESC:Allegro_PSOF-7_4.8x6.4mm_Pitch1.60mm" H 3550 1600 50  0001 C CNN
@@
 $EndComp
 $Comp
-L Sensor_Current:ACS780xLRTR-100U D3
+L Sensor_Current:ACS780xLRTR-100U U3
 U 1 1 5C2A6F93
 P 5250 1600
-F 0 "D3" H 5450 1950 50  0000 L CNN
+F 0 "U3" H 5450 1950 50  0000 L CNN
 F 1 "ACS780xLRTR-100U" H 5350 1200 50  0000 L CNN
 F 2 "Blue_ESC:Allegro_PSOF-7_4.8x6.4mm_Pitch1.60mm" H 5250 1600 50  0001 C CNN
@@
 $EndComp
 $Comp
-L Sensor_Current:ACS780xLRTR-100U D4
+L Sensor_Current:ACS780xLRTR-100U U4
 U 1 1 5C2B4ED1
 P 6950 1600
-F 0 "D4" H 7150 1900 50  0000 L CNN
+F 0 "U4" H 7150 1900 50  0000 L CNN
 F 1 "ACS780xLRTR-100U" H 7150 1200 50  0000 L CNN
 F 2 "Blue_ESC:Allegro_PSOF-7_4.8x6.4mm_Pitch1.60mm" H 6950 1600 50  0001 C CNN
@@
 Power_ESC_4
 $Comp
-L ESC:Blue_ESC U4
+L ESC:Blue_ESC U5
 U 1 1 5C31FC02
 P 3100 4000
-F 0 "U4" V 2450 4000 50  0000 C CNN
+F 0 "U5" V 2450 4000 50  0000 C CNN
 F 1 "ESC:Blue_ESC" V 3724 3950 50  0000 C CNN
 F 2 "Blue_ESC:Blue_ESC" H 3100 4000 50  0001 C CNN
@@
 $EndComp
 $Comp
-L ESC:Blue_ESC U3
+L ESC:Blue_ESC U6
 U 1 1 5C324647
 P 3100 5550
-F 0 "U3" V 2450 5550 50  0000 C CNN
+F 0 "U6" V 2450 5550 50  0000 C CNN
 F 1 "ESC:Blue_ESC" V 3724 5500 50  0000 C CNN
 F 2 "Blue_ESC:Blue_ESC" H 3100 5550 50  0001 C CNN
@@
 $EndComp
 $Comp
-L ESC:Blue_ESC U2
+L ESC:Blue_ESC U7
 U 1 1 5C32481F
 P 3050 7400
-F 0 "U2" V 2450 7400 50  0000 C CNN
+F 0 "U7" V 2450 7400 50  0000 C CNN
 F 1 "ESC:Blue_ESC" V 3674 7350 50  0000 C CNN
 F 2 "Blue_ESC:Blue_ESC" H 3050 7400 50  0001 C CNN
@@
 $EndComp
 $Comp
-L ESC:Blue_ESC U1
+L ESC:Blue_ESC U8
 U 1 1 5C324A6D
 P 3050 9050
-F 0 "U1" V 2450 9050 50  0000 C CNN
+F 0 "U8" V 2450 9050 50  0000 C CNN
 F 1 "ESC:Blue_ESC" V 3674 9000 50  0000 C CNN
 F 2 "Blue_ESC:Blue_ESC" H 3050 9050 50  0001 C CNN
