File: ESC-Board/ESC-Board.kicad_pcb (KiCad board)
At the start: 2 copper layers, 17.1 x 32 mm, 4 parts

Commit message: Final Draft(with net list)
Parts:
- removed REF** (x4): Blue_ESC, Blue_ESC:Blue_ESC
- added A1: Arduino_Nano_v3.x, Blue_ESC:Arduino_Nano, F.Cu at (176.5, 43.4)
- added D1: ACS780xLRTR-100U, Blue_ESC:Allegro_PSOF-7_4.8x6.4mm_Pitch1.60mm, F.Cu at (170.9, 42.4)
- added D2: ACS780xLRTR-100U, Blue_ESC:Allegro_PSOF-7_4.8x6.4mm_Pitch1.60mm, F.Cu at (85.8, 85.6)
- added D3: ACS780xLRTR-100U, Blue_ESC:Allegro_PSOF-7_4.8x6.4mm_Pitch1.60mm, F.Cu at (92.9, 85.6)
- added D4: ACS780xLRTR-100U, Blue_ESC:Allegro_PSOF-7_4.8x6.4mm_Pitch1.60mm, F.Cu at (127.0, 77.5)
- added F1: 10/15, Fuse_Holders_and_Fuses:Fuse_SMD1206_HandSoldering, F.Cu at (140.8, 77.6)
- added F2: 10/15, Fuse_Holders_and_Fuses:Fuse_SMD1206_HandSoldering, F.Cu at (126.9, 82.6)
- added F3: 10/15, Fuse_Holders_and_Fuses:Fuse_SMD1206_HandSoldering, F.Cu at (133.9, 75.5)
- added F4: 10/15, Fuse_Holders_and_Fuses:Fuse_SMD1206_HandSoldering, F.Cu at (92.5, 90.7)
- added F5: 500m, Fuse_Holders_and_Fuses:Fuse_SMD1206_HandSoldering, F.Cu at (85.7, 90.7)
- added I1: RJ45, Connectors:RJ45_8, F.Cu at (154.9, 42.9)
- added I2: RJ45, Connectors:RJ45_8, F.Cu at (154.7, 63.2)
- added J1: Molex, Blue_ESC:Molex_6pin, F.Cu at (104.9, 82.1)
- added J2: Molex, Blue_ESC:Molex_6pin, F.Cu at (117.3, 82.1)
- added J3: XT_60, Blue_ESC:XT60, F.Cu at (86.7, 78.0)
- added MH1: MountingHole, Mounting_Holes:MountingHole_3mm, F.Cu at (133.6, 84.3)
- added MH2: MountingHole, Mounting_Holes:MountingHole_3mm, F.Cu at (126.8, 87.5)
- added MH3: MountingHole, Mounting_Holes:MountingHole_3mm, F.Cu at (170.6, 49.2)
- added MH4: MountingHole, Mounting_Holes:MountingHole_3mm, F.Cu at (170.6, 55.7)
- added MH5: MountingHole, Mounting_Holes:MountingHole_3mm, F.Cu at (140.1, 82.5)
- added MH6: MountingHole, Mounting_Holes:MountingHole_3mm, F.Cu at (147.5, 77.2)
- added MH7: MountingHole, Mounting_Holes:MountingHole_3mm, F.Cu at (170.6, 62.3)
- added MH8: MountingHole, Mounting_Holes:MountingHole_3mm, F.Cu at (146.7, 83.8)
- added U1: ESC:Blue_ESC, Blue_ESC:Blue_ESC, F.Cu at (142.7, 56.4)
- added U2: ESC:Blue_ESC, Blue_ESC:Blue_ESC, F.Cu at (125.4, 56.4)
- added U3: ESC:Blue_ESC, Blue_ESC:Blue_ESC, F.Cu at (108.2, 56.4)
- added U4: ESC:Blue_ESC, Blue_ESC:Blue_ESC, F.Cu at (90.9, 56.4)

Commit message: Starting layout
Parts:
- U1, U2, U3, U4: moved to B.Cu
- moved D1 145.7 mm to (41.7, 109.8), turned to 180 degrees
- moved F5 134.5 mm to (214.9, 53.3)
- moved MH6 123.7 mm to (246.1, 151.9)
- moved MH4 117.6 mm to (238.8, 151.6)
- moved MH3 114.7 mm to (223.3, 151.1)
- moved MH5 114.2 mm to (230.9, 151.9)
- moved F1 109.3 mm to (41.0, 122.3)
- moved U1 103.3 mm to (42.2, 80.3)
- moved J3 98.9 mm to (183.9, 59.6), turned to 270 degrees
- moved MH8 97.1 mm to (215.6, 152.1)
- moved MH7 94.6 mm to (203.7, 150.9)
- moved MH2 93.9 mm to (194.6, 152.4)
- moved MH1 82.9 mm to (182.6, 151.1)
- moved I1 82.6 mm to (223.5, 89.0)
- moved F2 73.9 mm to (65.4, 123.5)
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Other:
- outline, holes or cut-outs redrawn

Commit message: e
Parts:
- removed MH1: MountingHole, Mounting_Holes:MountingHole_3mm
- moved I1 52.8 mm to (171.0, 83.1)
- moved I2 52.8 mm to (171.0, 55.4)
- moved A1 52.8 mm to (148.6, 55.4)
- moved J3 50.4 mm to (140.7, 85.5)
- moved F5 49.5 mm to (169.9, 74.0)
- moved F2 43.4 mm to (83.8, 84.2), turned to 270 degrees
- moved F4 41.9 mm to (132.3, 84.3), turned to 270 degrees
- moved F3 41.7 mm to (102.6, 84.2), turned to 270 degrees
- moved F1 40.3 mm to (54.1, 84.2), turned to 270 degrees
- moved D2 31.9 mm to (77.0, 79.7), turned to 270 degrees
- moved D1 30.6 mm to (47.2, 79.7), turned to 270 degrees
- moved D4 29.4 mm to (125.5, 79.8), turned to 270 degrees
- moved D3 29.1 mm to (95.8, 79.7), turned to 270 degrees
- moved U1 5.11 mm to (47.2, 79.7)

Commit message: Cur
Parts:
- moved D2 23.3 mm to (76.9, 103.0)
- moved D3 23.3 mm to (95.7, 103.0)
- moved D1 23.2 mm to (47.1, 102.9)
- moved D4 23.2 mm to (125.4, 103.0)
- moved F2 18.9 mm to (83.7, 103.1), turned to 90 degrees
- moved F3 18.9 mm to (102.5, 103.1), turned to 90 degrees
- moved F1 18.8 mm to (53.9, 103.0), turned to 90 degrees
- moved F4 18.8 mm to (132.2, 103.1), turned to 90 degrees
Changed lines of the file:
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@@
   )
   (module Blue_ESC:Allegro_PSOF-7_4.8x6.4mm_Pitch1.60mm (layer F.Cu)
-    (at 47.244 79.6925 270)
+    (at 47.1424 102.9208 270)
     (descr "Allegro Microsystems PSOF-7, 4.8x6.4mm Body, 1.60mm Pitch (http://www.allegromicro.com/~/media/Files/Datasheets/ACS780-Datasheet.ashx)")
     (tags "Allegro PSOF-7")
@@
     (fp_line (start -0.6 3.32) (end -2.47 3.32) (layer F.SilkS) (width 0.12))
     (fp_line (start 2.57 3.32) (end 0.7 3.32) (layer F.SilkS) (width 0.12))
-    (fp_text user %R (at 0 0 270) (layer F.Fab)
+    (fp_text user %R (at 0 0) (layer F.Fab)
       (effects (font (size 1 1) (thickness 0.15)))
     )
@@
   )
   (module Blue_ESC:Allegro_PSOF-7_4.8x6.4mm_Pitch1.60mm (layer F.Cu)
-    (at 76.962 79.7052 270)
+    (at 76.8604 102.9716 270)
     (descr "Allegro Microsystems PSOF-7, 4.8x6.4mm Body, 1.60mm Pitch (http://www.allegromicro.com/~/media/Files/Datasheets/ACS780-Datasheet.ashx)")
     (tags "Allegro PSOF-7")
@@
   )
   (module Blue_ESC:Allegro_PSOF-7_4.8x6.4mm_Pitch1.60mm (layer F.Cu)
-    (at 95.758 79.7052 270)
+    (at 95.6564 102.9716 270)
     (descr "Allegro Microsystems PSOF-7, 4.8x6.4mm Body, 1.60mm Pitch (http://www.allegromicro.com/~/media/Files/Datasheets/ACS780-Datasheet.ashx)")
     (tags "Allegro PSOF-7")
@@
   )
   (module Blue_ESC:Allegro_PSOF-7_4.8x6.4mm_Pitch1.60mm (layer F.Cu)
-    (at 125.476 79.756 270)
+    (at 125.3744 102.9716 270)
     (descr "Allegro Microsystems PSOF-7, 4.8x6.4mm Body, 1.60mm Pitch (http://www.allegromicro.com/~/media/Files/Datasheets/ACS780-Datasheet.ashx)")
     (tags "Allegro PSOF-7")
@@
   )
   (module Fuse_Holders_and_Fuses:Fuse_SMD1206_HandSoldering (layer F.Cu)
-    (at 54.102 84.1756 270)
+    (at 53.9496 103.0224 90)
     (descr "Fuse, Sicherung, SMD1206, Littlefuse-Wickmann 433 Series, Hand Soldering,")
     (tags "Fuse Sicherung SMD1206 Littlefuse-Wickmann 433 Series Hand Soldering ")
     (attr smd)
-    (fp_text reference F1 (at -0.05 -2.2 270) (layer F.SilkS)
-      (effects (font (size 1 1) (thickness 0.15)))
-    )
-    (fp_text value 10/15 (at -0.15 2.5 270) (layer F.Fab)
+    (fp_text reference F1 (at -0.05 -2.2 90) (layer F.SilkS)
+      (effects (font (size 1 1) (thickness 0.15)))
+    )
+    (fp_text value 10/15 (at -0.15 2.5 90) (layer F.Fab)
       (effects (font (size 1 1) (thickness 0.15)))
     )
@@
     (fp_line (start 3.35 1.58) (end 3.35 -1.58) (layer F.CrtYd) (width 0.05))
     (fp_line (start 3.35 1.58) (end -3.35 1.58) (layer F.CrtYd) (width 0.05))
-    (pad 1 smd rect (at -2.09 0) (size 2.03 2.65) (layers F.Cu F.Paste F.Mask)
+    (pad 1 smd rect (at -2.09 0 180) (size 2.03 2.65) (layers F.Cu F.Paste F.Mask)
       (net 1 "Net-(D1-Pad6)"))
-    (pad 2 smd rect (at 2.09 0) (size 2.03 2.65) (layers F.Cu F.Paste F.Mask)
+    (pad 2 smd rect (at 2.09 0 180) (size 2.03 2.65) (layers F.Cu F.Paste F.Mask)
       (net 23 +12V))
   )
   (module Fuse_Holders_and_Fuses:Fuse_SMD1206_HandSoldering (layer F.Cu)
-    (at 83.7692 84.1756 270)
+    (at 83.6676 103.0732 90)
     (descr "Fuse, Sicherung, SMD1206, Littlefuse-Wickmann 433 Series, Hand Soldering,")
     (tags "Fuse Sicherung SMD1206 Littlefuse-Wickmann 433 Series Hand Soldering ")
     (attr smd)
-    (fp_text reference F2 (at -0.05 -2.2 270) (layer F.SilkS)
-      (effects (font (size 1 1) (thickness 0.15)))
-    )
-    (fp_text value 10/15 (at -0.15 2.5 270) (layer F.Fab)
+    (fp_text reference F2 (at -0.05 -2.2 90) (layer F.SilkS)
+      (effects (font (size 1 1) (thickness 0.15)))
+    )
+    (fp_text value 10/15 (at -0.15 2.5 90) (layer F.Fab)
       (effects (font (size 1 1) (thickness 0.15)))
     )
@@
     (fp_line (start 1.6 0.8) (end -1.6 0.8) (layer F.Fab) (width 0.1))
     (fp_line (start -1.6 0.8) (end -1.6 -0.8) (layer F.Fab) (width 0.1))
-    (pad 2 smd rect (at 2.09 0) (size 2.03 2.65) (layers F.Cu F.Paste F.Mask)
+    (pad 2 smd rect (at 2.09 0 180) (size 2.03 2.65) (layers F.Cu F.Paste F.Mask)
       (net 23 +12V))
-    (pad 1 smd rect (at -2.09 0) (size 2.03 2.65) (layers F.Cu F.Paste F.Mask)
+    (pad 1 smd rect (at -2.09 0 180) (size 2.03 2.65) (layers F.Cu F.Paste F.Mask)
       (net 12 "Net-(D2-Pad6)"))
   )
   (module Fuse_Holders_and_Fuses:Fuse_SMD1206_HandSoldering (layer F.Cu)
-    (at 102.5652 84.1756 270)
+    (at 102.4636 103.0732 90)
     (descr "Fuse, Sicherung, SMD1206, Littlefuse-Wickmann 433 Series, Hand Soldering,")
     (tags "Fuse Sicherung SMD1206 Littlefuse-Wickmann 433 Series Hand Soldering ")
     (attr smd)
-    (fp_text reference F3 (at -0.05 -2.2 270) (layer F.SilkS)
-      (effects (font (size 1 1) (thickness 0.15)))
-    )
-    (fp_text value 10/15 (at -0.15 2.5 270) (layer F.Fab)
+    (fp_text reference F3 (at -0.05 -2.2 90) (layer F.SilkS)
+      (effects (font (size 1 1) (thickness 0.15)))
+    )
+    (fp_text value 10/15 (at -0.15 2.5 90) (layer F.Fab)
       (effects (font (size 1 1) (thickness 0.15)))
     )
@@
     (fp_line (start 3.35 1.58) (end 3.35 -1.58) (layer F.CrtYd) (width 0.05))
     (fp_line (start 3.35 1.58) (end -3.35 1.58) (layer F.CrtYd) (width 0.05))
-    (pad 1 smd rect (at -2.09 0) (size 2.03 2.65) (layers F.Cu F.Paste F.Mask)
+    (pad 1 smd rect (at -2.09 0 180) (size 2.03 2.65) (layers F.Cu F.Paste F.Mask)
       (net 13 "Net-(D3-Pad6)"))
-    (pad 2 smd rect (at 2.09 0) (size 2.03 2.65) (layers F.Cu F.Paste F.Mask)
+    (pad 2 smd rect (at 2.09 0 180) (size 2.03 2.65) (layers F.Cu F.Paste F.Mask)
       (net 23 +12V))
   )
   (module Fuse_Holders_and_Fuses:Fuse_SMD1206_HandSoldering (layer F.Cu)
-    (at 132.2832 84.2772 270)
+    (at 132.1816 103.124 90)
     (descr "Fuse, Sicherung, SMD1206, Littlefuse-Wickmann 433 Series, Hand Soldering,")
     (tags "Fuse Sicherung SMD1206 Littlefuse-Wickmann 433 Series Hand Soldering ")
     (attr smd)
-    (fp_text reference F4 (at -0.05 -2.2 270) (layer F.SilkS)
-      (effects (font (size 1 1) (thickness 0.15)))
-    )
-    (fp_text value 10/15 (at -0.15 2.5 270) (layer F.Fab)
+    (fp_text reference F4 (at -0.05 -2.2 90) (layer F.SilkS)
+      (effects (font (size 1 1) (thickness 0.15)))
+    )
+    (fp_text value 10/15 (at -0.15 2.5 90) (layer F.Fab)
       (effects (font (size 1 1) (thickness 0.15)))
     )
@@
     (fp_line (start 1.6 0.8) (end -1.6 0.8) (layer F.Fab) (width 0.1))
     (fp_line (start -1.6 0.8) (end -1.6 -0.8) (layer F.Fab) (width 0.1))
-    (pad 2 smd rect (at 2.09 0) (size 2.03 2.65) (layers F.Cu F.Paste F.Mask)
+    (pad 2 smd rect (at 2.09 0 180) (size 2.03 2.65) (layers F.Cu F.Paste F.Mask)
       (net 23 +12V))
-    (pad 1 smd rect (at -2.09 0) (size 2.03 2.65) (layers F.Cu F.Paste F.Mask)
+    (pad 1 smd rect (at -2.09 0 180) (size 2.03 2.65) (layers F.Cu F.Paste F.Mask)
       (net 22 "Net-(D4-Pad6)"))
   )

Commit message: e
Parts:
- moved J3 7.37 mm to (140.7, 92.9), turned to 90 degrees
Changed lines of the file:
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@@
   )
   (module Blue_ESC:XT60 (layer F.Cu)
-    (at 140.6652 85.4964 270)
-    (fp_text reference J3 (at 3.556 6.096 270) (layer F.SilkS)
+    (at 140.6652 92.8624 90)
+    (fp_text reference J3 (at 3.556 6.096 90) (layer F.SilkS)
       (effects (font (size 1 1) (thickness 0.15)))
     )
-    (fp_text value XT_60 (at 3.2 -5.9 270) (layer F.Fab)
+    (fp_text value XT_60 (at 3.2 -5.9 90) (layer F.Fab)
       (effects (font (size 1 1) (thickness 0.15)))
     )
@@
     (fp_line (start 7.5 -4) (end 3.1 -4) (layer F.SilkS) (width 0.1))
     (fp_line (start 7.2 4) (end 3 4) (layer F.SilkS) (width 0.1))
-    (pad 1 thru_hole circle (at 0 0 270) (size 6 6) (drill 4.5) (layers *.Cu *.Mask F.SilkS)
+    (pad 1 thru_hole circle (at 0 0 90) (size 6 6) (drill 4.5) (layers *.Cu *.Mask F.SilkS)
       (net 23 +12V))
-    (pad 2 thru_hole circle (at 7.5 0 270) (size 6 6) (drill 4.5) (layers *.Cu *.Mask F.SilkS)
+    (pad 2 thru_hole circle (at 7.5 0 90) (size 6 6) (drill 4.5) (layers *.Cu *.Mask F.SilkS)
       (net 6 GND))
   )

Commit message: w
Parts:
- U1, U2, U3, U4: moved to F.Cu
- turned U1 to 180 degrees
- turned U2 to 180 degrees
- turned U3 to 180 degrees
- turned U4 to 180 degrees

Commit message: I hate myself
Parts:
- moved MH7 193.7 mm to (39.0, 49.0)
- moved MH3 190.0 mm to (39.0, 105.0)
- moved MH8 107.0 mm to (187.0, 49.0)
- moved MH2 48.0 mm to (187.0, 105.0)
- moved U4 9.77 mm to (125.0, 70.0)
- moved U3 9.73 mm to (95.0, 70.0)
- moved U2 9.71 mm to (77.0, 70.0)
- moved U1 9.70 mm to (47.0, 70.0)
- moved J1 9.37 mm to (110.0, 64.0)
- moved J2 9.30 mm to (62.0, 64.0)
- moved D4 9.28 mm to (123.0, 94.0)
- moved F4 9.20 mm to (131.0, 94.0)
- moved D3 9.12 mm to (94.0, 94.0)
- moved F3 9.09 mm to (102.0, 94.0)
- moved F2 9.08 mm to (84.0, 94.0)
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Other:
- board size 17.1 x 32 mm -> 154 x 62 mm
Changed lines of the file:
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@@
   (general
     (thickness 1.6)
-    (drawings 0)
+    (drawings 5)
     (tracks 0)
     (zones 0)
@@
     (add_net Power_ESC_4)
   )
+  (module Fuse_Holders_and_Fuses:Fuse_SMD1206_HandSoldering (layer F.Cu)
+    (at 84 94 90)
+    (descr "Fuse, Sicherung, SMD1206, Littlefuse-Wickmann 433 Series, Hand Soldering,")
+    (tags "Fuse Sicherung SMD1206 Littlefuse-Wickmann 433 Series Hand Soldering ")
+    (attr smd)
+    (fp_text reference F2 (at -0.05 -2.2 90) (layer F.SilkS)
+      (effects (font (size 1 1) (thickness 0.15)))
+    )
+    (fp_text value 10/15 (at -0.15 2.5 90) (layer F.Fab)
+      (effects (font (size 1 1) (thickness 0.15)))
+    )
+    (fp_line (start 3.35 1.58) (end -3.35 1.58) (layer F.CrtYd) (width 0.05))
+    (fp_line (start 3.35 1.58) (end 3.35 -1.58) (layer F.CrtYd) (width 0.05))
+    (fp_line (start -3.35 -1.58) (end -3.35 1.58) (layer F.CrtYd) (width 0.05))
+    (fp_line (start -3.35 -1.58) (end 3.35 -1.58) (layer F.CrtYd) (width 0.05))
+    (fp_line (start -1 -1.07) (end 1 -1.07) (layer F.SilkS) (width 0.12))
+    (fp_line (start 1 1.07) (end -1 1.07) (layer F.SilkS) (width 0.12))
+    (fp_line (start -1.6 -0.8) (end 1.6 -0.8) (layer F.Fab) (width 0.1))
+    (fp_line (start 1.6 -0.8) (end 1.6 0.8) (layer F.Fab) (width 0.1))
+    (fp_line (start 1.6 0.8) (end -1.6 0.8) (layer F.Fab) (width 0.1))
+    (fp_line (start -1.6 0.8) (end -1.6 -0.8) (layer F.Fab) (width 0.1))
+    (pad 2 smd rect (at 2.09 0 180) (size 2.03 2.65) (layers F.Cu F.Paste F.Mask)
+      (net 23 +12V))
+    (pad 1 smd rect (at -2.09 0 180) (size 2.03 2.65) (layers F.Cu F.Paste F.Mask)
+      (net 12 "Net-(D2-Pad6)"))
+  )
   (module Blue_ESC:Allegro_PSOF-7_4.8x6.4mm_Pitch1.60mm (layer F.Cu)
-    (at 47.1424 102.9208 270)
+    (at 46 94 270)
     (descr "Allegro Microsystems PSOF-7, 4.8x6.4mm Body, 1.60mm Pitch (http://www.allegromicro.com/~/media/Files/Datasheets/ACS780-Datasheet.ashx)")
     (tags "Allegro PSOF-7")
@@
   )
   (module Blue_ESC:Allegro_PSOF-7_4.8x6.4mm_Pitch1.60mm (layer F.Cu)
-    (at 76.8604 102.9716 270)
+    (at 76 94 270)
     (descr "Allegro Microsystems PSOF-7, 4.8x6.4mm Body, 1.60mm Pitch (http://www.allegromicro.com/~/media/Files/Datasheets/ACS780-Datasheet.ashx)")
     (tags "Allegro PSOF-7")
@@
   )
   (module Blue_ESC:Allegro_PSOF-7_4.8x6.4mm_Pitch1.60mm (layer F.Cu)
-    (at 95.6564 102.9716 270)
+    (at 94 94 270)
     (descr "Allegro Microsystems PSOF-7, 4.8x6.4mm Body, 1.60mm Pitch (http://www.allegromicro.com/~/media/Files/Datasheets/ACS780-Datasheet.ashx)")
     (tags "Allegro PSOF-7")
@@
   )
   (module Blue_ESC:Allegro_PSOF-7_4.8x6.4mm_Pitch1.60mm (layer F.Cu)
-    (at 125.3744 102.9716 270)
+    (at 123 94 270)
     (descr "Allegro Microsystems PSOF-7, 4.8x6.4mm Body, 1.60mm Pitch (http://www.allegromicro.com/~/media/Files/Datasheets/ACS780-Datasheet.ashx)")
     (tags "Allegro PSOF-7")
@@
   )
   (module Fuse_Holders_and_Fuses:Fuse_SMD1206_HandSoldering (layer F.Cu)
-    (at 53.9496 103.0224 90)
+    (at 53 94 90)
     (descr "Fuse, Sicherung, SMD1206, Littlefuse-Wickmann 433 Series, Hand Soldering,")
     (tags "Fuse Sicherung SMD1206 Littlefuse-Wickmann 433 Series Hand Soldering ")
@@
   )
   (module Fuse_Holders_and_Fuses:Fuse_SMD1206_HandSoldering (layer F.Cu)
-    (at 83.6676 103.0732 90)
-    (descr "Fuse, Sicherung, SMD1206, Littlefuse-Wickmann 433 Series, Hand Soldering,")
-    (tags "Fuse Sicherung SMD1206 Littlefuse-Wickmann 433 Series Hand Soldering ")
-    (attr smd)
-    (fp_text reference F2 (at -0.05 -2.2 90) (layer F.SilkS)
-      (effects (font (size 1 1) (thickness 0.15)))
-    )
-    (fp_text value 10/15 (at -0.15 2.5 90) (layer F.Fab)
-      (effects (font (size 1 1) (thickness 0.15)))
-    )
-    (fp_line (start 3.35 1.58) (end -3.35 1.58) (layer F.CrtYd) (width 0.05))
-    (fp_line (start 3.35 1.58) (end 3.35 -1.58) (layer F.CrtYd) (width 0.05))
-    (fp_line (start -3.35 -1.58) (end -3.35 1.58) (layer F.CrtYd) (width 0.05))
-    (fp_line (start -3.35 -1.58) (end 3.35 -1.58) (layer F.CrtYd) (width 0.05))
-    (fp_line (start -1 -1.07) (end 1 -1.07) (layer F.SilkS) (width 0.12))
-    (fp_line (start 1 1.07) (end -1 1.07) (layer F.SilkS) (width 0.12))
-    (fp_line (start -1.6 -0.8) (end 1.6 -0.8) (layer F.Fab) (width 0.1))
-    (fp_line (start 1.6 -0.8) (end 1.6 0.8) (layer F.Fab) (width 0.1))
-    (fp_line (start 1.6 0.8) (end -1.6 0.8) (layer F.Fab) (width 0.1))
-    (fp_line (start -1.6 0.8) (end -1.6 -0.8) (layer F.Fab) (width 0.1))
-    (pad 2 smd rect (at 2.09 0 180) (size 2.03 2.65) (layers F.Cu F.Paste F.Mask)
-      (net 23 +12V))
-    (pad 1 smd rect (at -2.09 0 180) (size 2.03 2.65) (layers F.Cu F.Paste F.Mask)
-      (net 12 "Net-(D2-Pad6)"))
-  )
-  (module Fuse_Holders_and_Fuses:Fuse_SMD1206_HandSoldering (layer F.Cu)
-    (at 102.4636 103.0732 90)
+    (at 102 94 90)
     (descr "Fuse, Sicherung, SMD1206, Littlefuse-Wickmann 433 Series, Hand Soldering,")
     (tags "Fuse Sicherung SMD1206 Littlefuse-Wickmann 433 Series Hand Soldering ")
@@
   )
   (module Fuse_Holders_and_Fuses:Fuse_SMD1206_HandSoldering (layer F.Cu)
-    (at 132.1816 103.124 90)
+    (at 131 94 90)
     (descr "Fuse, Sicherung, SMD1206, Littlefuse-Wickmann 433 Series, Hand Soldering,")
     (tags "Fuse Sicherung SMD1206 Littlefuse-Wickmann 433 Series Hand Soldering ")
@@
   )
   (module Fuse_Holders_and_Fuses:Fuse_SMD1206_HandSoldering (layer F.Cu)
-    (at 169.926 73.9648)
+    (at 170.688 76.2)
     (descr "Fuse, Sicherung, SMD1206, Littlefuse-Wickmann 433 Series, Hand Soldering,")
     (tags "Fuse Sicherung SMD1206 Littlefuse-Wickmann 433 Series Hand Soldering ")
@@
   )
   (module Connectors:RJ45_8 (layer F.Cu)
-    (at 171.0436 83.1088)
+    (at 170.942 84.836)
     (tags RJ45)
     (fp_text reference I1 (at 4.7 11.18) (layer F.SilkS)
@@
   )
   (module Connectors:RJ45_8 (layer F.Cu)
-    (at 171.0436 55.4228)
+    (at 170.942 57.15)
     (tags RJ45)
     (fp_text reference I2 (at 4.7 11.18) (layer F.SilkS)
@@
   )
   (module Blue_ESC:Molex_6pin (layer F.Cu)
-    (at 110.5916 73.3552)
+    (at 110 64)
     (fp_text reference J1 (at 0.127 10.033) (layer F.SilkS)
       (effects (font (size 1 1) (thickness 0.15)))
@@
   )
   (module Blue_ESC:Molex_6pin (layer F.Cu)
-    (at 62.0776 73.3044)
+    (at 62 64)
     (fp_text reference J2 (at 0.127 10.033) (layer F.SilkS)
       (effects (font (size 1 1) (thickness 0.15)))
@@
   )
   (module Blue_ESC:XT60 (layer F.Cu)
-    (at 140.6652 92.8624 90)
+    (at 141 94 90)
     (fp_text reference J3 (at 3.556 6.096 90) (layer F.SilkS)
       (effects (font (size 1 1) (thickness 0.15)))
@@
   )
   (module Mounting_Holes:MountingHole_3mm (layer F.Cu)
-    (at 194.564 152.4)
+    (at 187 105)
     (descr "Mounting Hole 3mm, no annular")
     (tags "mounting hole 3mm no annular")
@@
   )
   (module Mounting_Holes:MountingHole_3mm (layer F.Cu)
-    (at 223.266 151.13)
+    (at 39 105)
     (descr "Mounting Hole 3mm, no annular")
     (tags "mounting hole 3mm no annular")
@@
   )
   (module Mounting_Holes:MountingHole_3mm (layer F.Cu)
-    (at 203.708 150.876)
+    (at 39 49)
     (descr "Mounting Hole 3mm, no annular")
     (tags "mounting hole 3mm no annular")
@@
   )
   (module Mounting_Holes:MountingHole_3mm (layer F.Cu)
-    (at 215.646 152.146)
+    (at 187 49)
     (descr "Mounting Hole 3mm, no annular")
     (tags "mounting hole 3mm no annular")
@@
   )
   (module Blue_ESC:Blue_ESC (layer F.Cu)
-    (at 47.244 79.6925 180)
+    (at 47 70 180)
     (fp_text reference U1 (at 0 10.16 180) (layer F.SilkS)
       (effects (font (size 1 1) (thickness 0.15)))
@@
   )
   (module Blue_ESC:Blue_ESC (layer F.Cu)
-    (at 76.962 79.7052 180)
+    (at 77 70 180)
     (fp_text reference U2 (at 0 10.16 180) (layer F.SilkS)
       (effects (font (size 1 1) (thickness 0.15)))
@@
   )
   (module Blue_ESC:Blue_ESC (layer F.Cu)
-    (at 95.758 79.7052 180)
+    (at 95 70 180)
     (fp_text reference U3 (at 0 10.16 180) (layer F.SilkS)
       (effects (font (size 1 1) (thickness 0.15)))
@@
   )
   (module Blue_ESC:Blue_ESC (layer F.Cu)
-    (at 125.476 79.756 180)
+    (at 125 70 180)
     (fp_text reference U4 (at 0 10.16 180) (layer F.SilkS)
       (effects (font (size 1 1) (thickness 0.15)))
@@
   )
   (module Blue_ESC:Arduino_Nano (layer F.Cu)
-    (at 148.6408 55.4228)
+    (at 149 57)
     (descr "Arduino Nano, http://www.mouser.com/pdfdocs/Gravitech_Arduino_Nano3_0.pdf")
     (tags "Arduino Nano")
@@
     )
   )
+  (gr_line (start 36 46) (end 36 54.7376) (layer Edge.Cuts) (width 0.15))
+  (gr_line (start 36 108) (end 36 54) (layer Edge.Cuts) (width 0.15))
+  (gr_line (start 190 108) (end 36 108) (layer Edge.Cuts) (width 0.15))
+  (gr_line (start 189.992 46) (end 36 46) (layer Edge.Cuts) (width 0.15))
+  (gr_line (start 190 108) (end 190 46) (layer Edge.Cuts) (width 0.15))
 )
