File: ESC-Board/ESC-Board.kicad_pcb (KiCad board)
At the start: 2 copper layers, 154 x 62 mm, 26 parts, among them J1 Molex, J2 Molex, J3 XT_60, U1 ESC:Blue_ESC, U2 ESC:Blue_ESC, U3 ESC:Blue_ESC, U4 ESC:Blue_ESC

Commit message: OOOF
Parts:
- moved I1 13.6 mm to (180.0, 95.0), turned to 180 degrees
Changed lines of the file:
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@@
   )
   (module Connectors:RJ45_8 (layer F.Cu)
-    (at 170.942 84.836)
+    (at 180 95 180)
     (tags RJ45)
-    (fp_text reference I1 (at 4.7 11.18) (layer F.SilkS)
+    (fp_text reference I1 (at 4.7 11.18 180) (layer F.SilkS)
       (effects (font (size 1 1) (thickness 0.15)))
     )
-    (fp_text value RJ45 (at 4.59 6.25) (layer F.Fab)
+    (fp_text value RJ45 (at 4.59 6.25 180) (layer F.Fab)
       (effects (font (size 1 1) (thickness 0.15)))
     )
@@
     (fp_line (start 12.07 -3.81) (end 12.06 5.18) (layer F.SilkS) (width 0.12))
     (fp_line (start -3.17 14.22) (end 12.07 14.22) (layer F.SilkS) (width 0.12))
-    (pad 8 thru_hole circle (at 8.89 -2.54) (size 1.5 1.5) (drill 0.9) (layers *.Cu *.Mask)
+    (pad 8 thru_hole circle (at 8.89 -2.54 180) (size 1.5 1.5) (drill 0.9) (layers *.Cu *.Mask)
       (net 25 "Net-(I1-Pad8)"))
-    (pad 7 thru_hole circle (at 7.62 0) (size 1.5 1.5) (drill 0.9) (layers *.Cu *.Mask)
+    (pad 7 thru_hole circle (at 7.62 0 180) (size 1.5 1.5) (drill 0.9) (layers *.Cu *.Mask)
       (net 26 "Net-(I1-Pad7)"))
-    (pad 6 thru_hole circle (at 6.35 -2.54) (size 1.5 1.5) (drill 0.9) (layers *.Cu *.Mask)
+    (pad 6 thru_hole circle (at 6.35 -2.54 180) (size 1.5 1.5) (drill 0.9) (layers *.Cu *.Mask)
       (net 27 "Net-(I1-Pad6)"))
-    (pad 5 thru_hole circle (at 5.08 0) (size 1.5 1.5) (drill 0.9) (layers *.Cu *.Mask)
+    (pad 5 thru_hole circle (at 5.08 0 180) (size 1.5 1.5) (drill 0.9) (layers *.Cu *.Mask)
       (net 28 "Net-(I1-Pad5)"))
-    (pad 4 thru_hole circle (at 3.81 -2.54) (size 1.5 1.5) (drill 0.9) (layers *.Cu *.Mask)
+    (pad 4 thru_hole circle (at 3.81 -2.54 180) (size 1.5 1.5) (drill 0.9) (layers *.Cu *.Mask)
       (net 29 "Net-(I1-Pad4)"))
-    (pad 3 thru_hole circle (at 2.54 0) (size 1.5 1.5) (drill 0.9) (layers *.Cu *.Mask)
+    (pad 3 thru_hole circle (at 2.54 0 180) (size 1.5 1.5) (drill 0.9) (layers *.Cu *.Mask)
       (net 6 GND))
-    (pad 2 thru_hole circle (at 1.27 -2.54) (size 1.5 1.5) (drill 0.9) (layers *.Cu *.Mask)
+    (pad 2 thru_hole circle (at 1.27 -2.54 180) (size 1.5 1.5) (drill 0.9) (layers *.Cu *.Mask)
       (net 30 I2C_SLC))
-    (pad 1 thru_hole rect (at 0 0) (size 1.5 1.5) (drill 0.9) (layers *.Cu *.Mask)
+    (pad 1 thru_hole rect (at 0 0 180) (size 1.5 1.5) (drill 0.9) (layers *.Cu *.Mask)
       (net 31 I2C_SDA))
-    (pad Hole np_thru_hole circle (at -1.49 6.35) (size 3.65 3.65) (drill 3.25) (layers *.Cu *.SilkS *.Mask))
-    (pad Hole np_thru_hole circle (at 10.38 6.35) (size 3.65 3.65) (drill 3.25) (layers *.Cu *.SilkS *.Mask))
+    (pad Hole np_thru_hole circle (at -1.49 6.35 180) (size 3.65 3.65) (drill 3.25) (layers *.Cu *.SilkS *.Mask))
+    (pad Hole np_thru_hole circle (at 10.38 6.35 180) (size 3.65 3.65) (drill 3.25) (layers *.Cu *.SilkS *.Mask))
     (model ${KISYS3DMOD}/Connectors.3dshapes/RJ45_8.wrl
       (offset (xyz 4.571999931335449 -6.349999904632568 0))
