File: PCS-Board/PCS-Board.sch (KiCad schematic (older format))
At the start: 4 parts

Commit message: PCS Sch cleanup
No changes to sch just cleaning it up
Other:
- note added: "12v_5v_LDO\n"
- note added: "Data and Power\n"
- note added: "I2C Switches\n"
Changed lines of the file:
@@
 L Connector_Generic:Conn_01x04 J?
 U 1 1 5C342410
-P 1200 1900
-F 0 "J?" H 1120 1475 50  0000 C CNN
-F 1 "Conn_01x04" H 1120 1566 50  0000 C CNN
-F 2 "" H 1200 1900 50  0001 C CNN
-F 3 "~" H 1200 1900 50  0001 C CNN
-	1    1200 1900
+P 4750 1950
+F 0 "J?" H 4670 1525 50  0000 C CNN
+F 1 "Conn_01x04" H 4670 1616 50  0000 C CNN
+F 2 "" H 4750 1950 50  0001 C CNN
+F 3 "~" H 4750 1950 50  0001 C CNN
+	1    4750 1950
 	-1   0    0    1
 $EndComp
@@
 L power:GND #PWR?
 U 1 1 5C342702
-P 1400 1900
-F 0 "#PWR?" H 1400 1650 50  0001 C CNN
-F 1 "GND" V 1405 1772 50  0000 R CNN
-F 2 "" H 1400 1900 50  0001 C CNN
-F 3 "" H 1400 1900 50  0001 C CNN
-	1    1400 1900
+P 4950 1950
+F 0 "#PWR?" H 4950 1700 50  0001 C CNN
+F 1 "GND" V 4955 1822 50  0000 R CNN
+F 2 "" H 4950 1950 50  0001 C CNN
+F 3 "" H 4950 1950 50  0001 C CNN
+	1    4950 1950
 	0    -1   -1   0
 $EndComp
@@
 L power:+12V #PWR?
 U 1 1 5C342D6C
-P 1400 2000
-F 0 "#PWR?" H 1400 1850 50  0001 C CNN
-F 1 "+12V" V 1415 2128 50  0000 L CNN
-F 2 "" H 1400 2000 50  0001 C CNN
-F 3 "" H 1400 2000 50  0001 C CNN
-	1    1400 2000
-	0    1    1    0
-$EndComp
-Text GLabel 1400 1700 2    50   Input ~ 0
+P 4950 2050
+F 0 "#PWR?" H 4950 1900 50  0001 C CNN
+F 1 "+12V" V 4965 2178 50  0000 L CNN
+F 2 "" H 4950 2050 50  0001 C CNN
+F 3 "" H 4950 2050 50  0001 C CNN
+	1    4950 2050
+	0    1    1    0
+$EndComp
+Text GLabel 4950 1750 2    50   Input ~ 0
 I2C_SDA
-Text GLabel 1400 1800 2    50   Input ~ 0
+Text GLabel 4950 1850 2    50   Input ~ 0
 I2C_SCL
 $Comp
 L Regulator_Linear:uA7805 U?
 U 1 1 5C3434C8
-P 3600 1700
-F 0 "U?" H 3600 1942 50  0000 C CNN
-F 1 "uA7805" H 3600 1851 50  0000 C CNN
-F 2 "" H 3625 1550 50  0001 L CIN
-F 3 "http://www.ti.com/lit/ds/symlink/ua78.pdf" H 3600 1650 50  0001 C CNN
-	1    3600 1700
+P 6300 1700
+F 0 "U?" H 6300 1942 50  0000 C CNN
+F 1 "uA7805" H 6300 1851 50  0000 C CNN
+F 2 "" H 6325 1550 50  0001 L CIN
+F 3 "http://www.ti.com/lit/ds/symlink/ua78.pdf" H 6300 1650 50  0001 C CNN
+	1    6300 1700
 	1    0    0    -1
 $EndComp
@@
 L power:+12V #PWR?
 U 1 1 5C3437F6
-P 3300 1700
-F 0 "#PWR?" H 3300 1550 50  0001 C CNN
-F 1 "+12V" V 3315 1828 50  0000 L CNN
-F 2 "" H 3300 1700 50  0001 C CNN
-F 3 "" H 3300 1700 50  0001 C CNN
-	1    3300 1700
+P 6000 1700
+F 0 "#PWR?" H 6000 1550 50  0001 C CNN
+F 1 "+12V" V 6015 1828 50  0000 L CNN
+F 2 "" H 6000 1700 50  0001 C CNN
+F 3 "" H 6000 1700 50  0001 C CNN
+	1    6000 1700
 	0    -1   -1   0
 $EndComp
@@
 L power:+5V #PWR?
 U 1 1 5C343835
-P 3900 1700
-F 0 "#PWR?" H 3900 1550 50  0001 C CNN
-F 1 "+5V" V 3915 1828 50  0000 L CNN
-F 2 "" H 3900 1700 50  0001 C CNN
-F 3 "" H 3900 1700 50  0001 C CNN
-	1    3900 1700
+P 6600 1700
+F 0 "#PWR?" H 6600 1550 50  0001 C CNN
+F 1 "+5V" V 6615 1828 50  0000 L CNN
+F 2 "" H 6600 1700 50  0001 C CNN
+F 3 "" H 6600 1700 50  0001 C CNN
+	1    6600 1700
 	0    1    1    0
 $EndComp
@@
 L power:GND #PWR?
 U 1 1 5C343867
-P 3600 2000
-F 0 "#PWR?" H 3600 1750 50  0001 C CNN
-F 1 "GND" H 3605 1827 50  0000 C CNN
-F 2 "" H 3600 2000 50  0001 C CNN
-F 3 "" H 3600 2000 50  0001 C CNN
-	1    3600 2000
+P 6300 2000
+F 0 "#PWR?" H 6300 1750 50  0001 C CNN
+F 1 "GND" H 6305 1827 50  0000 C CNN
+F 2 "" H 6300 2000 50  0001 C CNN
+F 3 "" H 6300 2000 50  0001 C CNN
+	1    6300 2000
 	1    0    0    -1
 $EndComp
@@
 Text GLabel 9600 4700 2    50   Input ~ 0
 SOLN_EN12
+Wire Notes Line
+	10350 1200 10350 6100
+Wire Notes Line
+	10350 6100 7100 6100
+Wire Notes Line
+	7100 6100 7100 1200
+Wire Notes Line
+	7100 1200 10350 1200
+Text Notes 8550 1300 0    50   ~ 0
+I2C Switches\n
+Wire Notes Line
+	5650 1200 6950 1200
+Wire Notes Line
+	6950 1200 6950 2250
+Wire Notes Line
+	6950 2250 5650 2250
+Wire Notes Line
+	5650 1200 5650 2250
+Text Notes 6100 1300 0    50   ~ 0
+12v_5v_LDO\n
+Wire Notes Line
+	4550 2200 5450 2200
+Wire Notes Line
+	5450 2200 5450 1200
+Wire Notes Line
+	5450 1200 4550 1200
+Wire Notes Line
+	4550 1200 4550 2200
+Text Notes 4700 1300 0    50   ~ 0
+Data and Power\n
 $EndSCHEMATC

Commit message: e
Parts:
- gave numbers to parts that had none: 4
Changed lines of the file:
@@
 $EndDescr
 $Comp
-L Analog_Switch:ADG715 U?
+L Analog_Switch:ADG715 U2
 U 1 1 5C342112
 P 8800 2600
-F 0 "U?" H 8800 3778 50  0000 C CNN
+F 0 "U2" H 8800 3778 50  0000 C CNN
 F 1 "ADG715" H 8800 3687 50  0000 C CNN
 F 2 "Package_SO:TSSOP-24_4.4x7.8mm_P0.65mm" H 9800 1850 50  0001 C CIN
@@
 $EndComp
 $Comp
-L Connector_Generic:Conn_01x04 J?
+L Connector_Generic:Conn_01x04 J1
 U 1 1 5C342410
 P 4750 1950
-F 0 "J?" H 4670 1525 50  0000 C CNN
+F 0 "J1" H 4670 1525 50  0000 C CNN
 F 1 "Conn_01x04" H 4670 1616 50  0000 C CNN
 F 2 "" H 4750 1950 50  0001 C CNN
@@
 $EndComp
 $Comp
-L power:GND #PWR?
+L power:GND #PWR0101
 U 1 1 5C342702
 P 4950 1950
-F 0 "#PWR?" H 4950 1700 50  0001 C CNN
+F 0 "#PWR0101" H 4950 1700 50  0001 C CNN
 F 1 "GND" V 4955 1822 50  0000 R CNN
 F 2 "" H 4950 1950 50  0001 C CNN
@@
 I2C_SCL
 $Comp
-L power:+5V #PWR?
+L power:+5V #PWR0102
 U 1 1 5C34290E
 P 8000 2800
-F 0 "#PWR?" H 8000 2650 50  0001 C CNN
+F 0 "#PWR0102" H 8000 2650 50  0001 C CNN
 F 1 "+5V" V 8015 2928 50  0000 L CNN
 F 2 "" H 8000 2800 50  0001 C CNN
@@
 $EndComp
 $Comp
-L power:GND #PWR?
+L power:GND #PWR0103
 U 1 1 5C3429C2
 P 8900 3400
-F 0 "#PWR?" H 8900 3150 50  0001 C CNN
+F 0 "#PWR0103" H 8900 3150 50  0001 C CNN
 F 1 "GND" H 8905 3227 50  0000 C CNN
 F 2 "" H 8900 3400 50  0001 C CNN
@@
 $EndComp
 $Comp
-L power:+12V #PWR?
+L power:+12V #PWR0104
 U 1 1 5C342D6C
 P 4950 2050
-F 0 "#PWR?" H 4950 1900 50  0001 C CNN
+F 0 "#PWR0104" H 4950 1900 50  0001 C CNN
 F 1 "+12V" V 4965 2178 50  0000 L CNN
 F 2 "" H 4950 2050 50  0001 C CNN
@@
 I2C_SCL
 $Comp
-L Regulator_Linear:uA7805 U?
+L Regulator_Linear:uA7805 U1
 U 1 1 5C3434C8
 P 6300 1700
-F 0 "U?" H 6300 1942 50  0000 C CNN
+F 0 "U1" H 6300 1942 50  0000 C CNN
 F 1 "uA7805" H 6300 1851 50  0000 C CNN
 F 2 "" H 6325 1550 50  0001 L CIN
@@
 $EndComp
 $Comp
-L power:+12V #PWR?
+L power:+12V #PWR0105
 U 1 1 5C3437F6
 P 6000 1700
-F 0 "#PWR?" H 6000 1550 50  0001 C CNN
+F 0 "#PWR0105" H 6000 1550 50  0001 C CNN
 F 1 "+12V" V 6015 1828 50  0000 L CNN
 F 2 "" H 6000 1700 50  0001 C CNN
@@
 $EndComp
 $Comp
-L power:+5V #PWR?
+L power:+5V #PWR0106
 U 1 1 5C343835
 P 6600 1700
-F 0 "#PWR?" H 6600 1550 50  0001 C CNN
+F 0 "#PWR0106" H 6600 1550 50  0001 C CNN
 F 1 "+5V" V 6615 1828 50  0000 L CNN
 F 2 "" H 6600 1700 50  0001 C CNN
@@
 $EndComp
 $Comp
-L power:GND #PWR?
+L power:GND #PWR0107
 U 1 1 5C343867
 P 6300 2000
-F 0 "#PWR?" H 6300 1750 50  0001 C CNN
+F 0 "#PWR0107" H 6300 1750 50  0001 C CNN
 F 1 "GND" H 6305 1827 50  0000 C CNN
 F 2 "" H 6300 2000 50  0001 C CNN
@@
 $EndComp
 $Comp
-L power:GND #PWR?
+L power:GND #PWR0108
 U 1 1 5C3441E1
 P 8700 3400
-F 0 "#PWR?" H 8700 3150 50  0001 C CNN
+F 0 "#PWR0108" H 8700 3150 50  0001 C CNN
 F 1 "GND" H 8705 3227 50  0000 C CNN
 F 2 "" H 8700 3400 50  0001 C CNN
@@
 $EndComp
 $Comp
-L power:+5V #PWR?
+L power:+5V #PWR0109
 U 1 1 5C3441FC
 P 8800 1600
-F 0 "#PWR?" H 8800 1450 50  0001 C CNN
+F 0 "#PWR0109" H 8800 1450 50  0001 C CNN
 F 1 "+5V" V 8815 1728 50  0000 L CNN
 F 2 "" H 8800 1600 50  0001 C CNN
@@
 	7800 2500 7800 2400
 $Comp
-L power:+5V #PWR?
+L power:+5V #PWR0110
 U 1 1 5C3447AD
 P 7800 1900
-F 0 "#PWR?" H 7800 1750 50  0001 C CNN
+F 0 "#PWR0110" H 7800 1750 50  0001 C CNN
 F 1 "+5V" V 7815 2028 50  0000 L CNN
 F 2 "" H 7800 1900 50  0001 C CNN
@@
 SOLN_EN7
 $Comp
-L power:GND #PWR?
+L power:GND #PWR0111
 U 1 1 5C3463EA
 P 8000 3100
-F 0 "#PWR?" H 8000 2850 50  0001 C CNN
+F 0 "#PWR0111" H 8000 2850 50  0001 C CNN
 F 1 "GND" V 8005 2972 50  0000 R CNN
 F 2 "" H 8000 3100 50  0001 C CNN
@@
 $EndComp
 $Comp
-L power:GND #PWR?
+L power:GND #PWR0112
 U 1 1 5C346405
 P 8000 3200
-F 0 "#PWR?" H 8000 2950 50  0001 C CNN
+F 0 "#PWR0112" H 8000 2950 50  0001 C CNN
 F 1 "GND" V 8005 3072 50  0000 R CNN
 F 2 "" H 8000 3200 50  0001 C CNN
@@
 $EndComp
 $Comp
-L Analog_Switch:ADG715 U?
+L Analog_Switch:ADG715 U3
 U 1 1 5C3466E2
 P 8800 5000
-F 0 "U?" H 8800 6178 50  0000 C CNN
+F 0 "U3" H 8800 6178 50  0000 C CNN
 F 1 "ADG715" H 8800 6087 50  0000 C CNN
 F 2 "Package_SO:TSSOP-24_4.4x7.8mm_P0.65mm" H 9800 4250 50  0001 C CIN
@@
 I2C_SCL
 $Comp
-L power:+5V #PWR?
+L power:+5V #PWR0113
 U 1 1 5C3466EB
 P 8000 5200
-F 0 "#PWR?" H 8000 5050 50  0001 C CNN
+F 0 "#PWR0113" H 8000 5050 50  0001 C CNN
 F 1 "+5V" V 8015 5328 50  0000 L CNN
 F 2 "" H 8000 5200 50  0001 C CNN
@@
 $EndComp
 $Comp
-L power:GND #PWR?
+L power:GND #PWR0114
 U 1 1 5C3466F1
 P 8900 5800
-F 0 "#PWR?" H 8900 5550 50  0001 C CNN
+F 0 "#PWR0114" H 8900 5550 50  0001 C CNN
 F 1 "GND" H 8905 5627 50  0000 C CNN
 F 2 "" H 8900 5800 50  0001 C CNN
@@
 $EndComp
 $Comp
-L power:GND #PWR?
+L power:GND #PWR0115
 U 1 1 5C3466F7
 P 8700 5800
-F 0 "#PWR?" H 8700 5550 50  0001 C CNN
+F 0 "#PWR0115" H 8700 5550 50  0001 C CNN
 F 1 "GND" H 8705 5627 50  0000 C CNN
 F 2 "" H 8700 5800 50  0001 C CNN
@@
 $EndComp
 $Comp
-L power:+5V #PWR?
+L power:+5V #PWR0116
 U 1 1 5C3466FD
 P 8800 4000
-F 0 "#PWR?" H 8800 3850 50  0001 C CNN
+F 0 "#PWR0116" H 8800 3850 50  0001 C CNN
 F 1 "+5V" V 8815 4128 50  0000 L CNN
 F 2 "" H 8800 4000 50  0001 C CNN
@@
 	7800 4900 7800 4800
 $Comp
-L power:+5V #PWR?
+L power:+5V #PWR0117
 U 1 1 5C346718
 P 7800 4300
-F 0 "#PWR?" H 7800 4150 50  0001 C CNN
+F 0 "#PWR0117" H 7800 4150 50  0001 C CNN
 F 1 "+5V" V 7815 4428 50  0000 L CNN
 F 2 "" H 7800 4300 50  0001 C CNN
@@
 Connection ~ 7800 4300
 $Comp
-L power:GND #PWR?
+L power:GND #PWR0118
 U 1 1 5C34671F
 P 8000 5600
-F 0 "#PWR?" H 8000 5350 50  0001 C CNN
+F 0 "#PWR0118" H 8000 5350 50  0001 C CNN
 F 1 "GND" V 8005 5472 50  0000 R CNN
 F 2 "" H 8000 5600 50  0001 C CNN
@@
 $EndComp
 $Comp
-L power:+5V #PWR?
+L power:+5V #PWR0119
 U 1 1 5C346A10
 P 8000 5500
-F 0 "#PWR?" H 8000 5350 50  0001 C CNN
+F 0 "#PWR0119" H 8000 5350 50  0001 C CNN
 F 1 "+5V" V 8015 5628 50  0000 L CNN
 F 2 "" H 8000 5500 50  0001 C CNN
