File: PCS-Board/PCS-Board.sch (KiCad schematic (older format))
At the start: 4 parts

Commit message: Update to PCS sch
Parts:
- added U?: MMPQ2222A, SOIC127P600X175-16N, symbol MMPQ2222A:MMPQ2222A
Changed lines of the file:
@@
 Text Notes 4700 1300 0    50   ~ 0
 Data and Power\n
+$Comp
+L MMPQ2222A:MMPQ2222A U?
+U 1 1 5C3558EC
+P 3050 3250
+F 0 "U?" H 3050 3920 50  0000 C CNN
+F 1 "MMPQ2222A" H 3050 3829 50  0000 C CNN
+F 2 "SOIC127P600X175-16N" H 3050 3250 50  0001 L BNN
+F 3 "MMPQ2222A" H 3050 3250 50  0001 L BNN
+F 4 "Unavailable" H 3050 3250 50  0001 L BNN "Field4"
+F 5 "MMPQ Series NPN 40 V 500 mA 1000 mW SMT General Purpose Amplifier - SOIC-16" H 3050 3250 50  0001 L BNN "Field5"
+F 6 "SOIC-16 ON Semiconductor" H 3050 3250 50  0001 L BNN "Field6"
+F 7 "ON Semiconductor" H 3050 3250 50  0001 L BNN "Field7"
+F 8 "None" H 3050 3250 50  0001 L BNN "Field8"
+	1    3050 3250
+	1    0    0    -1
+$EndComp
 $EndSCHEMATC

Commit message: Add gates
Parts:
- added U? (x3): MMPQ2222A, SOIC127P600X175-16N, symbol MMPQ2222A:MMPQ2222A
Connections:
- net labels added: SOLN_EN13, SOLN_EN14, SOLN_EN15
Changed lines of the file:
@@
 L MMPQ2222A:MMPQ2222A U?
 U 1 1 5C3558EC
-P 3050 3250
-F 0 "U?" H 3050 3920 50  0000 C CNN
-F 1 "MMPQ2222A" H 3050 3829 50  0000 C CNN
-F 2 "SOIC127P600X175-16N" H 3050 3250 50  0001 L BNN
-F 3 "MMPQ2222A" H 3050 3250 50  0001 L BNN
-F 4 "Unavailable" H 3050 3250 50  0001 L BNN "Field4"
-F 5 "MMPQ Series NPN 40 V 500 mA 1000 mW SMT General Purpose Amplifier - SOIC-16" H 3050 3250 50  0001 L BNN "Field5"
-F 6 "SOIC-16 ON Semiconductor" H 3050 3250 50  0001 L BNN "Field6"
-F 7 "ON Semiconductor" H 3050 3250 50  0001 L BNN "Field7"
-F 8 "None" H 3050 3250 50  0001 L BNN "Field8"
-	1    3050 3250
+P 2050 3950
+F 0 "U?" H 2050 4620 50  0000 C CNN
+F 1 "MMPQ2222A" H 2050 4529 50  0000 C CNN
+F 2 "SOIC127P600X175-16N" H 2050 3950 50  0001 L BNN
+F 3 "MMPQ2222A" H 2050 3950 50  0001 L BNN
+F 4 "Unavailable" H 2050 3950 50  0001 L BNN "Field4"
+F 5 "MMPQ Series NPN 40 V 500 mA 1000 mW SMT General Purpose Amplifier - SOIC-16" H 2050 3950 50  0001 L BNN "Field5"
+F 6 "SOIC-16 ON Semiconductor" H 2050 3950 50  0001 L BNN "Field6"
+F 7 "ON Semiconductor" H 2050 3950 50  0001 L BNN "Field7"
+F 8 "None" H 2050 3950 50  0001 L BNN "Field8"
+	1    2050 3950
 	1    0    0    -1
 $EndComp
+$Comp
+L MMPQ2222A:MMPQ2222A U?
+U 1 1 5C413089
+P 2050 5400
+F 0 "U?" H 2050 6070 50  0000 C CNN
+F 1 "MMPQ2222A" H 2050 5979 50  0000 C CNN
+F 2 "SOIC127P600X175-16N" H 2050 5400 50  0001 L BNN
+F 3 "MMPQ2222A" H 2050 5400 50  0001 L BNN
+F 4 "Unavailable" H 2050 5400 50  0001 L BNN "Field4"
+F 5 "MMPQ Series NPN 40 V 500 mA 1000 mW SMT General Purpose Amplifier - SOIC-16" H 2050 5400 50  0001 L BNN "Field5"
+F 6 "SOIC-16 ON Semiconductor" H 2050 5400 50  0001 L BNN "Field6"
+F 7 "ON Semiconductor" H 2050 5400 50  0001 L BNN "Field7"
+F 8 "None" H 2050 5400 50  0001 L BNN "Field8"
+	1    2050 5400
+	1    0    0    -1
+$EndComp
+$Comp
+L MMPQ2222A:MMPQ2222A U?
+U 1 1 5C413295
+P 4200 3950
+F 0 "U?" H 4200 4620 50  0000 C CNN
+F 1 "MMPQ2222A" H 4200 4529 50  0000 C CNN
+F 2 "SOIC127P600X175-16N" H 4200 3950 50  0001 L BNN
+F 3 "MMPQ2222A" H 4200 3950 50  0001 L BNN
+F 4 "Unavailable" H 4200 3950 50  0001 L BNN "Field4"
+F 5 "MMPQ Series NPN 40 V 500 mA 1000 mW SMT General Purpose Amplifier - SOIC-16" H 4200 3950 50  0001 L BNN "Field5"
+F 6 "SOIC-16 ON Semiconductor" H 4200 3950 50  0001 L BNN "Field6"
+F 7 "ON Semiconductor" H 4200 3950 50  0001 L BNN "Field7"
+F 8 "None" H 4200 3950 50  0001 L BNN "Field8"
+	1    4200 3950
+	1    0    0    -1
+$EndComp
+$Comp
+L MMPQ2222A:MMPQ2222A U?
+U 1 1 5C41331C
+P 4200 5400
+F 0 "U?" H 4200 6070 50  0000 C CNN
+F 1 "MMPQ2222A" H 4200 5979 50  0000 C CNN
+F 2 "SOIC127P600X175-16N" H 4200 5400 50  0001 L BNN
+F 3 "MMPQ2222A" H 4200 5400 50  0001 L BNN
+F 4 "Unavailable" H 4200 5400 50  0001 L BNN "Field4"
+F 5 "MMPQ Series NPN 40 V 500 mA 1000 mW SMT General Purpose Amplifier - SOIC-16" H 4200 5400 50  0001 L BNN "Field5"
+F 6 "SOIC-16 ON Semiconductor" H 4200 5400 50  0001 L BNN "Field6"
+F 7 "ON Semiconductor" H 4200 5400 50  0001 L BNN "Field7"
+F 8 "None" H 4200 5400 50  0001 L BNN "Field8"
+	1    4200 5400
+	1    0    0    -1
+$EndComp
+Text GLabel 9600 4800 2    50   Input ~ 0
+SOLN_EN13
+Text GLabel 9600 4900 2    50   Input ~ 0
+SOLN_EN14
+Text GLabel 9600 5000 2    50   Input ~ 0
+SOLN_EN15
 $EndSCHEMATC

Commit message: Alex is big ghey
Connections:
- net labels added: SOLN_PW0
Changed lines of the file:
@@
 Text GLabel 9600 5000 2    50   Input ~ 0
 SOLN_EN15
+Text GLabel 5300 6200 2    50   Input ~ 0
+SOLN_PW0
+Text GLabel 5600 4300 2    50   Input ~ 0
+SOLN_PW0
 $EndSCHEMATC
