File: PCS-Board/PCS-Board.sch (KiCad schematic (older format))
At the start: 20 parts

Commit message: Began work on pcs board
Parts:
- added MH1, MH2, MH3, MH4: MountingHole, Mounting_Holes:MountingHole_3.2mm_M3, symbol Mechanical:MountingHole
- J1: renamed from J?; footprint (none) -> PCS-Board:Dsub 25pin
- J2: renamed from J?; footprint (none) -> Connectors_Molex:Molex_Mini-Fit_Sr_42819-42XX_1x04_Pitch10.00mm_Vertical
- R1, R10, R11, R12, R2, R3, R4, R5, R6, R7, R8, R9: renamed from R?; footprint (none) -> Resistors_SMD:R_1206
- U4: renamed from U?; footprint (none) -> TO_SOT_Packages_SMD:TO-263-3_TabPin2
- gave numbers to parts that had none: 5

Commit message: Moving to destop
Parts:
- J2: footprint Connectors_Molex:Molex_Mini-Fit_Sr_42819-42XX_1x04_Pitch10.00mm_Vertical -> Connector_Molex:Molex_Micro-Fit_3.0_43045-0415_2x02_P3.00mm_Vertical
- U1, U2, U3: footprint SOIC127P600X175-16N -> .pretty:Soc-16
- U5, U6: footprint Package_SO:TSSOP-24_4.4x7.8mm_P0.65mm -> .pretty:TSSOP-24
Changed lines of the file:
@@
 F 0 "U5" H 9550 3178 50  0000 C CNN
 F 1 "ADG715" H 9550 3087 50  0000 C CNN
-F 2 "Package_SO:TSSOP-24_4.4x7.8mm_P0.65mm" H 10550 1250 50  0001 C CIN
+F 2 ".pretty:TSSOP-24" H 10550 1250 50  0001 C CIN
 F 3 "http://www.analog.com/media/en/technical-documentation/data-sheets/ADG714_715.pdf" H 9550 800 50  0001 C CNN
 	1    9550 2000
@@
 F 0 "J2" H 6920 2025 50  0000 C CNN
 F 1 "Conn_01x04" H 6920 2116 50  0000 C CNN
-F 2 "Connectors_Molex:Molex_Mini-Fit_Sr_42819-42XX_1x04_Pitch10.00mm_Vertical" H 7000 2450 50  0001 C CNN
+F 2 "Connector_Molex:Molex_Micro-Fit_3.0_43045-0415_2x02_P3.00mm_Vertical" H 7000 2450 50  0001 C CNN
 F 3 "~" H 7000 2450 50  0001 C CNN
 	1    7000 2450
@@
 F 0 "U6" H 9550 5578 50  0000 C CNN
 F 1 "ADG715" H 9550 5487 50  0000 C CNN
-F 2 "Package_SO:TSSOP-24_4.4x7.8mm_P0.65mm" H 10550 3650 50  0001 C CIN
+F 2 ".pretty:TSSOP-24" H 10550 3650 50  0001 C CIN
 F 3 "http://www.analog.com/media/en/technical-documentation/data-sheets/ADG714_715.pdf" H 9550 3200 50  0001 C CNN
 	1    9550 4400
@@
 F 0 "U1" H 2250 2220 50  0000 C CNN
 F 1 "MMPQ2222A" H 2250 2129 50  0000 C CNN
-F 2 "SOIC127P600X175-16N" H 2250 1550 50  0001 L BNN
+F 2 ".pretty:Soc-16" H 2250 1550 50  0001 L BNN
 F 3 "MMPQ2222A" H 2250 1550 50  0001 L BNN
 F 4 "Unavailable" H 2250 1550 50  0001 L BNN "Field4"
@@
 F 0 "U2" H 2250 3670 50  0000 C CNN
 F 1 "MMPQ2222A" H 2250 3579 50  0000 C CNN
-F 2 "SOIC127P600X175-16N" H 2250 3000 50  0001 L BNN
+F 2 ".pretty:Soc-16" H 2250 3000 50  0001 L BNN
 F 3 "MMPQ2222A" H 2250 3000 50  0001 L BNN
 F 4 "Unavailable" H 2250 3000 50  0001 L BNN "Field4"
@@
 F 0 "U3" H 4750 2220 50  0000 C CNN
 F 1 "MMPQ2222A" H 4750 2129 50  0000 C CNN
-F 2 "SOIC127P600X175-16N" H 4750 1550 50  0001 L BNN
+F 2 ".pretty:Soc-16" H 4750 1550 50  0001 L BNN
 F 3 "MMPQ2222A" H 4750 1550 50  0001 L BNN
 F 4 "Unavailable" H 4750 1550 50  0001 L BNN "Field4"

Commit message: Wiring has begun Im dead inside
Parts:
- J2: footprint Connector_Molex:Molex_Micro-Fit_3.0_43045-0415_2x02_P3.00mm_Vertical -> Connectors_Molex:Molex_MicroFit_3.0-43045-0410_04x3.00mm_Angled
Changed lines of the file:
@@
 F 0 "J2" H 6920 2025 50  0000 C CNN
 F 1 "Conn_01x04" H 6920 2116 50  0000 C CNN
-F 2 "Connector_Molex:Molex_Micro-Fit_3.0_43045-0415_2x02_P3.00mm_Vertical" H 7000 2450 50  0001 C CNN
+F 2 "Connectors_Molex:Molex_MicroFit_3.0-43045-0410_04x3.00mm_Angled" H 7000 2450 50  0001 C CNN
 F 3 "~" H 7000 2450 50  0001 C CNN
 	1    7000 2450

Commit message: More wiring and sadness
Connections:
- wire segments 51 -> 39
- no-connect marks 17 -> 30
Other:
- note added: "12v to comon postive\nsol 1a to colctor\n"
