File: PCS-Board/_saved_PCS-Board.sch (KiCad schematic (older format))
At the start: 20 parts, among them J1 DB25_Female_MountingHoles, J2 Conn_01x04, U1 MMPQ2222A, U2 MMPQ2222A, U3 MMPQ2222A, U4 uA7805, U5 ADG715, U6 ADG715

Commit message: Began work on pcs board
Parts:
- added MH1, MH2, MH3, MH4: MountingHole, Mounting_Holes:MountingHole_3.2mm_M3, symbol Mechanical:MountingHole
- J2: footprint (none) -> Connectors_Molex:Molex_Mini-Fit_Sr_42819-42XX_1x04_Pitch10.00mm_Vertical
- U1, U2, U3: footprint SOIC127P600X175-16N -> .pretty:Soc-16
Changed lines of the file:
@@
 F 0 "J2" H 6920 2025 50  0000 C CNN
 F 1 "Conn_01x04" H 6920 2116 50  0000 C CNN
-F 2 "" H 7000 2450 50  0001 C CNN
+F 2 "Connectors_Molex:Molex_Mini-Fit_Sr_42819-42XX_1x04_Pitch10.00mm_Vertical" H 7000 2450 50  0001 C CNN
 F 3 "~" H 7000 2450 50  0001 C CNN
 	1    7000 2450
@@
 F 0 "U1" H 2250 2220 50  0000 C CNN
 F 1 "MMPQ2222A" H 2250 2129 50  0000 C CNN
-F 2 "SOIC127P600X175-16N" H 2250 1550 50  0001 L BNN
+F 2 ".pretty:Soc-16" H 2250 1550 50  0001 L BNN
 F 3 "MMPQ2222A" H 2250 1550 50  0001 L BNN
 F 4 "Unavailable" H 2250 1550 50  0001 L BNN "Field4"
@@
 F 0 "U2" H 2250 3670 50  0000 C CNN
 F 1 "MMPQ2222A" H 2250 3579 50  0000 C CNN
-F 2 "SOIC127P600X175-16N" H 2250 3000 50  0001 L BNN
+F 2 ".pretty:Soc-16" H 2250 3000 50  0001 L BNN
 F 3 "MMPQ2222A" H 2250 3000 50  0001 L BNN
 F 4 "Unavailable" H 2250 3000 50  0001 L BNN "Field4"
@@
 F 0 "U3" H 4750 2220 50  0000 C CNN
 F 1 "MMPQ2222A" H 4750 2129 50  0000 C CNN
-F 2 "SOIC127P600X175-16N" H 4750 1550 50  0001 L BNN
+F 2 ".pretty:Soc-16" H 4750 1550 50  0001 L BNN
 F 3 "MMPQ2222A" H 4750 1550 50  0001 L BNN
 F 4 "Unavailable" H 4750 1550 50  0001 L BNN "Field4"
@@
 $EndComp
 Connection ~ 2950 2700
+$Comp
+L Mechanical:MountingHole MH1
+U 1 1 5C4F8D1F
+P 10350 5650
+F 0 "MH1" H 10450 5696 50  0000 L CNN
+F 1 "MountingHole" H 10450 5605 50  0000 L CNN
+F 2 "Mounting_Holes:MountingHole_3.2mm_M3" H 10350 5650 50  0001 C CNN
+F 3 "~" H 10350 5650 50  0001 C CNN
+	1    10350 5650
+	1    0    0    -1
+$EndComp
+$Comp
+L Mechanical:MountingHole MH2
+U 1 1 5C4F8EFA
+P 10350 5850
+F 0 "MH2" H 10450 5896 50  0000 L CNN
+F 1 "MountingHole" H 10450 5805 50  0000 L CNN
+F 2 "Mounting_Holes:MountingHole_3.2mm_M3" H 10350 5850 50  0001 C CNN
+F 3 "~" H 10350 5850 50  0001 C CNN
+	1    10350 5850
+	1    0    0    -1
+$EndComp
+$Comp
+L Mechanical:MountingHole MH3
+U 1 1 5C4F8F40
+P 10350 6050
+F 0 "MH3" H 10450 6096 50  0000 L CNN
+F 1 "MountingHole" H 10450 6005 50  0000 L CNN
+F 2 "Mounting_Holes:MountingHole_3.2mm_M3" H 10350 6050 50  0001 C CNN
+F 3 "~" H 10350 6050 50  0001 C CNN
+	1    10350 6050
+	1    0    0    -1
+$EndComp
+$Comp
+L Mechanical:MountingHole MH4
+U 1 1 5C4F8F84
+P 10350 6250
+F 0 "MH4" H 10450 6296 50  0000 L CNN
+F 1 "MountingHole" H 10450 6205 50  0000 L CNN
+F 2 "Mounting_Holes:MountingHole_3.2mm_M3" H 10350 6250 50  0001 C CNN
+F 3 "~" H 10350 6250 50  0001 C CNN
+	1    10350 6250
+	1    0    0    -1
+$EndComp
 $EndSCHEMATC
