File: PCS-Board/_autosave-PCS-Board.kicad_pcb (KiCad board)
At the start: 2 copper layers, 24 parts, among them J1 DB25_Female_MountingHoles, J2 Conn_01x04, U1 MMPQ2222A, U2 MMPQ2222A, U3 MMPQ2222A, U4 uA7805, U5 ADG715, U6 ADG715

Commit message: Moving to destop
Parts:
- J2: footprint Connectors_Molex:Molex_Mini-Fit_Sr_42819-42XX_1x04_Pitch10.00mm_Vertical -> Connector_Molex:Molex_Micro-Fit_3.0_43045-0410_2x02-1MP_P3.00mm_Horizontal
- moved J2 17.0 mm to (169.0, 98.0)
