File: PCS-Board/PCS-Board.kicad_pcb (KiCad board)
At the start: 2 copper layers, 22 parts, among them J1 DB25_Female_MountingHoles, J2 Conn_01x04, U1 MMPQ2222A, U2 MMPQ2222A, U3 MMPQ2222A, U4 uA7805

Commit message: Moving to destop
Parts:
- added U5: ADG715, .pretty:TSSOP-24, F.Cu at (155.0, 91.0)
- added U6: ADG715, .pretty:TSSOP-24, F.Cu at (155.0, 106.0)
- J2: footprint Connectors_Molex:Molex_Mini-Fit_Sr_42819-42XX_1x04_Pitch10.00mm_Vertical -> Connector_Molex:Molex_Micro-Fit_3.0_43045-0415_2x02_P3.00mm_Vertical
- moved J2 58.2 mm to (175.0, 99.0), turned to 0 degrees
- moved J1 55.1 mm to (110.0, 98.0)
- moved MH1 55.1 mm to (109.0, 60.0)
- moved MH2 55.1 mm to (177.0, 137.0)
- moved MH3 55.1 mm to (109.0, 136.0)
- moved MH4 55.1 mm to (177.0, 61.0)
- moved U1 55.1 mm to (130.0, 98.0)
- moved U2 55.1 mm to (130.0, 84.0)
- moved U3 55.1 mm to (130.0, 112.0)
- moved U4 55.1 mm to (137.0, 132.2)
- moved R1 55.1 mm to (144.4, 94.0)
- moved R10 55.1 mm to (144.4, 111.0)
- moved R11 55.1 mm to (144.4, 114.0)
- moved R12 55.1 mm to (144.4, 117.0)
- moved R2 55.1 mm to (144.4, 97.0)
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
Commit message: Wiring has begun Im dead inside
Parts:
- J2: footprint Connector_Molex:Molex_Micro-Fit_3.0_43045-0415_2x02_P3.00mm_Vertical -> Connectors_Molex:Molex_MicroFit_3.0-43045-0410_04x3.00mm_Angled
- moved J2 28.7 mm to (150.0, 113.0), turned to 270 degrees
- moved U1 24.1 mm to (126.8, 74.1)
- moved R1 24.1 mm to (141.2, 70.1)
- moved R2 24.1 mm to (141.2, 73.1)
- moved R3 24.1 mm to (141.2, 76.1)
- moved R4 24.1 mm to (141.2, 79.1)
- moved MH2 19.0 mm to (159.0, 131.0)
- moved MH4 18.4 mm to (159.0, 65.0)
- moved U4 10.4 mm to (135.0, 122.0)
- moved R10 9.49 mm to (141.4, 102.0)
- moved R11 9.49 mm to (141.4, 105.0)
- moved R12 9.49 mm to (141.4, 108.0)
- moved R9 9.49 mm to (141.4, 99.0), turned to 0 degrees
- moved U3 9.49 mm to (127.0, 103.0)
- moved U5 9.49 mm to (152.0, 82.0), turned to 270 degrees
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Routing:
- net GND: track 0.00 -> 69.0 mm
- net SOLN_PW0: track 0.00 -> 31.2 mm
- net SOLN_PW7: track 0.00 -> 29.8 mm
- net SOLN_PW4: track 0.00 -> 29.3 mm
- net SOLN_PW1: track 0.00 -> 29.0 mm
- net SOLN_PW11: track 0.00 -> 28.1 mm
- net SOLN_PW2: track 0.00 -> 26.4 mm
- net SOLN_PW5: track 0.00 -> 26.2 mm
- net SOLN_PW9: track 0.00 -> 25.6 mm
- net SOLN_PW8: track 0.00 -> 25.0 mm
- net SOLN_PW6: track 0.00 -> 22.9 mm
- net SOLN_PW10: track 0.00 -> 20.6 mm
- net SOLN_EN0: track 0.00 -> 18.1 mm
- net SOLN_EN7: track 0.00 -> 17.2 mm
- net SOLN_EN6: track 0.00 -> 13.7 mm
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Other:
- board outline added: 61 x 74 mm
- net class 12v added: clearance 0.3, trace_width 0.5, via_dia 0.8, via_drill 0.4
- net class GND added: clearance 0.2, trace_width 0.7, via_dia 0.8, via_drill 0.4

Commit message: More wiring and sadness
Connections:
- J1 pad 13: GND -> +12V
- U1 pad 1: +12V -> SOLN_PW0
- U1 pad 10: SOLN_PW2 -> GND
- U1 pad 12: SOLN_PW4 -> GND
- U1 pad 14: SOLN_PW1 -> GND
- U1 pad 16: SOLN_PW0 -> GND
- U1 pad 2: +12V -> Net-(U1-Pad2)
- U1 pad 3: +12V -> SOLN_PW1
- U1 pad 4: +12V -> Net-(U1-Pad4)
- U1 pad 5: +12V -> SOLN_PW2
- U1 pad 6: +12V -> Net-(U1-Pad6)
- U1 pad 7: +12V -> SOLN_PW4
- U1 pad 8: +12V -> Net-(U1-Pad8)
- U2 pad 1: +12V -> Net-(U2-Pad1)
- U2 pad 10: SOLN_PW6 -> GND
- U2 pad 12: SOLN_PW7 -> GND
- U2 pad 14: SOLN_PW5 -> GND
- U2 pad 16: SOLN_PW4 -> GND
- U2 pad 2: +12V -> Net-(U2-Pad2)
- U2 pad 3: +12V -> SOLN_PW5
- U2 pad 4: +12V -> Net-(U2-Pad4)
- U2 pad 5: +12V -> SOLN_PW6
- U2 pad 6: +12V -> Net-(U2-Pad6)
- U2 pad 7: +12V -> SOLN_PW7
- U2 pad 8: +12V -> Net-(U2-Pad8)
- U3 pad 1: +12V -> SOLN_PW8
- U3 pad 10: SOLN_PW10 -> GND
- U3 pad 12: SOLN_PW11 -> GND
- U3 pad 14: SOLN_PW9 -> GND
- U3 pad 16: SOLN_PW8 -> GND
- U3 pad 2: +12V -> Net-(U3-Pad2)
- U3 pad 3: +12V -> SOLN_PW9
- U3 pad 4: +12V -> Net-(U3-Pad4)
- U3 pad 5: +12V -> SOLN_PW10
- U3 pad 6: +12V -> Net-(U3-Pad6)
- U3 pad 7: +12V -> SOLN_PW11
- U3 pad 8: +12V -> Net-(U3-Pad8)
Routing:
- net +5V: track 0.00 -> 141.8 mm
- net GND: track 69.0 -> 149.7 mm
- net +12V: track 0.00 -> 51.1 mm, vias 0 -> 2
- net SOLN_PW11: track 28.1 -> 17.9 mm
- net SOLN_PW7: track 29.8 -> 21.2 mm
- net SOLN_PW9: track 25.6 -> 17.5 mm
- net SOLN_PW8: track 25.0 -> 17.1 mm
- net SOLN_PW0: track 31.2 -> 23.5 mm
- net SOLN_PW5: track 26.2 -> 20.5 mm
- net SOLN_PW1: track 29.0 -> 24.3 mm
- net SOLN_PW10: track 20.6 -> 17.7 mm
- net SOLN_PW4: track 29.3 -> 27.2 mm
- net SOLN_PW2: track 26.4 -> 24.4 mm
- net SOLN_PW6: track 22.9 -> 21.0 mm
- net SOLN_EN7: track 17.2 -> 16.5 mm
Other:
- net class GND: trace_width 0.7 -> 0.5

Commit message: Big oof
Routing:
- net +5V: track 141.8 -> 0.00 mm
- net I2C_SCL: track 0.00 -> 54.9 mm, vias 0 -> 3
- net I2C_SDA: track 0.00 -> 54.3 mm, vias 0 -> 3
- net SOLN_EN11: track 0.00 -> 19.5 mm
- net SOLN_EN8: track 0.00 -> 16.9 mm
- net SOLN_EN9: track 0.00 -> 16.5 mm
- net SOLN_EN10: track 0.00 -> 16.2 mm
Changed lines of the file:
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@@
     (thickness 1.6)
     (drawings 6)
-    (tracks 214)
+    (tracks 244)
     (zones 0)
     (modules 24)
@@
   (segment (start 127.305 101.1) (end 127.4 101.1) (width 0.7) (layer F.Cu) (net 13))
   (segment (start 127.3 101.095) (end 127.305 101.1) (width 0.7) (layer F.Cu) (net 13))
+  (segment (start 147.69 111.5) (end 147.69 108.41) (width 0.25) (layer F.Cu) (net 26) (status 400000))
+  (segment (start 149.725 101.875) (end 149.725 99.85) (width 0.25) (layer F.Cu) (net 26) (status 800000))
+  (segment (start 149.6 102) (end 149.725 101.875) (width 0.25) (layer F.Cu) (net 26))
+  (segment (start 146.5 102) (end 149.6 102) (width 0.25) (layer F.Cu) (net 26))
+  (segment (start 146.5 101.3) (end 146.5 102) (width 0.25) (layer F.Cu) (net 26))
+  (via (at 146.5 101.3) (size 0.8) (drill 0.4) (layers F.Cu B.Cu) (net 26))
+  (segment (start 146.5 107.2) (end 146.5 101.3) (width 0.25) (layer B.Cu) (net 26))
+  (segment (start 147.7 108.4) (end 146.5 107.2) (width 0.25) (layer B.Cu) (net 26))
+  (via (at 147.7 108.4) (size 0.8) (drill 0.4) (layers F.Cu B.Cu) (net 26))
+  (segment (start 147.69 108.41) (end 147.7 108.4) (width 0.25) (layer F.Cu) (net 26))
+  (segment (start 146.5 101.3) (end 146.5 76.1) (width 0.25) (layer B.Cu) (net 26))
+  (segment (start 154.275 75.225) (end 154.275 79.15) (width 0.25) (layer F.Cu) (net 26) (status 800000))
+  (segment (start 154.4 75.1) (end 154.275 75.225) (width 0.25) (layer F.Cu) (net 26))
+  (via (at 154.4 75.1) (size 0.8) (drill 0.4) (layers F.Cu B.Cu) (net 26))
+  (segment (start 147.5 75.1) (end 154.4 75.1) (width 0.25) (layer B.Cu) (net 26))
+  (segment (start 146.5 76.1) (end 147.5 75.1) (width 0.25) (layer B.Cu) (net 26))
+  (segment (start 148.425 99.85) (end 148.425 100.375) (width 0.25) (layer F.Cu) (net 27) (status C00000))
+  (segment (start 150.1 113.6) (end 149.2 114.5) (width 0.25) (layer F.Cu) (net 27))
+  (segment (start 150.1 108.4) (end 150.1 113.6) (width 0.25) (layer F.Cu) (net 27))
+  (segment (start 150.2 108.3) (end 150.1 108.4) (width 0.25) (layer F.Cu) (net 27))
+  (via (at 150.2 108.3) (size 0.8) (drill 0.4) (layers F.Cu B.Cu) (net 27))
+  (segment (start 150.2 103.8) (end 150.2 108.3) (width 0.25) (layer B.Cu) (net 27))
+  (segment (start 147.6 101.2) (end 150.2 103.8) (width 0.25) (layer B.Cu) (net 27))
+  (via (at 147.6 101.2) (size 0.8) (drill 0.4) (layers F.Cu B.Cu) (net 27))
+  (segment (start 148.425 100.375) (end 147.6 101.2) (width 0.25) (layer F.Cu) (net 27) (status 400000))
+  (segment (start 147.69 114.5) (end 149.2 114.5) (width 0.25) (layer F.Cu) (net 27) (status 400000))
+  (segment (start 147.6 101.2) (end 147.6 101.149998) (width 0.25) (layer B.Cu) (net 27))
+  (segment (start 155.575 76.075) (end 155.575 79.15) (width 0.25) (layer F.Cu) (net 27) (status 800000))
+  (segment (start 155.5 76) (end 155.575 76.075) (width 0.25) (layer F.Cu) (net 27))
+  (via (at 155.5 76) (size 0.8) (drill 0.4) (layers F.Cu B.Cu) (net 27))
+  (segment (start 147.4 76) (end 155.5 76) (width 0.25) (layer B.Cu) (net 27))
+  (segment (start 147 76.4) (end 147.4 76) (width 0.25) (layer B.Cu) (net 27))
+  (segment (start 147 100.549998) (end 147 76.4) (width 0.25) (layer B.Cu) (net 27))
+  (segment (start 147.6 101.149998) (end 147 100.549998) (width 0.25) (layer B.Cu) (net 27))
   (segment (start 137.54 116.225) (end 137.54 112.06) (width 0.5) (layer F.Cu) (net 28) (status 400000))
   (segment (start 152.31 109.91) (end 152.31 111.5) (width 0.5) (layer F.Cu) (net 28) (status 800000))
@@
   (segment (start 145.849998 91.050002) (end 151.749998 91.050002) (width 0.25) (layer F.Cu) (net 44))
   (segment (start 143.3 93.6) (end 145.849998 91.050002) (width 0.25) (layer F.Cu) (net 44))
+  (segment (start 142.9 99) (end 144.1 99) (width 0.25) (layer F.Cu) (net 45) (status 400000))
+  (segment (start 151.675 103.525) (end 151.675 99.85) (width 0.25) (layer F.Cu) (net 45) (status 800000))
+  (segment (start 151.2 104) (end 151.675 103.525) (width 0.25) (layer F.Cu) (net 45))
+  (segment (start 145.3 104) (end 151.2 104) (width 0.25) (layer F.Cu) (net 45))
+  (segment (start 144.650002 103.350002) (end 145.3 104) (width 0.25) (layer F.Cu) (net 45))
+  (segment (start 144.650002 99.550002) (end 144.650002 103.350002) (width 0.25) (layer F.Cu) (net 45))
+  (segment (start 144.1 99) (end 144.650002 99.550002) (width 0.25) (layer F.Cu) (net 45))
   (segment (start 129.7 99.825) (end 139.175 99.825) (width 0.25) (layer F.Cu) (net 46) (status 400000))
   (segment (start 139.175 99.825) (end 140 99) (width 0.25) (layer F.Cu) (net 46) (status 800000))
   (segment (start 129.7 102.365) (end 139.635 102.365) (width 0.25) (layer F.Cu) (net 47) (status C00000))
   (segment (start 139.635 102.365) (end 140 102) (width 0.25) (layer F.Cu) (net 47) (status C00000))
+  (segment (start 142.9 102) (end 143.9 102) (width 0.25) (layer F.Cu) (net 48) (status 400000))
+  (segment (start 152.975 104.125) (end 152.975 99.85) (width 0.25) (layer F.Cu) (net 48) (status 800000))
+  (segment (start 152.6 104.5) (end 152.975 104.125) (width 0.25) (layer F.Cu) (net 48))
+  (segment (start 144.8 104.5) (end 152.6 104.5) (width 0.25) (layer F.Cu) (net 48))
+  (segment (start 144.2 103.9) (end 144.8 104.5) (width 0.25) (layer F.Cu) (net 48))
+  (segment (start 144.2 102.3) (end 144.2 103.9) (width 0.25) (layer F.Cu) (net 48))
+  (segment (start 143.9 102) (end 144.2 102.3) (width 0.25) (layer F.Cu) (net 48))
+  (segment (start 142.9 105) (end 153.8 105) (width 0.25) (layer F.Cu) (net 49) (status 400000))
+  (segment (start 154.275 104.525) (end 154.275 99.85) (width 0.25) (layer F.Cu) (net 49) (status 800000))
+  (segment (start 153.8 105) (end 154.275 104.525) (width 0.25) (layer F.Cu) (net 49))
   (segment (start 129.7 104.905) (end 139.905 104.905) (width 0.25) (layer F.Cu) (net 50) (status C00000))
   (segment (start 139.905 104.905) (end 140 105) (width 0.25) (layer F.Cu) (net 50) (status C00000))
+  (segment (start 142.9 108) (end 143.6 108) (width 0.25) (layer F.Cu) (net 51) (status 400000))
+  (segment (start 155.575 104.625) (end 155.575 99.85) (width 0.25) (layer F.Cu) (net 51) (status 800000))
+  (segment (start 154.7 105.5) (end 155.575 104.625) (width 0.25) (layer F.Cu) (net 51))
+  (segment (start 145.050002 105.5) (end 154.7 105.5) (width 0.25) (layer F.Cu) (net 51))
+  (segment (start 144.5 106.050002) (end 145.050002 105.5) (width 0.25) (layer F.Cu) (net 51))
+  (segment (start 144.5 107.1) (end 144.5 106.050002) (width 0.25) (layer F.Cu) (net 51))
+  (segment (start 143.6 108) (end 144.5 107.1) (width 0.25) (layer F.Cu) (net 51))
   (segment (start 129.7 107.445) (end 139.445 107.445) (width 0.25) (layer F.Cu) (net 52) (status 400000))
   (segment (start 139.445 107.445) (end 140 108) (width 0.25) (layer F.Cu) (net 52) (status 800000))
-  (segment (start 149.075 79.15) (end 149.075 82.3) (width 0.25) (layer F.Cu) (net 53) (status 400000))
-  (segment (start 149.075 82.3) (end 149.075 84.85) (width 0.25) (layer F.Cu) (net 53) (status 800000))
-  (segment (start 150.375 84.85) (end 150.375 79.15) (width 0.25) (layer F.Cu) (net 53) (status C00000))
-  (segment (start 149.075 82.3) (end 150.25 82.3) (width 0.25) (layer F.Cu) (net 53))
-  (segment (start 159.9 82.3) (end 157.9 82.3) (width 0.25) (layer F.Cu) (net 53))
-  (segment (start 160.2 82.6) (end 159.9 82.3) (width 0.25) (layer F.Cu) (net 53))
-  (segment (start 160.2 102.7) (end 160.2 96.9) (width 0.25) (layer F.Cu) (net 53))
-  (segment (start 160.2 96.9) (end 160.2 82.6) (width 0.25) (layer F.Cu) (net 53))
-  (segment (start 159.7 103.2) (end 160.2 102.7) (width 0.25) (layer F.Cu) (net 53))
-  (segment (start 151.2 103.2) (end 159.7 103.2) (width 0.25) (layer F.Cu) (net 53))
-  (segment (start 150.1 104.3) (end 151.2 103.2) (width 0.25) (layer F.Cu) (net 53))
-  (segment (start 150.1 108.6) (end 150.1 104.3) (width 0.25) (layer F.Cu) (net 53))
-  (segment (start 149.2 109.5) (end 150.1 108.6) (width 0.25) (layer F.Cu) (net 53))
-  (segment (start 133.6 109.5) (end 149.2 109.5) (width 0.25) (layer F.Cu) (net 53))
-  (segment (start 132.46 110.64) (end 133.6 109.5) (width 0.25) (layer F.Cu) (net 53))
-  (segment (start 132.46 110.64) (end 132.46 116.225) (width 0.25) (layer F.Cu) (net 53) (status 800000))
-  (segment (start 150.25 82.3) (end 157.9 82.3) (width 0.25) (layer F.Cu) (net 53))
-  (segment (start 151.675 79.15) (end 151.675 84.85) (width 0.25) (layer F.Cu) (net 53) (status C00000))
-  (segment (start 152.975 84.85) (end 152.975 79.15) (width 0.25) (layer F.Cu) (net 53) (status C00000))
-  (segment (start 154.925 84.85) (end 154.925 79.15) (width 0.25) (layer F.Cu) (net 53) (status C00000))
-  (segment (start 154.925 99.85) (end 154.925 94.15) (width 0.25) (layer F.Cu) (net 53) (status C00000))
-  (segment (start 153.625 99.85) (end 153.625 94.15) (width 0.25) (layer F.Cu) (net 53) (status C00000))
-  (segment (start 152.325 99.85) (end 152.325 94.15) (width 0.25) (layer F.Cu) (net 53) (status C00000))
-  (segment (start 151.025 99.85) (end 151.025 94.15) (width 0.25) (layer F.Cu) (net 53) (status C00000))
-  (segment (start 149.075 99.85) (end 149.075 94.15) (width 0.25) (layer F.Cu) (net 53) (status C00000))
-  (segment (start 148.425 94.15) (end 148.425 96.525) (width 0.25) (layer F.Cu) (net 53) (status 400000))
-  (segment (start 148.8 96.9) (end 160.2 96.9) (width 0.25) (layer F.Cu) (net 53))
-  (segment (start 148.425 96.525) (end 148.8 96.9) (width 0.25) (layer F.Cu) (net 53))
 )

Commit message: Finalized the Wiring for PCS
Routing:
- net +5V: track 0.00 -> 21.1 mm
- net GND: track 149.7 -> 162.7 mm, vias 0 -> 4
- added copper zone on F.Cu, net +5V
- added copper zone on B.Cu, net GND
Changed lines of the file:
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@@
     (thickness 1.6)
     (drawings 6)
-    (tracks 244)
+    (tracks 293)
     (zones 0)
     (modules 24)
@@
   (segment (start 127.305 101.1) (end 127.4 101.1) (width 0.7) (layer F.Cu) (net 13))
   (segment (start 127.3 101.095) (end 127.305 101.1) (width 0.7) (layer F.Cu) (net 13))
+  (segment (start 150.375 99.85) (end 150.375 101.275) (width 0.5) (layer F.Cu) (net 13) (status 400000))
+  (via (at 150.6 101.5) (size 0.8) (drill 0.4) (layers F.Cu B.Cu) (net 13))
+  (segment (start 150.375 101.275) (end 150.6 101.5) (width 0.5) (layer F.Cu) (net 13))
+  (segment (start 150.375 94.15) (end 150.375 91.925) (width 0.5) (layer F.Cu) (net 13) (status 400000))
+  (via (at 150.4 91.9) (size 0.8) (drill 0.4) (layers F.Cu B.Cu) (net 13))
+  (segment (start 150.375 91.925) (end 150.4 91.9) (width 0.5) (layer F.Cu) (net 13))
+  (segment (start 153.625 84.85) (end 153.625 86.675) (width 0.5) (layer F.Cu) (net 13) (status 400000))
+  (segment (start 155.2 86.7) (end 153.6 86.7) (width 0.5) (layer F.Cu) (net 13))
+  (segment (start 155.575 86.325) (end 155.2 86.7) (width 0.5) (layer F.Cu) (net 13))
+  (segment (start 155.575 86.325) (end 155.575 84.85) (width 0.5) (layer F.Cu) (net 13) (status 800000))
+  (segment (start 153.625 86.675) (end 153.6 86.7) (width 0.5) (layer F.Cu) (net 13))
+  (via (at 153.6 86.7) (size 0.8) (drill 0.4) (layers F.Cu B.Cu) (net 13))
+  (segment (start 154.275 84.85) (end 153.625 84.85) (width 0.5) (layer F.Cu) (net 13) (status C00000))
+  (segment (start 153.625 79.15) (end 153.625 77.425) (width 0.5) (layer F.Cu) (net 13) (status 400000))
+  (via (at 153.3 77.1) (size 0.8) (drill 0.4) (layers F.Cu B.Cu) (net 13))
+  (segment (start 153.625 77.425) (end 153.3 77.1) (width 0.5) (layer F.Cu) (net 13))
+  (segment (start 149.725 94.15) (end 150.375 94.15) (width 0.5) (layer F.Cu) (net 13) (status C00000))
   (segment (start 147.69 111.5) (end 147.69 108.41) (width 0.25) (layer F.Cu) (net 26) (status 400000))
   (segment (start 149.725 101.875) (end 149.725 99.85) (width 0.25) (layer F.Cu) (net 26) (status 800000))
@@
   (segment (start 129.7 107.445) (end 139.445 107.445) (width 0.25) (layer F.Cu) (net 52) (status 400000))
   (segment (start 139.445 107.445) (end 140 108) (width 0.25) (layer F.Cu) (net 52) (status 800000))
+  (segment (start 152.975 79.15) (end 152.975 80.475) (width 0.25) (layer F.Cu) (net 53) (status 400000))
+  (segment (start 152.975 80.475) (end 153 80.5) (width 0.25) (layer F.Cu) (net 53))
+  (segment (start 154.925 79.15) (end 154.925 80.425) (width 0.25) (layer F.Cu) (net 53) (status 400000))
+  (segment (start 154.925 80.425) (end 155 80.5) (width 0.25) (layer F.Cu) (net 53))
+  (segment (start 149.075 79.15) (end 149.075 80.475) (width 0.25) (layer F.Cu) (net 53) (status 400000))
+  (segment (start 149.075 80.475) (end 149.1 80.5) (width 0.25) (layer F.Cu) (net 53))
+  (segment (start 151.675 79.15) (end 151.675 80.475) (width 0.25) (layer F.Cu) (net 53) (status 400000))
+  (segment (start 151.675 80.475) (end 151.7 80.5) (width 0.25) (layer F.Cu) (net 53))
+  (segment (start 150.375 79.15) (end 150.375 80.475) (width 0.25) (layer F.Cu) (net 53) (status 400000))
+  (segment (start 150.375 80.475) (end 150.4 80.5) (width 0.25) (layer F.Cu) (net 53))
+  (segment (start 150.375 84.85) (end 150.375 83.725) (width 0.25) (layer F.Cu) (net 53) (status 400000))
+  (segment (start 150.375 83.725) (end 150.4 83.7) (width 0.25) (layer F.Cu) (net 53))
+  (segment (start 152.975 84.85) (end 152.975 83.625) (width 0.25) (layer F.Cu) (net 53) (status 400000))
+  (segment (start 152.975 83.625) (end 153 83.6) (width 0.25) (layer F.Cu) (net 53))
+  (segment (start 154.925 84.85) (end 154.925 83.675) (width 0.25) (layer F.Cu) (net 53) (status 400000))
+  (segment (start 154.925 83.675) (end 155 83.6) (width 0.25) (layer F.Cu) (net 53))
+  (segment (start 149.075 84.85) (end 149.075 83.725) (width 0.25) (layer F.Cu) (net 53) (status 400000))
+  (segment (start 149.075 83.725) (end 149.1 83.7) (width 0.25) (layer F.Cu) (net 53))
+  (segment (start 151.675 84.85) (end 151.675 83.725) (width 0.25) (layer F.Cu) (net 53) (status 400000))
+  (segment (start 151.675 83.725) (end 151.7 83.7) (width 0.25) (layer F.Cu) (net 53))
+  (segment (start 148.425 94.15) (end 148.425 95.425) (width 0.25) (layer F.Cu) (net 53) (status 400000))
+  (segment (start 148.425 95.425) (end 148.5 95.5) (width 0.25) (layer F.Cu) (net 53))
+  (segment (start 149.075 94.15) (end 149.075 95.475) (width 0.25) (layer F.Cu) (net 53) (status 400000))
+  (segment (start 149.075 95.475) (end 149.1 95.5) (width 0.25) (layer F.Cu) (net 53))
+  (segment (start 151.025 94.15) (end 151.025 95.425) (width 0.25) (layer F.Cu) (net 53) (status 400000))
+  (segment (start 151.025 95.425) (end 151.1 95.5) (width 0.25) (layer F.Cu) (net 53))
+  (segment (start 152.325 94.15) (end 152.325 95.425) (width 0.25) (layer F.Cu) (net 53) (status 400000))
+  (segment (start 152.325 95.425) (end 152.4 95.5) (width 0.25) (layer F.Cu) (net 53))
+  (segment (start 153.625 94.15) (end 153.625 95.425) (width 0.25) (layer F.Cu) (net 53) (status 400000))
+  (segment (start 153.625 95.425) (end 153.7 95.5) (width 0.25) (layer F.Cu) (net 53))
+  (segment (start 154.925 94.15) (end 154.925 95.425) (width 0.25) (layer F.Cu) (net 53) (status 400000))
+  (segment (start 154.925 95.425) (end 155 95.5) (width 0.25) (layer F.Cu) (net 53))
+  (zone (net 53) (net_name +5V) (layer F.Cu) (hatch edge 0.508)
+    (connect_pads yes (clearance 0.508))
+    (min_thickness 0.254)
+    (fill yes (arc_segments 16) (thermal_gap 0.508) (thermal_bridge_width 0.508))
+    (polygon
+      (pts
+        (xy 163 120.5) (xy 130.8 120.5) (xy 130.8 109.4) (xy 146.1 109.4) (xy 146.1 61)
+        (xy 163 61)
+      )
+    )
+  )
+  (zone (net 13) (net_name GND) (layer B.Cu) (hatch edge 0.508)
+    (connect_pads yes (clearance 0.508))
+    (min_thickness 0.254)
+    (fill yes (arc_segments 16) (thermal_gap 0.508) (thermal_bridge_width 0.508))
+    (polygon
+      (pts
+        (xy 163 135) (xy 102 135) (xy 102 61) (xy 163 61)
+      )
+    )
+  )
 )
