File: SP-Board/USP-Board.sch (KiCad schematic (older format))
At the start: 28 parts, among them J1 Conn_01x02, J10 RJ45, J11 RJ45, J2 Conn_01x02, J3 Conn_01x02, J4 Conn_01x02, J6 Conn_01x03, J7 Conn_01x04, J8 Conn_01x03, J9 Conn_01x04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

Commit message: ee
Parts:
- added J?: Conn_02x05_Odd_Even, symbol Connector_Generic:Conn_02x05_Odd_Even
Other:
- note added: "RX 232\n"
- note added: "RX UART (IMU)"
- note added: "TX 232"
- note added: "TX UART (IMU)"
Changed lines of the file:
@@
 NoConn ~ 7400 4450
 NoConn ~ 7400 4550
+$Comp
+L Connector_Generic:Conn_02x05_Odd_Even J?
+U 1 1 5C9EDC18
+P 2450 6200
+F 0 "J?" H 2500 6617 50  0000 C CNN
+F 1 "Conn_02x05_Odd_Even" H 2500 6526 50  0000 C CNN
+F 2 "" H 2450 6200 50  0001 C CNN
+F 3 "~" H 2450 6200 50  0001 C CNN
+	1    2450 6200
+	1    0    0    -1
+$EndComp
+Text Notes 3050 6000 0    50   ~ 0
+TX 232
+Text Notes 3000 6450 0    50   ~ 0
+RX 232\n
+Text Notes 5250 6450 0    50   ~ 0
+TX UART (IMU)
+Text Notes 5250 6000 0    50   ~ 0
+RX UART (IMU)
 $EndSCHEMATC

Commit message: eeeeeeeee
Connections:
- net at U2.11 (T1IN): now also J?.7 (Pin_7)
- net at U2.9 (R2OUT): now also J?.8 (Pin_8)
- no-connect marks 5 -> 13
Changed lines of the file:
@@
 Text Notes 5250 6000 0    50   ~ 0
 RX UART (IMU)
+Wire Wire Line
+	2250 6300 2000 6300
+Wire Wire Line
+	2000 6300 2000 5650
+Wire Wire Line
+	2000 5650 3200 5650
+Wire Wire Line
+	3200 5650 3200 5850
+Wire Wire Line
+	3200 5850 3450 5850
+Wire Wire Line
+	3450 6450 3400 6450
+Wire Wire Line
+	3400 6450 3400 6300
+Wire Wire Line
+	3400 6300 2750 6300
+NoConn ~ 2250 6000
+NoConn ~ 2250 6100
+NoConn ~ 2250 6200
+NoConn ~ 2250 6400
+NoConn ~ 2750 6400
+NoConn ~ 2750 6200
+NoConn ~ 2750 6100
+NoConn ~ 2750 6000
 $EndSCHEMATC

Commit message: Assigining footprints
eeeeeeeeeeeeeeeeeeeeeeeeeeeeeeeeeeeeeeeeeeeeeeeeeeeeeeeeee
Parts:
- added J?: Conn_01x04, symbol Connector_Generic:Conn_01x04
Connections:
- net +5V: now also J?.3 (Pin_3)
- net GND: now also J?.4 (Pin_4)
- net at U2.14 (T1OUT): now also J?.1 (Pin_1)
- net at U2.8 (R2IN): now also J?.2 (Pin_2)
Other:
- moved on the sheet: J6, J7, J8
Changed lines of the file:
@@
 L Connector_Generic:Conn_01x03 J6
 U 1 1 5C6F621E
-P 7200 4550
-F 0 "J6" H 7120 4225 50  0000 C CNN
-F 1 "Conn_01x03" H 7120 4316 50  0000 C CNN
-F 2 "" H 7200 4550 50  0001 C CNN
-F 3 "~" H 7200 4550 50  0001 C CNN
-	1    7200 4550
+P 8050 4550
+F 0 "J6" H 7970 4225 50  0000 C CNN
+F 1 "Conn_01x03" H 7970 4316 50  0000 C CNN
+F 2 "" H 8050 4550 50  0001 C CNN
+F 3 "~" H 8050 4550 50  0001 C CNN
+	1    8050 4550
 	-1   0    0    1
 $EndComp
-Text GLabel 7400 4650 2    50   Input ~ 0
+Text GLabel 8250 4650 2    50   Input ~ 0
 EXT_PWM_LED
 $Comp
 L Connector_Generic:Conn_01x04 J7
 U 1 1 5C6F63B5
-P 7200 5400
-F 0 "J7" H 7120 4975 50  0000 C CNN
-F 1 "Conn_01x04" H 7120 5066 50  0000 C CNN
-F 2 "" H 7200 5400 50  0001 C CNN
-F 3 "~" H 7200 5400 50  0001 C CNN
-	1    7200 5400
+P 8050 5400
+F 0 "J7" H 7970 4975 50  0000 C CNN
+F 1 "Conn_01x04" H 7970 5066 50  0000 C CNN
+F 2 "" H 8050 5400 50  0001 C CNN
+F 3 "~" H 8050 5400 50  0001 C CNN
+	1    8050 5400
 	-1   0    0    1
 $EndComp
-Text GLabel 7400 5200 2    50   Input ~ 0
+Text GLabel 8250 5200 2    50   Input ~ 0
 I2C_SDA
-Text GLabel 7400 5300 2    50   Input ~ 0
+Text GLabel 8250 5300 2    50   Input ~ 0
 I2C_SCL
 $Comp
 L power:GND #PWR0120
 U 1 1 5C6F6B79
-P 7400 5400
-F 0 "#PWR0120" H 7400 5150 50  0001 C CNN
-F 1 "GND" V 7405 5272 50  0000 R CNN
-F 2 "" H 7400 5400 50  0001 C CNN
-F 3 "" H 7400 5400 50  0001 C CNN
-	1    7400 5400
+P 8250 5400
+F 0 "#PWR0120" H 8250 5150 50  0001 C CNN
+F 1 "GND" V 8255 5272 50  0000 R CNN
+F 2 "" H 8250 5400 50  0001 C CNN
+F 3 "" H 8250 5400 50  0001 C CNN
+	1    8250 5400
 	0    -1   -1   0
 $EndComp
@@
 L power:+12V #PWR0121
 U 1 1 5C6F6BA6
-P 7400 5500
-F 0 "#PWR0121" H 7400 5350 50  0001 C CNN
-F 1 "+12V" V 7415 5628 50  0000 L CNN
-F 2 "" H 7400 5500 50  0001 C CNN
-F 3 "" H 7400 5500 50  0001 C CNN
-	1    7400 5500
+P 8250 5500
+F 0 "#PWR0121" H 8250 5350 50  0001 C CNN
+F 1 "+12V" V 8265 5628 50  0000 L CNN
+F 2 "" H 8250 5500 50  0001 C CNN
+F 3 "" H 8250 5500 50  0001 C CNN
+	1    8250 5500
 	0    1    1    0
 $EndComp
@@
 L Connector_Generic:Conn_01x03 J8
 U 1 1 5C6F7BD4
-P 7200 6050
-F 0 "J8" H 7120 5725 50  0000 C CNN
-F 1 "Conn_01x03" H 7120 5816 50  0000 C CNN
-F 2 "" H 7200 6050 50  0001 C CNN
-F 3 "~" H 7200 6050 50  0001 C CNN
-	1    7200 6050
+P 8050 6050
+F 0 "J8" H 7970 5725 50  0000 C CNN
+F 1 "Conn_01x03" H 7970 5816 50  0000 C CNN
+F 2 "" H 8050 6050 50  0001 C CNN
+F 3 "~" H 8050 6050 50  0001 C CNN
+	1    8050 6050
 	-1   0    0    1
 $EndComp
@@
 L power:GND #PWR0122
 U 1 1 5C6F7CC0
-P 7400 5950
-F 0 "#PWR0122" H 7400 5700 50  0001 C CNN
-F 1 "GND" V 7400 5750 50  0000 C CNN
-F 2 "" H 7400 5950 50  0001 C CNN
-F 3 "" H 7400 5950 50  0001 C CNN
-	1    7400 5950
+P 8250 5950
+F 0 "#PWR0122" H 8250 5700 50  0001 C CNN
+F 1 "GND" V 8250 5750 50  0000 C CNN
+F 2 "" H 8250 5950 50  0001 C CNN
+F 3 "" H 8250 5950 50  0001 C CNN
+	1    8250 5950
 	0    -1   -1   0
 $EndComp
@@
 Text GLabel 5650 2150 2    50   Input ~ 0
 I2C_SDA
-Text GLabel 7400 6050 2    50   Input ~ 0
+Text GLabel 8250 6050 2    50   Input ~ 0
 ANLG_HAL_SENS
 Text GLabel 4850 1850 0    50   Input ~ 0
@@
 L power:+5V #PWR0125
 U 1 1 5C998D8E
-P 7400 6150
-F 0 "#PWR0125" H 7400 6000 50  0001 C CNN
-F 1 "+5V" V 7415 6278 50  0000 L CNN
-F 2 "" H 7400 6150 50  0001 C CNN
-F 3 "" H 7400 6150 50  0001 C CNN
-	1    7400 6150
+P 8250 6150
+F 0 "#PWR0125" H 8250 6000 50  0001 C CNN
+F 1 "+5V" V 8265 6278 50  0000 L CNN
+F 2 "" H 8250 6150 50  0001 C CNN
+F 3 "" H 8250 6150 50  0001 C CNN
+	1    8250 6150
 	0    1    1    0
 $EndComp
@@
 	3550 4200 4250 4200
 Connection ~ 4250 4200
-NoConn ~ 7400 4450
-NoConn ~ 7400 4550
+NoConn ~ 8250 4450
+NoConn ~ 8250 4550
 $Comp
 L Connector_Generic:Conn_02x05_Odd_Even J?
@@
 NoConn ~ 2750 6100
 NoConn ~ 2750 6000
+$Comp
+L Connector_Generic:Conn_01x04 J?
+U 1 1 5CAD182A
+P 6650 6000
+F 0 "J?" H 6730 5992 50  0000 L CNN
+F 1 "Conn_01x04" H 6730 5901 50  0000 L CNN
+F 2 "" H 6650 6000 50  0001 C CNN
+F 3 "~" H 6650 6000 50  0001 C CNN
+	1    6650 6000
+	1    0    0    -1
+$EndComp
+Wire Wire Line
+	5050 5850 5800 5850
+Wire Wire Line
+	5800 5850 5800 5900
+Wire Wire Line
+	5800 5900 6450 5900
+Wire Wire Line
+	5050 6450 5150 6450
+Wire Wire Line
+	5150 6450 5150 6050
+Wire Wire Line
+	5150 6050 5850 6050
+Wire Wire Line
+	5850 6050 5850 6000
+Wire Wire Line
+	5850 6000 6450 6000
+$Comp
+L power:+5V #PWR?
+U 1 1 5CAD263E
+P 6450 6100
+F 0 "#PWR?" H 6450 5950 50  0001 C CNN
+F 1 "+5V" V 6465 6228 50  0000 L CNN
+F 2 "" H 6450 6100 50  0001 C CNN
+F 3 "" H 6450 6100 50  0001 C CNN
+	1    6450 6100
+	0    -1   -1   0
+$EndComp
+$Comp
+L power:GND #PWR?
+U 1 1 5CAD26E6
+P 6450 6200
+F 0 "#PWR?" H 6450 5950 50  0001 C CNN
+F 1 "GND" V 6455 6072 50  0000 R CNN
+F 2 "" H 6450 6200 50  0001 C CNN
+F 3 "" H 6450 6200 50  0001 C CNN
+	1    6450 6200
+	0    1    1    0
+$EndComp
 $EndSCHEMATC

Commit message: moving to pc
Parts:
- C1: footprint (none) -> Capacitor_Tantalum_SMD:CP_EIA-1608-08_AVX-J_Pad1.25x1.05mm_HandSolder
- J1, J2, J3, J4: footprint (none) -> 2.54mm_Pin_Headers:PinHeader_1x02_P2.54mm_Vertical
- J12: renamed from J?; footprint (none) -> 2.54mm_Pin_Headers:PinHeader_1x04_P2.54mm_Vertical
- J6, J8: footprint (none) -> 2.54mm_Pin_Headers:PinHeader_1x03_P2.54mm_Vertical
- J7, J9: footprint (none) -> 2.54mm_Pin_Headers:PinHeader_1x04_P2.54mm_Vertical
- R4: footprint (none) -> Resistor_SMD:R_1206_3216Metric_Pad1.42x1.75mm_HandSolder
- U2: footprint (none) -> Package_SO:SOIC-16_3.9x9.9mm_P1.27mm
- gave numbers to parts that had none: 1
Connections:
- no-connect marks 13 -> 18
Changed lines of the file:
@@
 F 0 "R4" H 2380 1504 50  0000 R CNN
 F 1 "240" H 2380 1595 50  0000 R CNN
-F 2 "" V 2380 1550 50  0001 C CNN
+F 2 "Resistor_SMD:R_1206_3216Metric_Pad1.42x1.75mm_HandSolder" V 2380 1550 50  0001 C CNN
 F 3 "~" H 2450 1550 50  0001 C CNN
 	1    2450 1550
@@
 F 0 "J9" H 7220 1525 50  0000 C CNN
 F 1 "Conn_01x04" H 7220 1616 50  0000 C CNN
-F 2 "" H 7300 1950 50  0001 C CNN
+F 2 "2.54mm_Pin_Headers:PinHeader_1x04_P2.54mm_Vertical" H 7300 1950 50  0001 C CNN
 F 3 "~" H 7300 1950 50  0001 C CNN
 	1    7300 1950
@@
 F 0 "J1" H 1420 3375 50  0000 C CNN
 F 1 "Conn_01x02" H 1420 3466 50  0000 C CNN
-F 2 "" H 1500 3700 50  0001 C CNN
+F 2 "2.54mm_Pin_Headers:PinHeader_1x02_P2.54mm_Vertical" H 1500 3700 50  0001 C CNN
 F 3 "~" H 1500 3700 50  0001 C CNN
 	1    1500 3700
@@
 F 0 "J2" H 1420 3825 50  0000 C CNN
 F 1 "Conn_01x02" H 1420 3916 50  0000 C CNN
-F 2 "" H 1500 4150 50  0001 C CNN
+F 2 "2.54mm_Pin_Headers:PinHeader_1x02_P2.54mm_Vertical" H 1500 4150 50  0001 C CNN
 F 3 "~" H 1500 4150 50  0001 C CNN
 	1    1500 4150
@@
 F 0 "J3" H 1420 4275 50  0000 C CNN
 F 1 "Conn_01x02" H 1420 4366 50  0000 C CNN
-F 2 "" H 1500 4600 50  0001 C CNN
+F 2 "2.54mm_Pin_Headers:PinHeader_1x02_P2.54mm_Vertical" H 1500 4600 50  0001 C CNN
 F 3 "~" H 1500 4600 50  0001 C CNN
 	1    1500 4600
@@
 F 0 "J4" H 1420 4725 50  0000 C CNN
 F 1 "Conn_01x02" H 1420 4816 50  0000 C CNN
-F 2 "" H 1500 5050 50  0001 C CNN
+F 2 "2.54mm_Pin_Headers:PinHeader_1x02_P2.54mm_Vertical" H 1500 5050 50  0001 C CNN
 F 3 "~" H 1500 5050 50  0001 C CNN
 	1    1500 5050
@@
 F 0 "J6" H 7970 4225 50  0000 C CNN
 F 1 "Conn_01x03" H 7970 4316 50  0000 C CNN
-F 2 "" H 8050 4550 50  0001 C CNN
+F 2 "2.54mm_Pin_Headers:PinHeader_1x03_P2.54mm_Vertical" H 8050 4550 50  0001 C CNN
 F 3 "~" H 8050 4550 50  0001 C CNN
 	1    8050 4550
@@
 F 0 "J7" H 7970 4975 50  0000 C CNN
 F 1 "Conn_01x04" H 7970 5066 50  0000 C CNN
-F 2 "" H 8050 5400 50  0001 C CNN
+F 2 "2.54mm_Pin_Headers:PinHeader_1x04_P2.54mm_Vertical" H 8050 5400 50  0001 C CNN
 F 3 "~" H 8050 5400 50  0001 C CNN
 	1    8050 5400
@@
 F 0 "J8" H 7970 5725 50  0000 C CNN
 F 1 "Conn_01x03" H 7970 5816 50  0000 C CNN
-F 2 "" H 8050 6050 50  0001 C CNN
+F 2 "2.54mm_Pin_Headers:PinHeader_1x03_P2.54mm_Vertical" H 8050 6050 50  0001 C CNN
 F 3 "~" H 8050 6050 50  0001 C CNN
 	1    8050 6050
@@
 F 0 "C1" H 5342 1296 50  0000 L CNN
 F 1 "C_Small" H 5342 1205 50  0000 L CNN
-F 2 "" H 5250 1250 50  0001 C CNN
+F 2 "Capacitor_Tantalum_SMD:CP_EIA-1608-08_AVX-J_Pad1.25x1.05mm_HandSolder" H 5250 1250 50  0001 C CNN
 F 3 "~" H 5250 1250 50  0001 C CNN
 	1    5250 1250
@@
 F 0 "U2" H 4000 4700 50  0000 C CNN
 F 1 "MAX232" H 4050 6800 50  0000 C CNN
-F 2 "" H 4300 4700 50  0001 L CNN
+F 2 "Package_SO:SOIC-16_3.9x9.9mm_P1.27mm" H 4300 4700 50  0001 L CNN
 F 3 "http://www.ti.com/lit/ds/symlink/max232.pdf" H 4250 5850 50  0001 C CNN
 	1    4250 5750
@@
 NoConn ~ 8250 4550
 $Comp
-L Connector_Generic:Conn_02x05_Odd_Even J?
+L Connector_Generic:Conn_02x05_Odd_Even J5
 U 1 1 5C9EDC18
 P 2450 6200
-F 0 "J?" H 2500 6617 50  0000 C CNN
+F 0 "J5" H 2500 6617 50  0000 C CNN
 F 1 "Conn_02x05_Odd_Even" H 2500 6526 50  0000 C CNN
 F 2 "" H 2450 6200 50  0001 C CNN
@@
 NoConn ~ 2750 6000
 $Comp
-L Connector_Generic:Conn_01x04 J?
+L Connector_Generic:Conn_01x04 J12
 U 1 1 5CAD182A
 P 6650 6000
-F 0 "J?" H 6730 5992 50  0000 L CNN
+F 0 "J12" H 6730 5992 50  0000 L CNN
 F 1 "Conn_01x04" H 6730 5901 50  0000 L CNN
-F 2 "" H 6650 6000 50  0001 C CNN
+F 2 "2.54mm_Pin_Headers:PinHeader_1x04_P2.54mm_Vertical" H 6650 6000 50  0001 C CNN
 F 3 "~" H 6650 6000 50  0001 C CNN
 	1    6650 6000
@@
 	5850 6000 6450 6000
 $Comp
-L power:+5V #PWR?
+L power:+5V #PWR0112
 U 1 1 5CAD263E
 P 6450 6100
-F 0 "#PWR?" H 6450 5950 50  0001 C CNN
+F 0 "#PWR0112" H 6450 5950 50  0001 C CNN
 F 1 "+5V" V 6465 6228 50  0000 L CNN
 F 2 "" H 6450 6100 50  0001 C CNN
@@
 $EndComp
 $Comp
-L power:GND #PWR?
+L power:GND #PWR0113
 U 1 1 5CAD26E6
 P 6450 6200
-F 0 "#PWR?" H 6450 5950 50  0001 C CNN
+F 0 "#PWR0113" H 6450 5950 50  0001 C CNN
 F 1 "GND" V 6455 6072 50  0000 R CNN
 F 2 "" H 6450 6200 50  0001 C CNN
@@
 	0    1    1    0
 $EndComp
+NoConn ~ 5050 6050
+NoConn ~ 5050 6250
+NoConn ~ 3450 6250
+NoConn ~ 3450 6050
+NoConn ~ 9350 7900
 $EndSCHEMATC

Commit message: Needs wires board layout 95%
Parts:
- J5: footprint (none) -> Blue_ESC:Amphenol 98424-G52-10LF
Changed lines of the file:
@@
 F 0 "J5" H 2500 6617 50  0000 C CNN
 F 1 "Conn_02x05_Odd_Even" H 2500 6526 50  0000 C CNN
-F 2 "" H 2450 6200 50  0001 C CNN
+F 2 "Blue_ESC:Amphenol 98424-G52-10LF" H 2450 6200 50  0001 C CNN
 F 3 "~" H 2450 6200 50  0001 C CNN
 	1    2450 6200

Commit message: added xt60
Parts:
- added J13: Conn_01x02, Blue_ESC:XT60, symbol Connector_Generic:Conn_01x02
Connections:
- net +12V: now also J13.2 (Pin_2)
- net GND: now also J13.1 (Pin_1)
Changed lines of the file:
@@
 NoConn ~ 3450 6050
 NoConn ~ 9350 7900
+$Comp
+L Connector_Generic:Conn_01x02 J13
+U 1 1 5CAE7EF4
+P 7500 3400
+F 0 "J13" H 7420 3075 50  0000 C CNN
+F 1 "Conn_01x02" H 7420 3166 50  0000 C CNN
+F 2 "Blue_ESC:XT60" H 7500 3400 50  0001 C CNN
+F 3 "~" H 7500 3400 50  0001 C CNN
+	1    7500 3400
+	-1   0    0    1
+$EndComp
+$Comp
+L power:+12V #PWR0118
+U 1 1 5CAE8AB8
+P 7700 3300
+F 0 "#PWR0118" H 7700 3150 50  0001 C CNN
+F 1 "+12V" V 7715 3428 50  0000 L CNN
+F 2 "" H 7700 3300 50  0001 C CNN
+F 3 "" H 7700 3300 50  0001 C CNN
+	1    7700 3300
+	0    1    1    0
+$EndComp
+$Comp
+L power:GND #PWR0119
+U 1 1 5CAEB9AD
+P 7700 3400
+F 0 "#PWR0119" H 7700 3150 50  0001 C CNN
+F 1 "GND" V 7705 3272 50  0000 R CNN
+F 2 "" H 7700 3400 50  0001 C CNN
+F 3 "" H 7700 3400 50  0001 C CNN
+	1    7700 3400
+	0    -1   -1   0
+$EndComp
 $EndSCHEMATC

Commit message: wiring done
Parts:
- removed H1, H2, H3, H4: MountingHole, MountingHole:MountingHole_3mm_Pad, symbol Mechanical:MountingHole
Changed lines of the file:
@@
 Leak_Sig
-$Comp
-L Mechanical:MountingHole H1
-U 1 1 5C84499E
-P 1200 6150
-F 0 "H1" H 1300 6196 50  0000 L CNN
-F 1 "MountingHole" H 1300 6105 50  0000 L CNN
-F 2 "MountingHole:MountingHole_3mm_Pad" H 1200 6150 50  0001 C CNN
-F 3 "~" H 1200 6150 50  0001 C CNN
-	1    1200 6150
-	1    0    0    -1
-$EndComp
-$Comp
-L Mechanical:MountingHole H2
-U 1 1 5C8449DE
-P 1200 6500
-F 0 "H2" H 1300 6546 50  0000 L CNN
-F 1 "MountingHole" H 1300 6455 50  0000 L CNN
-F 2 "MountingHole:MountingHole_3mm_Pad" H 1200 6500 50  0001 C CNN
-F 3 "~" H 1200 6500 50  0001 C CNN
-	1    1200 6500
-	1    0    0    -1
-$EndComp
-$Comp
-L Mechanical:MountingHole H3
-U 1 1 5C844A42
-P 1200 6900
-F 0 "H3" H 1300 6946 50  0000 L CNN
-F 1 "MountingHole" H 1300 6855 50  0000 L CNN
-F 2 "MountingHole:MountingHole_3mm_Pad" H 1200 6900 50  0001 C CNN
-F 3 "~" H 1200 6900 50  0001 C CNN
-	1    1200 6900
-	1    0    0    -1
-$EndComp
-$Comp
-L Mechanical:MountingHole H4
-U 1 1 5C844AA4
-P 1200 7200
-F 0 "H4" H 1300 7246 50  0000 L CNN
-F 1 "MountingHole" H 1300 7155 50  0000 L CNN
-F 2 "MountingHole:MountingHole_3mm_Pad" H 1200 7200 50  0001 C CNN
-F 3 "~" H 1200 7200 50  0001 C CNN
-	1    1200 7200
-	1    0    0    -1
-$EndComp
 $Comp
 L power:+5V #PWR0125
